Commit message: Corrected wheel dimensions

File: rover_desc_pkg/urdf/wheel.urdf.xacro (robot description, xacro)
@@ -2,6 +2,6 @@
 <robot name="wheel" xmlns:xacro="http://www.ros.org/wiki/xacro">
     <!-- Wheels -->
-    <xacro:property name="wheel_radius" value="0.18"/>
-    <xacro:property name="wheel_height" value="0.12"/>
+    <xacro:property name="wheel_radius" value="0.178"/>
+    <xacro:property name="wheel_height" value="0.114"/>
     <xacro:property name="wheel_mass" value="1.0"/> <!-- in Kg -->
     <xacro:property name="base_x_origin_to_wheel_origin" value="0.25"/>

Commit message: Removed xacro properties and included joints_links file.

File: rover_desc_pkg/urdf/wheel.urdf.xacro (robot description, xacro)
@@ -1,16 +1,8 @@
 <?xml version="1.0"?>
 <robot name="wheel" xmlns:xacro="http://www.ros.org/wiki/xacro">
-    <!-- Wheels -->
-    <xacro:property name="wheel_radius" value="0.178"/>
-    <xacro:property name="wheel_height" value="0.114"/>
-    <xacro:property name="wheel_mass" value="1.0"/> <!-- in Kg -->
-    <xacro:property name="base_x_origin_to_wheel_origin" value="0.25"/>
-    <xacro:property name="base_y_origin_to_wheel_origin" value="0.3"/>
-    <xacro:property name="base_z_origin_to_wheel_origin" value="0.0"/>
-    <xacro:macro name="cylinder_inertia" params="m r h">
-        <intertia ixx="${m*(3*r*r+h*h)/12}" ixy="0.0" ixz="0.0"
-                  iyy="${m*(3*r*r+h*h)/12}" iyz="0.0"
-                  izz="${m*r*r/2}"/>
-    </xacro:macro>
+    <!-- Begin - Include -->
+    <xacro:include filename="$(find rover_desc_pkg)/urdf/robot_parameters.xacro"/>
+    <xacro:include filename="$(find rover_desc_pkg)/urdf/links_joints.xacro"/>
+    <!-- End - Include -->
     <xacro:macro name="wheel" params="fb ls parent translateX translateY flipY"> <!-- fb: front, back; ls: left, right -->
         <link name="${fb}_{ls}_wheel">

Commit message: Modified wheels macro

File: rover_desc_pkg/urdf/wheel.urdf.xacro (robot description, xacro)
@@ -5,6 +5,6 @@
     <xacro:include filename="$(find rover_desc_pkg)/urdf/links_joints.xacro"/>
     <!-- End - Include -->
-    <xacro:macro name="wheel" params="fb ls parent translateX translateY flipY"> <!-- fb: front, back; ls: left, right -->
-        <link name="${fb}_{ls}_wheel">
+    <xacro:macro name="wheel" params="fb lr parent translateX translateY"> <!-- fb: front, back; lr: left, right -->
+        <!-- <link name="${fb}_{ls}_wheel">
             <visual>
                 <origin xyz="0 0 0" rpy="${flipY*M_PI/2} 0 0"/>
@@ -25,6 +25,24 @@
                 </inertial>
             </visual>
-        </link>
-        <joint name="${fb}_{ls}_wheel_joint" type="continuous">
+        </link> -->
+        <m_joint name="${r_link_01_name}__${fb}_{ls}_wheel" type="fixed"
+                 axis_xyz="0 0 0"
+                 origin_rpy="0 0 0" origin_xyz="${translateX * base_x_origin_to_wheel_origin} ${translateY * base_y_origin_to_wheel_origin} ${wheel_radius/2}"
+                 parent="${parent}" child="${fb}_{ls}_wheel"
+                 limit_e="0" limit_l="0" limit_u="0" limit_v="0"/>
+        <m_link_mesh name="${fb}_{ls}_wheel"
+                     color="Black"
+                     origin_rpy="0 0 0" origin_xyz="${translateX * base_x_origin_to_wheel_origin} ${translateY * base_y_origin_to_wheel_origin} ${wheel_radius/2}"
+                     mass="1.0"
+                     ixx="0.0001" ixy="0.0" ixz="0.0"
+                     iyy="0.0001" iyz="0.0"
+                     izz="0.0001"
+                     meshfile="package://rover_desc_pkg/meshes/rover_wheel.stl"
+                     meshscale="1 1 1"/>
+        <gazebo reference="${fb}_{ls}_wheel">
+            <material>Gazebo/Black</material>
+            <turnGravityOff>false</turnGravityOff>
+        </gazebo>
+        <!-- <joint name="${fb}_{ls}_wheel_joint" type="continuous">
             <parent link="${parent}"/>
             <child link="${fb}_{lr}_wheel"/>
@@ -35,7 +53,7 @@
             <limit effort="100" velocity="100"/>
             <joint_properties damping="0.0" friction="0.0"/>
-        </joint>
+        </joint> -->
         <!-- Transmission is important to link the joints and the controller -->
-        <transmission name="${fb}_${lr}_wheel_joint_trans">
+        <!-- <transmission name="${fb}_${lr}_wheel_joint_trans">
             <type>transmission_interface/SimpleTransmission</type>
             <joint name="${fb}_${lr}_wheel_joint"/>
@@ -44,5 +62,5 @@
                 <mechanicalReduction>1</mechanicalReduction>
             </actuator>
-        </transmission>
+        </transmission> -->
     </xacro:macro>
 </robot>

Commit message: Fixed various syntax errors

File: rover_desc_pkg/urdf/wheel.urdf.xacro (robot description, xacro)
@@ -5,6 +5,6 @@
     <xacro:include filename="$(find rover_desc_pkg)/urdf/links_joints.xacro"/>
     <!-- End - Include -->
-    <xacro:macro name="wheel" params="fb lr parent translateX translateY"> <!-- fb: front, back; lr: left, right -->
-        <!-- <link name="${fb}_{ls}_wheel">
+    <xacro:macro name="wheel" params="fr lr parent translateX translateY"> <!-- fr: front, rear; lr: left, right -->
+        <!-- <link name="${fr}_${lr}_wheel">
             <visual>
                 <origin xyz="0 0 0" rpy="${flipY*M_PI/2} 0 0"/>
@@ -26,10 +26,10 @@
             </visual>
         </link> -->
-        <m_joint name="${r_link_01_name}__${fb}_{ls}_wheel" type="fixed"
+        <m_joint name="${r_link_01_name}__${fr}_${lr}_wheel" type="fixed"
                  axis_xyz="0 0 0"
                  origin_rpy="0 0 0" origin_xyz="${translateX * base_x_origin_to_wheel_origin} ${translateY * base_y_origin_to_wheel_origin} ${wheel_radius/2}"
-                 parent="${parent}" child="${fb}_{ls}_wheel"
+                 parent="${parent}" child="${fr}_${lr}_wheel"
                  limit_e="0" limit_l="0" limit_u="0" limit_v="0"/>
-        <m_link_mesh name="${fb}_{ls}_wheel"
+        <m_link_mesh name="${fr}_${lr}_wheel"
                      color="Black"
                      origin_rpy="0 0 0" origin_xyz="${translateX * base_x_origin_to_wheel_origin} ${translateY * base_y_origin_to_wheel_origin} ${wheel_radius/2}"
@@ -40,11 +40,11 @@
                      meshfile="package://rover_desc_pkg/meshes/rover_wheel.stl"
                      meshscale="1 1 1"/>
-        <gazebo reference="${fb}_{ls}_wheel">
+        <gazebo reference="${fr}_${lr}_wheel">
             <material>Gazebo/Black</material>
             <turnGravityOff>false</turnGravityOff>
         </gazebo>
-        <!-- <joint name="${fb}_{ls}_wheel_joint" type="continuous">
+        <!-- <joint name="${fr}_${lr}_wheel_joint" type="continuous">
             <parent link="${parent}"/>
-            <child link="${fb}_{lr}_wheel"/>
+            <child link="${fr}_${lr}_wheel"/>
             <origin xyz="${translateX * base_x_origin_to_wheel_origin}
                          ${translateY * base_y_origin_to_wheel_origin}
@@ -55,8 +55,8 @@
         </joint> -->
         <!-- Transmission is important to link the joints and the controller -->
-        <!-- <transmission name="${fb}_${lr}_wheel_joint_trans">
+        <!-- <transmission name="${fr}_${lr}_wheel_joint_trans">
             <type>transmission_interface/SimpleTransmission</type>
-            <joint name="${fb}_${lr}_wheel_joint"/>
-            <actuator name="${fb}_{lr}_wheel_joint_motor">
+            <joint name="${fr}_${lr}_wheel_joint"/>
+            <actuator name="${fr}_${lr}_wheel_joint_motor">
                 <hardwareInterface>EffortJointInterface</hardwareInterface>
                 <mechanicalReduction>1</mechanicalReduction>

Commit message: Cleaned up the file

File: rover_desc_pkg/urdf/wheel.urdf.xacro (robot description, xacro)
@@ -6,27 +6,7 @@
     <!-- End - Include -->
     <xacro:macro name="wheel" params="fr lr parent translateX translateY"> <!-- fr: front, rear; lr: left, right -->
-        <!-- <link name="${fr}_${lr}_wheel">
-            <visual>
-                <origin xyz="0 0 0" rpy="${flipY*M_PI/2} 0 0"/>
-                <geometry>
-                    <cylinder length="${wheel_height}" radius="${wheel_radius}"/>
-                </geometry>
-                <material name="DarkGrey"/>
-                <collision>
-                    <origin xyz="0 0 0" rpy="${flipY*M_PI/2} 0 0"/>
-                    <geometry>
-                        <cylinder length="${wheel_height}" radius="${wheel_radius}"/>
-                    </geometry>
-                </collision>
-                <inertial>
-                    <origin xyz="0 0 0"/>
-                    <mass value="${wheel_mass}"/>
-                    <cylinder_inertia m="${wheel_mass}" r="${wheel_radius}" h="${wheel_height}"/>
-                </inertial>
-            </visual>
-        </link> -->
         <m_joint name="${r_link_01_name}__${fr}_${lr}_wheel" type="fixed"
                  axis_xyz="0 0 0"
-                 origin_rpy="0 0 0" origin_xyz="${translateX * base_x_origin_to_wheel_origin} ${translateY * base_y_origin_to_wheel_origin} ${wheel_radius/2}"
+                 origin_rpy="0 0 0" origin_xyz="0 0 0"
                  parent="${parent}" child="${fr}_${lr}_wheel"
                  limit_e="0" limit_l="0" limit_u="0" limit_v="0"/>
@@ -38,5 +18,5 @@
                      iyy="0.0001" iyz="0.0"
                      izz="0.0001"
-                     meshfile="package://rover_desc_pkg/meshes/rover_wheel.stl"
+                     meshfile="package://rover_desc_pkg/meshes/rover_wheel.dae"
                      meshscale="1 1 1"/>
         <gazebo reference="${fr}_${lr}_wheel">
@@ -44,14 +24,4 @@
             <turnGravityOff>false</turnGravityOff>
         </gazebo>
-        <!-- <joint name="${fr}_${lr}_wheel_joint" type="continuous">
-            <parent link="${parent}"/>
-            <child link="${fr}_${lr}_wheel"/>
-            <origin xyz="${translateX * base_x_origin_to_wheel_origin}
-                         ${translateY * base_y_origin_to_wheel_origin}
-                         ${base_z_origin_to_wheel_origin}" rpy="0 0 0"/>
-            <axis xyz="0 1 0" rpy="0 0 0"/>
-            <limit effort="100" velocity="100"/>
-            <joint_properties damping="0.0" friction="0.0"/>
-        </joint> -->
         <!-- Transmission is important to link the joints and the controller -->
         <!-- <transmission name="${fr}_${lr}_wheel_joint_trans">

Commit message: Changed visual for Gazebo

File: rover_desc_pkg/urdf/wheel.urdf.xacro (robot description, xacro)
@@ -21,5 +21,11 @@
                      meshscale="1 1 1"/>
         <gazebo reference="${fr}_${lr}_wheel">
-            <material>Gazebo/Black</material>
+            <visual name="${fr}_${lr}_wheel_visual">
+                <material>
+                    <ambient>0.5 0.5 0.5 1.0</ambient>
+                    <specular>0.8 0.8 0.8 0.1</specular>
+                    <diffuse>1.0 1.0 1.0 1.0</diffuse>
+                </material>
+            </visual>
             <turnGravityOff>false</turnGravityOff>
         </gazebo>
