Commit message: Added inverter properties and dimension. Added green color.

File: rover_desc_pkg/urdf/robot_parameters.xacro (robot description, xacro)
@@ -3,4 +3,5 @@
     <xacro:property name="r_link_00_name" value="chassis_footprint"/>
     <xacro:property name="r_link_01_name" value="chassis_link"/>
+    <xacro:property name="r_link_02_name" value="inverter_link"/>
     <!-- Color parameters -->
     <material name="Black">
@@ -16,12 +17,20 @@
         <color rgba="${0.0/255} ${0.0/255} ${204/255} ${255/255}"/>
     </material>
+    <material name="Green">
+        <color rgba="${0.0/255} ${204/255} ${0.0/255} ${255/255}"/>
+    </material>
     <!-- All the units are in m-kg-s-radians unit system -->
     <xacro:property name="M_PI" value="3.141592653"/>
     <xacro:property name="DEG_TO_RAD" value="0.017453293"/>
-    <!-- Main body dimensions -->
+    <!-- Chassis dimensions -->
     <xacro:property name="chassis_length" value="1.016"/>
     <xacro:property name="chassis_width" value="0.6096"/>
     <xacro:property name="chassis_height" value="0.4445"/>
     <xacro:property name="chassis_mass" value="5"/> <!-- in Kg -->
+    <!-- Inverter dimensions -->
+    <xacro:property name="inverter_length" value="0.400"/>
+    <xacro:property name="inverter_width" value="0.2353"/>
+    <xacro:property name="inverter_height" value="0.400"/>
+    <xacro:property name="inverter_mass" value="5"/> <!-- in Kg -->
     <!-- Wheels -->
     <xacro:property name="wheel_radius" value="0.178"/>

Commit message: Calculated correct values for the parameters

File: rover_desc_pkg/urdf/robot_parameters.xacro (robot description, xacro)
@@ -37,7 +37,7 @@
     <xacro:property name="wheel_height" value="0.114"/>
     <xacro:property name="wheel_mass" value="1.0"/> <!-- in Kg -->
-    <xacro:property name="base_x_origin_to_wheel_origin" value="0.25"/>
-    <xacro:property name="base_y_origin_to_wheel_origin" value="0.3"/>
-    <xacro:property name="base_z_origin_to_wheel_origin" value="0.0"/>
+    <xacro:property name="base_x_origin_to_wheel_origin" value="0.413"/>
+    <xacro:property name="base_y_origin_to_wheel_origin" value="0.430"/>
+    <xacro:property name="base_z_origin_to_wheel_origin" value="0.339"/>
     <xacro:macro name="cylinder_inertia" params="m r h">
         <intertia ixx="${m*(3*r*r+h*h)/12}" ixy="0.0" ixz="0.0"

Commit message: Corrected color macros

File: rover_desc_pkg/urdf/robot_parameters.xacro (robot description, xacro)
@@ -5,19 +5,34 @@
     <xacro:property name="r_link_02_name" value="inverter_link"/>
     <!-- Color parameters -->
-    <material name="Black">
-        <color rgba="${0.0/255} ${0.0/255} ${0.0/255} ${255/255}"/>
-    </material>
-    <material name="Red">
-        <color rgba="${204/255} ${0.0/255} ${0.0/255} ${255/255}"/>
-    </material>
-    <material name="White">
-        <color rgba="${255/255} ${255/255} ${255/255} ${255/255}"/>
-    </material>
-    <material name="Blue">
-        <color rgba="${0.0/255} ${0.0/255} ${204/255} ${255/255}"/>
-    </material>
-    <material name="Green">
-        <color rgba="${0.0/255} ${204/255} ${0.0/255} ${255/255}"/>
-    </material>
+    <xacro:property name="Red_Value" value="{204/255} ${0.0/255} ${0.0/255} ${255/255}"/>
+    <xacro:property name="Green_Value" value="${0.0/255} ${204/255} ${0.0/255} ${255/255}"/>
+    <xacro:property name="Blue_Value" value="${0.0/255} ${0.0/255} ${204/255} ${255/255}"/>
+    <xacro:property name="Black_Value" value="${0.0/255} ${0.0/255} ${0.0/255} ${255/255}"/>
+    <xacro:property name="White_Value" value="${255/255} ${255/255} ${255/255} ${255/255}"/>
+    <xacro:macro name="Red">
+        <material name="">
+            <color rgba="${Red_Value}"/>
+        </material>
+    </xacro:macro>
+    <xacro:macro name="Green">
+        <material name="">
+            <color rgba="${Green_Value}"/>
+        </material>
+    </xacro:macro>
+    <xacro:macro name="Blue">
+        <material name="">
+            <color rgba="${Blue_Value}"/>
+        </material>
+    </xacro:macro>
+    <xacro:macro name="Black">
+        <material name="">
+            <color rgba="${Black_Value}"/>
+        </material>
+    </xacro:macro>
+    <xacro:macro name="White">
+        <material name="">
+            <color rgba="${White_Value}"/>
+        </material>
+    </xacro:macro>
     <!-- All the units are in m-kg-s-radians unit system -->
     <xacro:property name="M_PI" value="3.141592653"/>

Commit message: Removed inverter link and added steer link. Renamed wheel.urdf.xacro to wheel.xacro.

File: rover_desc_pkg/urdf/robot_parameters.xacro (robot description, xacro)
@@ -3,5 +3,5 @@
     <xacro:property name="r_link_00_name" value="chassis_footprint"/>
     <xacro:property name="r_link_01_name" value="chassis_link"/>
-    <xacro:property name="r_link_02_name" value="inverter_link"/>
+    <xacro:property name="r_link_02_name" value="steer_link"/>
     <!-- Color parameters -->
     <xacro:property name="Red_Value" value="{204/255} ${0.0/255} ${0.0/255} ${255/255}"/>

File: rover_desc_pkg/urdf/rover_robot.xacro (robot description, xacro)
@@ -4,5 +4,6 @@
     <xacro:include filename="$(find rover_desc_pkg)/urdf/robot_parameters.xacro"/>
     <xacro:include filename="$(find rover_desc_pkg)/urdf/links_joints.xacro"/>
-    <xacro:include filename="$(find rover_desc_pkg)/urdf/wheel.urdf.xacro"/>
+    <xacro:include filename="$(find rover_desc_pkg)/urdf/steer.xacro"/>
+    <xacro:include filename="$(find rover_desc_pkg)/urdf/wheel.xacro"/>
     <!-- End - Include -->
     <!-- Begin - Robot Description -->
@@ -43,33 +44,13 @@
         <turnGravityOff>false</turnGravityOff>
     </gazebo>
-    <m_joint name="${r_link_01_name}__${r_link_02_name}" type="fixed"
-             axis_xyz="0 0 0"
-             origin_rpy="0 0 0" origin_xyz="0 0 0"
-             parent="${r_link_01_name}" child="${r_link_02_name}"
-             limit_e="0" limit_l="0" limit_u="0" limit_v="0"/>
-    <m_link_mesh name="${r_link_02_name}"
-                 color="Green"
-                 origin_rpy="0 0 0" origin_xyz="${(chassis_length/2)-(inverter_length/2)-0.03} 0 ${inverter_height/2}"
-                 mass="1.0"
-                 ixx="0.0001" ixy="0.0" ixz="0.0"
-                 iyy="0.0001" iyz="0.0"
-                 izz="0.0001"
-                 meshfile="package://rover_desc_pkg/meshes/inverter.dae"
-                 meshscale="1 1 1"/>
-    <gazebo reference="${r_link_02_name}">
-        <visual name="${r_link_02_name}_visual">
-            <material>
-                <ambient>0.5 0.5 0.5 1.0</ambient>
-                <specular>0.8 0.8 0.8 0.1</specular>
-                <diffuse>1.0 1.0 1.0 1.0</diffuse>
-            </material>
-        </visual>
-        <turnGravityOff>false</turnGravityOff>
-    </gazebo>
-    <!-- Wheel -->
-    <wheel fr="front" lr="right" parent="${r_link_01_name}" translateX="1" translateY="-1"/>
-    <wheel fr="front" lr="left" parent="${r_link_01_name}" translateX="1" translateY="1"/>
-    <wheel fr="rear" lr="right" parent="${r_link_01_name}" translateX="-1" translateY="-1"/>
-    <wheel fr="rear" lr="left" parent="${r_link_01_name}" translateX="-1" translateY="1"/>
+    <!-- Steers & Wheels -->
+    <steer fr="front" lr="right" type="fixed" parent="${r_link_01_name}" translateX="1" translateY="-1"/>
+    <wheel fr="front" lr="right" parent="front_right_steer" translateX="1" translateY="-1"/>
+    <steer fr="front" lr="left" type="fixed" parent="${r_link_01_name}" translateX="1" translateY="1"/>
+    <wheel fr="front" lr="left" parent="front_left_steer" translateX="1" translateY="1"/>
+    <steer fr="rear" lr="right" type="fixed" parent="${r_link_01_name}" translateX="-1" translateY="-1"/>
+    <wheel fr="rear" lr="right" parent="rear_right_steer" translateX="-1" translateY="-1"/>
+    <steer fr="rear" lr="left" type="fixed" parent="${r_link_01_name}" translateX="-1" translateY="1"/>
+    <wheel fr="rear" lr="left" parent="rear_left_steer" translateX="-1" translateY="1"/>
     <!-- End - Robot Description -->
     <!-- Rover -->

Commit message: Added steer assembly parameters.

File: rover_desc_pkg/urdf/robot_parameters.xacro (robot description, xacro)
@@ -48,4 +48,12 @@
     <xacro:property name="inverter_height" value="0.400"/>
     <xacro:property name="inverter_mass" value="5"/> <!-- in Kg -->
+    <!-- Steer dimensions -->
+    <xacro:property name="steer_length" value="0.217"/>
+    <xacro:property name="steer_width" value="0.234"/>
+    <xacro:property name="steer_height" value="0.618"/>
+    <xacro:property name="steer_mass" value="5"/> <!-- in Kg -->
+    <xacro:property name="chassis_x_origin_to_steer_x_origin" value="0.3715"/> <!-- Distance from chassis origin to mount point in X direction -->
+    <xacro:property name="chassis_y_origin_to_steer_y_origin" value="0.3148"/> <!-- Distance from chassis origin to mount point in Y direction -->
+    <xacro:property name="chassis_z_origin_to_steer_z_origin" value="0.1305"/> <!-- Distance from chassis origin to mount point in Z direction -->
     <!-- Wheels -->
     <xacro:property name="wheel_radius" value="0.178"/>

Commit message: Renamed wheel origin parameters

File: rover_desc_pkg/urdf/robot_parameters.xacro (robot description, xacro)
@@ -60,7 +60,7 @@
     <xacro:property name="wheel_height" value="0.114"/>
     <xacro:property name="wheel_mass" value="1.0"/> <!-- in Kg -->
-    <xacro:property name="base_x_origin_to_wheel_origin" value="0.413"/>
-    <xacro:property name="base_y_origin_to_wheel_origin" value="0.430"/>
-    <xacro:property name="base_z_origin_to_wheel_origin" value="0.339"/>
+    <xacro:property name="chassis_x_origin_to_wheel_x_origin" value="0.413"/>
+    <xacro:property name="chassis_y_origin_to_wheel_y_origin" value="0.3153"/>
+    <xacro:property name="chassis_z_origin_to_wheel_z_origin" value="0.339"/>
     <xacro:macro name="cylinder_inertia" params="m r h">
         <intertia ixx="${m*(3*r*r+h*h)/12}" ixy="0.0" ixz="0.0"

Commit message: Renamed origin parameters with correct reference frames.

File: rover_desc_pkg/urdf/robot_parameters.xacro (robot description, xacro)
@@ -43,4 +43,7 @@
     <xacro:property name="chassis_height" value="0.4445"/>
     <xacro:property name="chassis_mass" value="5"/> <!-- in Kg -->
+    <xacro:property name="world_x_origin_to_chassis_x_origin" value="0.0"/>
+    <xacro:property name="world_y_origin_to_chassis_y_origin" value="0.0"/>
+    <xacro:property name="world_z_origin_to_chassis_z_origin" value="0.0"/>
     <!-- Inverter dimensions -->
     <xacro:property name="inverter_length" value="0.400"/>
@@ -53,14 +56,16 @@
     <xacro:property name="steer_height" value="0.618"/>
     <xacro:property name="steer_mass" value="5"/> <!-- in Kg -->
-    <xacro:property name="chassis_x_origin_to_steer_x_origin" value="0.3715"/> <!-- Distance from chassis origin to mount point in X direction -->
-    <xacro:property name="chassis_y_origin_to_steer_y_origin" value="0.3148"/> <!-- Distance from chassis origin to mount point in Y direction -->
-    <xacro:property name="chassis_z_origin_to_steer_z_origin" value="0.1305"/> <!-- Distance from chassis origin to mount point in Z direction -->
+    <xacro:property name="world_x_origin_to_steer_x_origin" value="0.3715"/> <!-- Distance from world origin to mount point in X direction -->
+    <xacro:property name="world_y_origin_to_steer_y_origin" value="0.3148"/> <!-- Distance from world origin to mount point in Y direction -->
+    <xacro:property name="world_z_origin_to_steer_z_origin" value="0.0"/> <!-- Distance from world origin to mount point in Z direction -->
+    <xacro:property name="chassis_z_origin_to_steer_z_origin" value="0.1305"/>
     <!-- Wheels -->
     <xacro:property name="wheel_radius" value="0.178"/>
     <xacro:property name="wheel_height" value="0.114"/>
     <xacro:property name="wheel_mass" value="1.0"/> <!-- in Kg -->
-    <xacro:property name="chassis_x_origin_to_wheel_x_origin" value="0.413"/>
-    <xacro:property name="chassis_y_origin_to_wheel_y_origin" value="0.3153"/>
-    <xacro:property name="chassis_z_origin_to_wheel_z_origin" value="0.339"/>
+    <xacro:property name="world_x_origin_to_wheel_x_origin" value="0.4025"/>
+    <xacro:property name="world_y_origin_to_wheel_y_origin" value="0.3153"/>
+    <xacro:property name="world_z_origin_to_wheel_z_origin" value="0.0"/>
+    <xacro:property name="steer_z_origin_to_wheel_z_origin" value="0.4625"/>
     <xacro:macro name="cylinder_inertia" params="m r h">
         <intertia ixx="${m*(3*r*r+h*h)/12}" ixy="0.0" ixz="0.0"

Commit message: Defined wheel position relative to steer position.

File: rover_desc_pkg/urdf/robot_parameters.xacro (robot description, xacro)
@@ -3,5 +3,4 @@
   <xacro:property name="r_link_00_name" value="chassis_footprint"/>
   <xacro:property name="r_link_01_name" value="chassis_link"/>
-  <xacro:property name="r_link_02_name" value="steer_link"/>
   <!-- Color parameters -->
   <xacro:property name="Red_Value" value="${204/255} ${0.0/255} ${0.0/255} ${255/255}"/>
@@ -67,5 +66,7 @@
   <xacro:property name="world_y_origin_to_wheel_y_origin" value="0.3153"/>
   <xacro:property name="world_z_origin_to_wheel_z_origin" value="0.0"/>
-  <xacro:property name="steer_z_origin_to_wheel_z_origin" value="0.4625"/>
+  <xacro:property name="steer_x_origin_to_wheel_x_origin" value="0.0317"/>
+  <xacro:property name="steer_y_origin_to_wheel_y_origin" value="0.0"/>
+  <xacro:property name="steer_z_origin_to_wheel_z_origin" value="0.4620"/>
   <xacro:macro name="cylinder_inertia" params="m r h">
     <intertia ixx="${m*(3*r*r+h*h)/12}" ixy="0.0" ixz="0.0"

Commit message: Fixed color macros.

File: rover_desc_pkg/urdf/robot_parameters.xacro (robot description, xacro)
@@ -4,32 +4,42 @@
   <xacro:property name="r_link_01_name" value="chassis_link"/>
   <!-- Color parameters -->
-  <xacro:property name="Red_Value" value="${204/255} ${0.0/255} ${0.0/255} ${255/255}"/>
-  <xacro:property name="Green_Value" value="${0.0/255} ${204/255} ${0.0/255} ${255/255}"/>
-  <xacro:property name="Blue_Value" value="${0.0/255} ${0.0/255} ${204/255} ${255/255}"/>
-  <xacro:property name="Black_Value" value="${0.0/255} ${0.0/255} ${0.0/255} ${255/255}"/>
-  <xacro:property name="White_Value" value="${255/255} ${255/255} ${255/255} ${255/255}"/>
-  <xacro:macro name="Red">
+  <xacro:macro name="red">
     <material name="">
-      <color rgba="${Red_Value}"/>
+      <color rgba="${204/255} ${0.0/255} ${0.0/255} ${255/255}"/>
     </material>
   </xacro:macro>
-  <xacro:macro name="Green">
+  <xacro:macro name="green">
     <material name="">
-      <color rgba="${Green_Value}"/>
+      <color rgba="${0.0/255} ${204/255} ${0.0/255} ${255/255}"/>
     </material>
   </xacro:macro>
-  <xacro:macro name="Blue">
+  <xacro:macro name="blue">
     <material name="">
-      <color rgba="${Blue_Value}"/>
+      <color rgba="${0.0/255} ${0.0/255} ${204/255} ${255/255}"/>
     </material>
   </xacro:macro>
-  <xacro:macro name="Black">
+  <xacro:macro name="black">
     <material name="">
-      <color rgba="${Black_Value}"/>
+      <color rgba="${0.0/255} ${0.0/255} ${0.0/255} ${255/255}"/>
     </material>
   </xacro:macro>
-  <xacro:macro name="White">
+  <xacro:macro name="white">
     <material name="">
-      <color rgba="${White_Value}"/>
+      <color rgba="${255/255} ${255/255} ${255/255} ${255/255}"/>
+    </material>
+  </xacro:macro>
+  <xacro:macro name="gray">
+    <material name="">
+      <color rgba="${178.5/255} ${178.5/255} ${178.5/255} ${255/255}"/>
+    </material>
+  </xacro:macro>
+  <xacro:macro name="darkgray">
+    <material name="">
+      <color rgba="${76.5/255} ${76.5/255} ${76.5/255} ${255/255}"/>
+    </material>
+  </xacro:macro>
+  <xacro:macro name="yellow">
+    <material name="">
+      <color rgba="${204/255} ${204/255} ${204/255} ${255/255}"/>
     </material>
   </xacro:macro>
