Commit message: Added steer description.

File: rover_desc_pkg/urdf/steer.xacro (robot description, xacro)
@@ -1,25 +1,25 @@
 <?xml version="1.0"?>
-<robot name="wheel" xmlns:xacro="http://www.ros.org/wiki/xacro">
+<robot name="steer" xmlns:xacro="http://www.ros.org/wiki/xacro">
     <!-- Begin - Include -->
     <xacro:include filename="$(find rover_desc_pkg)/urdf/robot_parameters.xacro"/>
     <xacro:include filename="$(find rover_desc_pkg)/urdf/links_joints.xacro"/>
     <!-- End - Include -->
-    <xacro:macro name="wheel" params="fr lr parent translateX translateY"> <!-- fr: front, rear; lr: left, right -->
-        <m_joint name="${r_link_01_name}__${fr}_${lr}_wheel" type="fixed"
+    <xacro:macro name="steer" params="fr lr type parent translateX translateY"> <!-- fr: front, rear; lr: left, right -->
+        <m_joint name="${parent}__${fr}_${lr}_steer" type="${type}"
                  axis_xyz="0 0 0"
                  origin_rpy="0 0 0" origin_xyz="0 0 0"
-                 parent="${parent}" child="${fr}_${lr}_wheel"
+                 parent="${parent}" child="${fr}_${lr}_steer"
                  limit_e="0" limit_l="0" limit_u="0" limit_v="0"/>
-        <m_link_mesh name="${fr}_${lr}_wheel"
-                     color="Black"
-                     origin_rpy="0 0 0" origin_xyz="${translateX * base_x_origin_to_wheel_origin} ${translateY * base_y_origin_to_wheel_origin} ${wheel_radius/2}"
+        <m_link_mesh name="${fr}_${lr}_steer"
+                     color="White"
+                     origin_rpy="0 0 0" origin_xyz="0 0 ${(chassis_height/2) + 0.1397}"
                      mass="1.0"
                      ixx="0.0001" ixy="0.0" ixz="0.0"
                      iyy="0.0001" iyz="0.0"
                      izz="0.0001"
-                     meshfile="package://rover_desc_pkg/meshes/rover_wheel.dae"
+                     meshfile="package://rover_desc_pkg/meshes/rover_steer.dae"
                      meshscale="1 1 1"/>
-        <gazebo reference="${fr}_${lr}_wheel">
-            <visual name="${fr}_${lr}_wheel_visual">
+        <gazebo reference="${fr}_${lr}_steer">
+            <visual name="${fr}_${lr}_steer_visual">
                 <material>
                     <ambient>0.5 0.5 0.5 1.0</ambient>
@@ -31,8 +31,8 @@
         </gazebo>
         <!-- Transmission is important to link the joints and the controller -->
-        <!-- <transmission name="${fr}_${lr}_wheel_joint_trans">
+        <!-- <transmission name="${fr}_${lr}_steer_joint_trans">
             <type>transmission_interface/SimpleTransmission</type>
-            <joint name="${fr}_${lr}_wheel_joint"/>
-            <actuator name="${fr}_${lr}_wheel_joint_motor">
+            <joint name="${fr}_${lr}_steer_joint"/>
+            <actuator name="${fr}_${lr}_steer_joint_motor">
                 <hardwareInterface>EffortJointInterface</hardwareInterface>
                 <mechanicalReduction>1</mechanicalReduction>

Commit message: Separate macro for front and rear.

File: rover_desc_pkg/urdf/steer.xacro (robot description, xacro)
@@ -5,13 +5,16 @@
     <xacro:include filename="$(find rover_desc_pkg)/urdf/links_joints.xacro"/>
     <!-- End - Include -->
-    <xacro:macro name="steer" params="fr lr type parent translateX translateY"> <!-- fr: front, rear; lr: left, right -->
-        <m_joint name="${parent}__${fr}_${lr}_steer" type="${type}"
+    <xacro:macro name="steer_f" params="lr parent translateX translateY"> <!-- lr: left, right -->
+        <m_joint name="${parent}__front_${lr}_steer" type="fixed"
                  axis_xyz="0 0 0"
                  origin_rpy="0 0 0" origin_xyz="0 0 0"
-                 parent="${parent}" child="${fr}_${lr}_steer"
+                 parent="${parent}" child="front_${lr}_steer"
                  limit_e="0" limit_l="0" limit_u="0" limit_v="0"/>
-        <m_link_mesh name="${fr}_${lr}_steer"
+        <m_link_mesh name="front_${lr}_steer"
                      color="White"
-                     origin_rpy="0 0 0" origin_xyz="0 0 ${(chassis_height/2) + 0.1397}"
+                     origin_rpy="0 0 0"
+                     origin_xyz="${translateX * chassis_x_origin_to_steer_x_origin}
+                                 ${translateY * chassis_y_origin_to_steer_y_origin}
+                                 ${(chassis_height/2) + chassis_z_origin_to_steer_z_origin}"
                      mass="1.0"
                      ixx="0.0001" ixy="0.0" ixz="0.0"
@@ -20,6 +23,6 @@
                      meshfile="package://rover_desc_pkg/meshes/rover_steer.dae"
                      meshscale="1 1 1"/>
-        <gazebo reference="${fr}_${lr}_steer">
-            <visual name="${fr}_${lr}_steer_visual">
+        <gazebo reference="front_${lr}_steer">
+            <visual name="front_${lr}_steer_visual">
                 <material>
                     <ambient>0.5 0.5 0.5 1.0</ambient>
@@ -31,8 +34,46 @@
         </gazebo>
         <!-- Transmission is important to link the joints and the controller -->
-        <!-- <transmission name="${fr}_${lr}_steer_joint_trans">
+        <!-- <transmission name="front_${lr}_steer_joint_trans">
             <type>transmission_interface/SimpleTransmission</type>
-            <joint name="${fr}_${lr}_steer_joint"/>
-            <actuator name="${fr}_${lr}_steer_joint_motor">
+            <joint name="front_${lr}_steer_joint"/>
+            <actuator name="front_${lr}_steer_joint_motor">
+                <hardwareInterface>EffortJointInterface</hardwareInterface>
+                <mechanicalReduction>1</mechanicalReduction>
+            </actuator>
+        </transmission> -->
+    </xacro:macro>
+    <xacro:macro name="steer_r" params="lr parent translateX translateY"> <!-- lr: left, right -->
+        <m_joint name="${parent}__rear_${lr}_steer" type="fixed"
+                 axis_xyz="0 0 0"
+                 origin_rpy="0 0 0" origin_xyz="0 0 0"
+                 parent="${parent}" child="rear_${lr}_steer"
+                 limit_e="0" limit_l="0" limit_u="0" limit_v="0"/>
+        <m_link_mesh name="rear_${lr}_steer"
+                     color="White"
+                     origin_rpy="0 0 0"
+                     origin_xyz="${translateX * (chassis_x_origin_to_steer_x_origin + 0.063)}
+                                 ${translateY * chassis_y_origin_to_steer_y_origin}
+                                 ${(chassis_height/2) + chassis_z_origin_to_steer_z_origin}"
+                     mass="1.0"
+                     ixx="0.0001" ixy="0.0" ixz="0.0"
+                     iyy="0.0001" iyz="0.0"
+                     izz="0.0001"
+                     meshfile="package://rover_desc_pkg/meshes/rover_steer.dae"
+                     meshscale="1 1 1"/>
+        <gazebo reference="rear_${lr}_steer">
+            <visual name="rear_${lr}_steer_visual">
+                <material>
+                    <ambient>0.5 0.5 0.5 1.0</ambient>
+                    <specular>0.8 0.8 0.8 0.1</specular>
+                    <diffuse>1.0 1.0 1.0 1.0</diffuse>
+                </material>
+            </visual>
+            <turnGravityOff>false</turnGravityOff>
+        </gazebo>
+        <!-- Transmission is important to link the joints and the controller -->
+        <!-- <transmission name="rear_${lr}_steer_joint_trans">
+            <type>transmission_interface/SimpleTransmission</type>
+            <joint name="rear_${lr}_steer_joint"/>
+            <actuator name="rear_${lr}_steer_joint_motor">
                 <hardwareInterface>EffortJointInterface</hardwareInterface>
                 <mechanicalReduction>1</mechanicalReduction>

Commit message: Position steer along X depending on front and rear. Choose steer mesh file depending on right and left.

File: rover_desc_pkg/urdf/steer.xacro (robot description, xacro)
@@ -5,24 +5,46 @@
     <xacro:include filename="$(find rover_desc_pkg)/urdf/links_joints.xacro"/>
     <!-- End - Include -->
-    <xacro:macro name="steer_f" params="lr parent translateX translateY"> <!-- lr: left, right -->
-        <m_joint name="${parent}__front_${lr}_steer" type="fixed"
+    <xacro:macro name="steer" params="fr lr parent translateX translateY"> <!-- fr: front, rear; lr: left, right -->
+        <!-- Compute steer position based on its location -->
+        <xacro:if value="${fr == 'front'}">
+            <xacro:property name="origin_steer"
+                            value="${translateX * chassis_x_origin_to_steer_x_origin}
+                                   ${translateY * chassis_y_origin_to_steer_y_origin}
+                                   ${(chassis_height/2) + chassis_z_origin_to_steer_z_origin}"/>
+        </xacro:if>
+        <xacro:if value="${fr == 'rear'}">
+            <xacro:property name="origin_steer"
+                            value="${translateX * (chassis_x_origin_to_steer_x_origin + 0.063)}
+                                   ${translateY * chassis_y_origin_to_steer_y_origin}
+                                   ${(chassis_height/2) + chassis_z_origin_to_steer_z_origin}"/>
+        </xacro:if>
+        <!-- Decide steer mesh file based on its location -->
+        <xacro:if value="${lr == 'right'}">
+            <xacro:property name="mesh_file"
+                            value="package://rover_desc_pkg/meshes/rover_steer_r.dae"/>
+        </xacro:if>
+        <xacro:if value="${lr == 'left'}">
+            <xacro:property name="mesh_file"
+                            value="package://rover_desc_pkg/meshes/rover_steer_l.dae"/>
+        </xacro:if>
+        <!-- Joint description -->
+        <m_joint name="${parent}__${fr}_${lr}_steer" type="fixed"
                  axis_xyz="0 0 0"
                  origin_rpy="0 0 0" origin_xyz="0 0 0"
-                 parent="${parent}" child="front_${lr}_steer"
+                 parent="${parent}" child="${fr}_${lr}_steer"
                  limit_e="0" limit_l="0" limit_u="0" limit_v="0"/>
-        <m_link_mesh name="front_${lr}_steer"
+        <!-- Link description -->
+        <m_link_mesh name="${fr}_${lr}_steer"
                      color="White"
                      origin_rpy="0 0 0"
-                     origin_xyz="${translateX * chassis_x_origin_to_steer_x_origin}
-                                 ${translateY * chassis_y_origin_to_steer_y_origin}
-                                 ${(chassis_height/2) + chassis_z_origin_to_steer_z_origin}"
+                     origin_xyz="${origin_steer}"
                      mass="1.0"
                      ixx="0.0001" ixy="0.0" ixz="0.0"
                      iyy="0.0001" iyz="0.0"
                      izz="0.0001"
-                     meshfile="package://rover_desc_pkg/meshes/rover_steer.dae"
+                     meshfile="${mesh_file}"
                      meshscale="1 1 1"/>
-        <gazebo reference="front_${lr}_steer">
-            <visual name="front_${lr}_steer_visual">
+        <gazebo reference="${fr}_${lr}_steer">
+            <visual name="${fr}_${lr}_steer_visual">
                 <material>
                     <ambient>0.5 0.5 0.5 1.0</ambient>
@@ -34,46 +56,8 @@
         </gazebo>
         <!-- Transmission is important to link the joints and the controller -->
-        <!-- <transmission name="front_${lr}_steer_joint_trans">
+        <!-- <transmission name="${fr}_${lr}_steer_joint_trans">
             <type>transmission_interface/SimpleTransmission</type>
-            <joint name="front_${lr}_steer_joint"/>
-            <actuator name="front_${lr}_steer_joint_motor">
-                <hardwareInterface>EffortJointInterface</hardwareInterface>
-                <mechanicalReduction>1</mechanicalReduction>
-            </actuator>
-        </transmission> -->
-    </xacro:macro>
-    <xacro:macro name="steer_r" params="lr parent translateX translateY"> <!-- lr: left, right -->
-        <m_joint name="${parent}__rear_${lr}_steer" type="fixed"
-                 axis_xyz="0 0 0"
-                 origin_rpy="0 0 0" origin_xyz="0 0 0"
-                 parent="${parent}" child="rear_${lr}_steer"
-                 limit_e="0" limit_l="0" limit_u="0" limit_v="0"/>
-        <m_link_mesh name="rear_${lr}_steer"
-                     color="White"
-                     origin_rpy="0 0 0"
-                     origin_xyz="${translateX * (chassis_x_origin_to_steer_x_origin + 0.063)}
-                                 ${translateY * chassis_y_origin_to_steer_y_origin}
-                                 ${(chassis_height/2) + chassis_z_origin_to_steer_z_origin}"
-                     mass="1.0"
-                     ixx="0.0001" ixy="0.0" ixz="0.0"
-                     iyy="0.0001" iyz="0.0"
-                     izz="0.0001"
-                     meshfile="package://rover_desc_pkg/meshes/rover_steer.dae"
-                     meshscale="1 1 1"/>
-        <gazebo reference="rear_${lr}_steer">
-            <visual name="rear_${lr}_steer_visual">
-                <material>
-                    <ambient>0.5 0.5 0.5 1.0</ambient>
-                    <specular>0.8 0.8 0.8 0.1</specular>
-                    <diffuse>1.0 1.0 1.0 1.0</diffuse>
-                </material>
-            </visual>
-            <turnGravityOff>false</turnGravityOff>
-        </gazebo>
-        <!-- Transmission is important to link the joints and the controller -->
-        <!-- <transmission name="rear_${lr}_steer_joint_trans">
-            <type>transmission_interface/SimpleTransmission</type>
-            <joint name="rear_${lr}_steer_joint"/>
-            <actuator name="rear_${lr}_steer_joint_motor">
+            <joint name="${fr}_${lr}_steer_joint"/>
+            <actuator name="${fr}_${lr}_steer_joint_motor">
                 <hardwareInterface>EffortJointInterface</hardwareInterface>
                 <mechanicalReduction>1</mechanicalReduction>

Commit message: Offseted steer based on the location.

File: rover_desc_pkg/urdf/steer.xacro (robot description, xacro)
@@ -7,24 +7,24 @@
     <xacro:macro name="steer" params="fr lr parent translateX translateY"> <!-- fr: front, rear; lr: left, right -->
         <!-- Compute steer position based on its location -->
-        <xacro:if value="${fr == 'front'}">
-            <xacro:property name="origin_steer"
-                            value="${translateX * chassis_x_origin_to_steer_x_origin}
-                                   ${translateY * chassis_y_origin_to_steer_y_origin}
-                                   ${(chassis_height/2) + chassis_z_origin_to_steer_z_origin}"/>
-        </xacro:if>
+        <xacro:property name="steer_x" value="${translateX * world_x_origin_to_steer_x_origin}" scope="local"/>
+        <xacro:property name="steer_y" value="${translateY * world_y_origin_to_steer_y_origin}" scope="local"/>
+        <xacro:property name="steer_z" value="${wheel_radius + steer_z_origin_to_wheel_z_origin}" scope="local"/>
         <xacro:if value="${fr == 'rear'}">
-            <xacro:property name="origin_steer"
-                            value="${translateX * (chassis_x_origin_to_steer_x_origin + 0.063)}
-                                   ${translateY * chassis_y_origin_to_steer_y_origin}
-                                   ${(chassis_height/2) + chassis_z_origin_to_steer_z_origin}"/>
+            <xacro:property name="steer_x"
+                            value="${translateX * (world_x_origin_to_steer_x_origin + 0.063)}"
+                            scope="local"/>
         </xacro:if>
         <!-- Decide steer mesh file based on its location -->
         <xacro:if value="${lr == 'right'}">
-            <xacro:property name="mesh_file"
-                            value="package://rover_desc_pkg/meshes/rover_steer_r.dae"/>
+            <xacro:property name="mesh_file" value="package://rover_desc_pkg/meshes/rover_steer_r.dae"/>
+            <xacro:property name="steer_z"
+                            value="${wheel_radius + steer_z_origin_to_wheel_z_origin + 0.0032}"
+                            scope="local"/>
         </xacro:if>
         <xacro:if value="${lr == 'left'}">
-            <xacro:property name="mesh_file"
-                            value="package://rover_desc_pkg/meshes/rover_steer_l.dae"/>
+            <xacro:property name="mesh_file" value="package://rover_desc_pkg/meshes/rover_steer_l.dae"/>
+            <!-- <xacro:property name="steer_z"
+                                 value="${wheel_radius + steer_z_origin_to_wheel_z_origin}"
+                                 scope="local"/> -->
         </xacro:if>
         <!-- Joint description -->
@@ -38,5 +38,5 @@
                      color="White"
                      origin_rpy="0 0 0"
-                     origin_xyz="${origin_steer}"
+                     origin_xyz="${steer_x} ${steer_y} ${steer_z}"
                      mass="1.0"
                      ixx="0.0001" ixy="0.0" ixz="0.0"

Commit message: Fixed links origin and made it relative to parent. Separated joint types.

File: rover_desc_pkg/urdf/steer.xacro (robot description, xacro)
@@ -5,5 +5,5 @@
   <xacro:include filename="$(find rover_desc_pkg)/urdf/links_joints.xacro"/>
   <!-- End - Include -->
-  <xacro:macro name="steer" params="fr lr parent translateX translateY"> <!-- fr: front, rear; lr: left, right -->
+  <xacro:macro name="steer" params="fr lr parent type translateX translateY"> <!-- fr: front, rear; lr: left, right -->
     <!-- Compute steer position based on its location -->
     <xacro:property name="steer_x" value="${translateX * world_x_origin_to_steer_x_origin}" scope="local"/>
@@ -28,15 +28,9 @@
                            scope="local"/> -->
     </xacro:if>
-    <!-- Joint description -->
-    <m_joint name="${parent}__${fr}_${lr}_steer" type="fixed"
-             axis_xyz="0 0 0"
-             origin_rpy="0 0 0" origin_xyz="0 0 0"
-             parent="${parent}" child="${fr}_${lr}_steer"
-             limit_e="0" limit_l="0" limit_u="0" limit_v="0"/>
     <!-- Link description -->
     <m_link_mesh name="${fr}_${lr}_steer"
                  color="${Red_Value}"
                  origin_rpy="0 0 0"
-                 origin_xyz="${steer_x} ${steer_y} ${steer_z}"
+                 origin_xyz="0 0 0"
                  mass="1.0"
                  ixx="0.0001" ixy="0.0" ixz="0.0"
@@ -47,12 +41,25 @@
     <gazebo reference="${fr}_${lr}_steer">
       <visual name="${fr}_${lr}_steer_visual">
-          <material>
-              <ambient>0.5 0.5 0.5 1.0</ambient>
-              <specular>0.8 0.8 0.8 0.1</specular>
-              <diffuse>1.0 1.0 1.0 1.0</diffuse>
-          </material>
+        <material>
+          <ambient>0.5 0.5 0.5 1.0</ambient>
+          <specular>0.8 0.8 0.8 0.1</specular>
+          <diffuse>1.0 1.0 1.0 1.0</diffuse>
+        </material>
       </visual>
       <turnGravityOff>false</turnGravityOff>
     </gazebo>
+    <!-- Joint description -->
+    <xacro:if value="${type == 'fixed'}">
+      <m_joint_fixed name="${parent}__${fr}_${lr}_steer"
+                     origin_rpy="0 0 0" origin_xyz="${steer_x} ${steer_y} ${steer_z}"
+                     parent="${parent}" child="${fr}_${lr}_steer"/>
+    </xacro:if>
+    <xacro:if value="${type == 'revolute'}">
+      <m_joint_rev name="${parent}__${fr}_${lr}_steer"
+                   axis_xyz="0 0 1"
+                   origin_rpy="0 0 0" origin_xyz="${steer_x} ${steer_y} ${steer_z}"
+                   parent="${parent}" child="${fr}_${lr}_steer"
+                   limit_e="100" limit_l="-${M_PI/2}" limit_u="${M_PI/2}" limit_v="100"/>
+    </xacro:if>
     <!-- Transmission is important to link the joints and the controller -->
     <!-- <transmission name="${fr}_${lr}_steer_joint_trans">
