Commit message: Suppressed xml warning by adding xacro to links and joints. Fixed color in gazebo reference. Fixed color for the links.

File: rover_desc_pkg/urdf/steer.xacro (robot description, xacro)
@@ -29,30 +29,29 @@
     </xacro:if>
     <!-- Link description -->
-    <m_link_mesh name="${fr}_${lr}_steer"
-                 color="${Red_Value}"
-                 origin_rpy="0 0 0"
-                 origin_xyz="0 0 0"
-                 mass="1.0"
-                 ixx="0.0001" ixy="0.0" ixz="0.0"
-                 iyy="0.0001" iyz="0.0"
-                 izz="0.0001"
-                 meshfile="${mesh_file}"
-                 meshscale="1 1 1"/>
+    <xacro:m_link_mesh name="${fr}_${lr}_steer"
+                       color="darkgray"
+                       origin_rpy="0 0 0"
+                       origin_xyz="0 0 0"
+                       mass="1.0"
+                       ixx="0.0001" ixy="0.0" ixz="0.0"
+                       iyy="0.0001" iyz="0.0"
+                       izz="0.0001"
+                       meshfile="${mesh_file}"
+                       meshscale="1 1 1"/>
     <gazebo reference="${fr}_${lr}_steer">
       <material>Gazebo/Grey</material>
-      <turnGravityOff>false</turnGravityOff>
     </gazebo>
     <!-- Joint description -->
     <xacro:if value="${type == 'fixed'}">
-      <m_joint_fixed name="${parent}__${fr}_${lr}_steer"
-                     origin_rpy="0 0 0" origin_xyz="${steer_x} ${steer_y} ${steer_z}"
-                     parent="${parent}" child="${fr}_${lr}_steer"/>
+      <xacro:m_joint_fixed name="${parent}__${fr}_${lr}_steer"
+                           origin_rpy="0 0 0" origin_xyz="${steer_x} ${steer_y} ${steer_z}"
+                           parent="${parent}" child="${fr}_${lr}_steer"/>
     </xacro:if>
     <xacro:if value="${type == 'revolute'}">
-      <m_joint_rev name="${parent}__${fr}_${lr}_steer"
-                   axis_xyz="0 0 1"
-                   origin_rpy="0 0 0" origin_xyz="${steer_x} ${steer_y} ${steer_z}"
-                   parent="${parent}" child="${fr}_${lr}_steer"
-                   limit_e="100" limit_l="-${M_PI/2}" limit_u="${M_PI/2}" limit_v="100"/>
+      <xacro:m_joint_rev name="${parent}__${fr}_${lr}_steer"
+                         axis_xyz="0 0 1"
+                         origin_rpy="0 0 0" origin_xyz="${steer_x} ${steer_y} ${steer_z}"
+                         parent="${parent}" child="${fr}_${lr}_steer"
+                         limit_e="100" limit_l="-${M_PI/2}" limit_u="${M_PI/2}" limit_v="100"/>
     </xacro:if>
     <!-- Transmission is important to link the joints and the controller -->

File: rover_desc_pkg/urdf/wheel.xacro (robot description, xacro)
@@ -17,14 +17,14 @@
         <xacro:property name="wheel_z" value="${wheel_radius + 0.0032}" scope="local"/>
     </xacro:if>
-    <m_link_mesh name="${fr}_${lr}_wheel"
-                 color="${Black_Value}"
-                 origin_rpy="0 0 0"
-                 origin_xyz="0 0 0"
-                 mass="${m}"
-                 ixx="${m*(3*r*r+h*h)/12}" ixy="0.0" ixz="0.0"
-                 iyy="${m*(3*r*r+h*h)/12}" iyz="0.0"
-                 izz="${m*r*r/2}"
-                 meshfile="package://rover_desc_pkg/meshes/rover_wheel.dae"
-                 meshscale="1 1 1"/>
+    <xacro:m_link_mesh name="${fr}_${lr}_wheel"
+                       color="black"
+                       origin_rpy="0 0 0"
+                       origin_xyz="0 0 0"
+                       mass="${m}"
+                       ixx="${m*(3*r*r+h*h)/12}" ixy="0.0" ixz="0.0"
+                       iyy="${m*(3*r*r+h*h)/12}" iyz="0.0"
+                       izz="${m*r*r/2}"
+                       meshfile="package://rover_desc_pkg/meshes/rover_wheel.dae"
+                       meshscale="1 1 1"/>
     <gazebo reference="${fr}_${lr}_wheel">
       <mu1>1.0</mu1>
@@ -33,17 +33,14 @@
       <kd>1.0</kd>
       <fdir1>0 1 0</fdir1>
-      <visual name="${fr}_${lr}_wheel_visual">
-        <material>Gazebo/Grey</material>
-      </visual>
-      <turnGravityOff>false</turnGravityOff>
+      <material>Gazebo/Black</material>
     </gazebo>
-    <m_joint_cont name="${parent}__${fr}_${lr}_wheel"
-                  axis_xyz="0 1 0"
-                  origin_rpy="0 0 0"
-                  origin_xyz="${steer_x_origin_to_wheel_x_origin}
-                              ${steer_y_origin_to_wheel_y_origin}
-                              ${-steer_z_origin_to_wheel_z_origin}"
-                  parent="${parent}" child="${fr}_${lr}_wheel"
-                  limit_e="100" limit_v="100"/>
+    <xacro:m_joint_cont name="${parent}__${fr}_${lr}_wheel"
+                        axis_xyz="0 1 0"
+                        origin_rpy="0 0 0"
+                        origin_xyz="${steer_x_origin_to_wheel_x_origin}
+                                    ${steer_y_origin_to_wheel_y_origin}
+                                    ${-steer_z_origin_to_wheel_z_origin}"
+                        parent="${parent}" child="${fr}_${lr}_wheel"
+                        limit_e="100" limit_v="100"/>
     <!-- Transmission is important to link the joints and the controller -->
     <!-- <transmission name="${fr}_${lr}_wheel_joint_trans">

Commit message: Steering limits=+-75 deg.

File: rover_desc_pkg/urdf/steer.xacro (robot description, xacro)
@@ -53,15 +53,6 @@
                          origin_rpy="0 0 0" origin_xyz="${steer_x} ${steer_y} ${steer_z}"
                          parent="${parent}" child="${fr}_${lr}_steer"
-                         limit_e="100" limit_l="-${M_PI/2}" limit_u="${M_PI/2}" limit_v="100"/>
+                         limit_e="100" limit_l="-${5*M_PI/12}" limit_u="${5*M_PI/12}" limit_v="100"/>
     </xacro:if>
-    <!-- Transmission is important to link the joints and the controller -->
-    <!-- <transmission name="${fr}_${lr}_steer_joint_trans">
-      <type>transmission_interface/SimpleTransmission</type>
-      <joint name="${fr}_${lr}_steer_joint"/>
-      <actuator name="${fr}_${lr}_steer_joint_motor">
-          <hardwareInterface>EffortJointInterface</hardwareInterface>
-          <mechanicalReduction>1</mechanicalReduction>
-      </actuator>
-    </transmission> -->
   </xacro:macro>
 </robot>
