Commit message: Offseted right side wheels Z position.

File: rover_desc_pkg/urdf/wheel.xacro (robot description, xacro)
@@ -6,4 +6,11 @@
     <!-- End - Include -->
     <xacro:macro name="wheel" params="fr lr parent translateX translateY"> <!-- fr: front, rear; lr: left, right -->
+        <!-- Compute wheel position based on its location -->
+        <xacro:property name="wheel_x" value="${translateX * world_x_origin_to_wheel_x_origin}" scope="local"/>
+        <xacro:property name="wheel_y" value="${translateY * world_y_origin_to_wheel_y_origin}" scope="local"/>
+        <xacro:property name="wheel_z" value="${wheel_radius}" scope="local"/>
+        <xacro:if value="${lr == 'right'}">
+            <xacro:property name="wheel_z" value="${wheel_radius + 0.0032}" scope="local"/>
+        </xacro:if>
         <m_joint name="${r_link_01_name}__${fr}_${lr}_wheel" type="fixed"
                  axis_xyz="0 0 0"
@@ -14,7 +21,5 @@
                      color="Black"
                      origin_rpy="0 0 0"
-                     origin_xyz="${translateX * chassis_x_origin_to_wheel_x_origin}
-                                 ${translateY * chassis_y_origin_to_wheel_y_origin}
-                                 ${wheel_radius}"
+                     origin_xyz="${wheel_x} ${wheel_y} ${wheel_z}"
                      mass="1.0"
                      ixx="0.0001" ixy="0.0" ixz="0.0"

Commit message: Fixed wheel joint types and corrected inertia. Made wheels position relative to steer links.

File: rover_desc_pkg/urdf/wheel.xacro (robot description, xacro)
@@ -6,4 +6,8 @@
   <!-- End - Include -->
   <xacro:macro name="wheel" params="fr lr parent translateX translateY"> <!-- fr: front, rear; lr: left, right -->
+    <!-- Parameters to compute inertia -->
+    <xacro:property name="m" value="${wheel_mass}" scope="local"/>
+    <xacro:property name="r" value="${wheel_radius}" scope="local"/>
+    <xacro:property name="h" value="${wheel_height}" scope="local"/>
     <!-- Compute wheel position based on its location -->
     <xacro:property name="wheel_x" value="${translateX * world_x_origin_to_wheel_x_origin}" scope="local"/>
@@ -13,17 +17,12 @@
         <xacro:property name="wheel_z" value="${wheel_radius + 0.0032}" scope="local"/>
     </xacro:if>
-    <m_joint name="${r_link_01_name}__${fr}_${lr}_wheel" type="fixed"
-             axis_xyz="0 0 0"
-             origin_rpy="0 0 0" origin_xyz="0 0 0"
-             parent="${parent}" child="${fr}_${lr}_wheel"
-             limit_e="0" limit_l="0" limit_u="0" limit_v="0"/>
     <m_link_mesh name="${fr}_${lr}_wheel"
                  color="${Black_Value}"
                  origin_rpy="0 0 0"
-                 origin_xyz="${wheel_x} ${wheel_y} ${wheel_z}"
-                 mass="1.0"
-                 ixx="0.0001" ixy="0.0" ixz="0.0"
-                 iyy="0.0001" iyz="0.0"
-                 izz="0.0001"
+                 origin_xyz="0 0 0"
+                 mass="${m}"
+                 ixx="${m*(3*r*r+h*h)/12}" ixy="0.0" ixz="0.0"
+                 iyy="${m*(3*r*r+h*h)/12}" iyz="0.0"
+                 izz="${m*r*r/2}"
                  meshfile="package://rover_desc_pkg/meshes/rover_wheel.dae"
                  meshscale="1 1 1"/>
@@ -38,4 +37,12 @@
       <turnGravityOff>false</turnGravityOff>
     </gazebo>
+    <m_joint_cont name="${parent}__${fr}_${lr}_wheel"
+                  axis_xyz="0 1 0"
+                  origin_rpy="0 0 0"
+                  origin_xyz="${steer_x_origin_to_wheel_x_origin}
+                              ${steer_y_origin_to_wheel_y_origin}
+                              ${-steer_z_origin_to_wheel_z_origin}"
+                  parent="${parent}" child="${fr}_${lr}_wheel"
+                  limit_e="100" limit_v="100"/>
     <!-- Transmission is important to link the joints and the controller -->
     <!-- <transmission name="${fr}_${lr}_wheel_joint_trans">

Commit message: Changed velocity limit. Removed friction parameters.

File: rover_desc_pkg/urdf/wheel.xacro (robot description, xacro)
@@ -28,9 +28,4 @@
                        meshscale="1 1 1"/>
     <gazebo reference="${fr}_${lr}_wheel">
-      <mu1>1.0</mu1>
-      <mu2>1.0</mu2>
-      <kp>10000000.0</kp>
-      <kd>1.0</kd>
-      <fdir1>0 1 0</fdir1>
       <material>Gazebo/Black</material>
     </gazebo>
@@ -42,14 +37,5 @@
                                     ${-steer_z_origin_to_wheel_z_origin}"
                         parent="${parent}" child="${fr}_${lr}_wheel"
-                        limit_e="100" limit_v="100"/>
-    <!-- Transmission is important to link the joints and the controller -->
-    <!-- <transmission name="${fr}_${lr}_wheel_joint_trans">
-      <type>transmission_interface/SimpleTransmission</type>
-      <joint name="${fr}_${lr}_wheel_joint"/>
-      <actuator name="${fr}_${lr}_wheel_joint_motor">
-        <hardwareInterface>EffortJointInterface</hardwareInterface>
-        <mechanicalReduction>1</mechanicalReduction>
-      </actuator>
-    </transmission> -->
+                        limit_e="100" limit_v="25"/>
   </xacro:macro>
 </robot>
