Commit message: Changed tab size.

File: rover_desc_pkg/urdf/links_joints.xacro (robot description, xacro)
@@ -1,92 +1,98 @@
 <?xml version="1.0"?>
 <robot xmlns:xacro="http://www.ros.org/wiki/xacro">
-    <!-- Joint Macro -->
-    <xacro:macro name="m_joint" params="name type axis_xyz origin_xyz origin_rpy parent child limit_e limit_l limit_u limit_v">
-        <joint name="${name}" type="${type}">
-            <axis xyz="${axis_xyz}"/>
-            <limit effort="${limit_e}" lower="${limit_l}" upper="${limit_u}" velocity="${limit_v}"/>
-            <origin rpy="${origin_rpy}" xyz="${origin_xyz}"/>
-            <parent link="${parent}"/>
-            <child link="${child}"/>
-        </joint>
-        <transmission name="trans_${name}">
-            <type>transmission_interface/SimpleTransmission</type>
-            <joint name="${name}">
-                <hardwareInterface>hardware_interface/EffortJointInterface</hardwareInterface>
-            </joint>
-            <actuator name="motor_${name}">
-                <hardwareInterface>hardware_interface/EffortJointInterface</hardwareInterface>
-                <mechanicalReduction>1</mechanicalReduction>
-            </actuator>
-        </transmission>
-    </xacro:macro>
-    <!-- Cylinder link Macro -->
-    <xacro:macro name="m_link_cylinder" params="name color origin_xyz origin_rpy radius length mass ixx ixy ixz iyy iyz izz">
-        <link name="${name}">
-            <inertial>
-                <mass value="${mass}"/>
-                <origin rpy="${origin_rpy}" xyz="${origin_xyz}"/>
-                <inertia ixx="${ixx}" ixy="${ixy}" ixz="${ixz}" iyy="${iyy}" iyz="${iyz}" izz="${izz}"/>
-            </inertial>
-            <collision>
-                <origin rpy="${origin_rpy}" xyz="${origin_xyz}"/>
-                <geometry>
-                    <cylinder radius="${radius}" length="${length}"/>
-                </geometry>
-            </collision>
-            <visual>
-                <origin rpy="${origin_rpy}" xyz="${origin_xyz}"/>
-                <geometry>
-                    <cylinder radius="${radius}" length="${length}"/>
-                </geometry>
-                <material name="${color}"/>
-            </visual>
-        </link>
-    </xacro:macro>
-    <!-- Box link Macro -->
-    <xacro:macro name="m_link_box" params="name color origin_xyz origin_rpy size mass ixx ixy ixz iyy iyz izz">
-        <link name="${name}">
-            <inertial>
-                <mass value="${mass}"/>
-                <origin rpy="${origin_rpy}" xyz="${origin_xyz}"/>
-                <inertia ixx="${ixx}" ixy="${ixy}" ixz="${ixz}" iyy="${iyy}" iyz="${iyz}" izz="${izz}"/>
-            </inertial>
-            <collision>
-                <origin rpy="${origin_rpy}" xyz="${origin_xyz}"/>
-                <geometry>
-                    <box size="${size}"/>
-                </geometry>
-            </collision>
-            <visual>
-                <origin rpy="${origin_rpy}" xyz="${origin_xyz}"/>
-                <geometry>
-                    <box size="${size}"/>
-                </geometry>
-                <material name="${color}"/>
-            </visual>
-        </link>
-    </xacro:macro>
-    <!-- Mesh link Macro -->
-    <xacro:macro name="m_link_mesh" params="name color origin_xyz origin_rpy meshfile meshscale mass ixx ixy ixz iyy iyz izz">
-        <link name="${name}">
-            <inertial>
-                <mass value="${mass}"/>
-                <origin rpy="${origin_rpy}" xyz="${origin_xyz}"/>
-                <inertia ixx="${ixx}" ixy="${ixy}" ixz="${ixz}" iyy="${iyy}" iyz="${iyz}" izz="${izz}"/>
-            </inertial>
-            <collision>
-                <origin rpy="${origin_rpy}" xyz="${origin_xyz}"/>
-                <geometry>
-                    <mesh filename="${meshfile}" scale="${meshscale}"/>
-                </geometry>
-            </collision>
-            <visual>
-                <origin rpy="${origin_rpy}" xyz="${origin_xyz}"/>
-                <geometry>
-                    <mesh filename="${meshfile}" scale="${meshscale}"/>
-                </geometry>
-                <material name="${color}"/>
-            </visual>
-        </link>
-    </xacro:macro>
+  <!-- Joint Macro -->
+  <xacro:macro name="m_joint" params="name type axis_xyz origin_xyz origin_rpy parent child limit_e limit_l limit_u limit_v">
+    <joint name="${name}" type="${type}">
+      <axis xyz="${axis_xyz}"/>
+      <limit effort="${limit_e}" lower="${limit_l}" upper="${limit_u}" velocity="${limit_v}"/>
+      <origin rpy="${origin_rpy}" xyz="${origin_xyz}"/>
+      <parent link="${parent}"/>
+      <child link="${child}"/>
+    </joint>
+    <transmission name="trans_${name}">
+      <type>transmission_interface/SimpleTransmission</type>
+      <joint name="${name}">
+        <hardwareInterface>hardware_interface/EffortJointInterface</hardwareInterface>
+      </joint>
+      <actuator name="motor_${name}">
+        <hardwareInterface>hardware_interface/EffortJointInterface</hardwareInterface>
+        <mechanicalReduction>1</mechanicalReduction>
+      </actuator>
+    </transmission>
+  </xacro:macro>
+  <!-- Cylinder link Macro -->
+  <xacro:macro name="m_link_cylinder" params="name color origin_xyz origin_rpy radius length mass ixx ixy ixz iyy iyz izz">
+    <link name="${name}">
+      <inertial>
+        <mass value="${mass}"/>
+        <origin rpy="${origin_rpy}" xyz="${origin_xyz}"/>
+        <inertia ixx="${ixx}" ixy="${ixy}" ixz="${ixz}" iyy="${iyy}" iyz="${iyz}" izz="${izz}"/>
+      </inertial>
+      <collision>
+        <origin rpy="${origin_rpy}" xyz="${origin_xyz}"/>
+        <geometry>
+          <cylinder radius="${radius}" length="${length}"/>
+        </geometry>
+      </collision>
+      <visual>
+        <origin rpy="${origin_rpy}" xyz="${origin_xyz}"/>
+        <geometry>
+          <cylinder radius="${radius}" length="${length}"/>
+        </geometry>
+        <material name="">
+          <color rgba="${color}"/>
+        </material>
+      </visual>
+    </link>
+  </xacro:macro>
+  <!-- Box link Macro -->
+  <xacro:macro name="m_link_box" params="name color origin_xyz origin_rpy size mass ixx ixy ixz iyy iyz izz">
+    <link name="${name}">
+      <inertial>
+        <mass value="${mass}"/>
+        <origin rpy="${origin_rpy}" xyz="${origin_xyz}"/>
+        <inertia ixx="${ixx}" ixy="${ixy}" ixz="${ixz}" iyy="${iyy}" iyz="${iyz}" izz="${izz}"/>
+      </inertial>
+      <collision>
+        <origin rpy="${origin_rpy}" xyz="${origin_xyz}"/>
+        <geometry>
+          <box size="${size}"/>
+        </geometry>
+      </collision>
+      <visual>
+        <origin rpy="${origin_rpy}" xyz="${origin_xyz}"/>
+        <geometry>
+          <box size="${size}"/>
+        </geometry>
+        <material name="">
+          <color rgba="${color}"/>
+        </material>
+      </visual>
+    </link>
+  </xacro:macro>
+  <!-- Mesh link Macro -->
+  <xacro:macro name="m_link_mesh" params="name color origin_xyz origin_rpy meshfile meshscale mass ixx ixy ixz iyy iyz izz">
+    <link name="${name}">
+      <inertial>
+        <mass value="${mass}"/>
+        <origin rpy="${origin_rpy}" xyz="${origin_xyz}"/>
+        <inertia ixx="${ixx}" ixy="${ixy}" ixz="${ixz}" iyy="${iyy}" iyz="${iyz}" izz="${izz}"/>
+      </inertial>
+      <collision>
+        <origin rpy="${origin_rpy}" xyz="${origin_xyz}"/>
+        <geometry>
+            <mesh filename="${meshfile}" scale="${meshscale}"/>
+        </geometry>
+      </collision>
+      <visual>
+        <origin rpy="${origin_rpy}" xyz="${origin_xyz}"/>
+        <geometry>
+            <mesh filename="${meshfile}" scale="${meshscale}"/>
+        </geometry>
+        <material name="">
+            <color rgba="${color}"/>
+        </material>
+      </visual>
+    </link>
+  </xacro:macro>
 </robot>

File: rover_desc_pkg/urdf/robot_parameters.xacro (robot description, xacro)
@@ -1,75 +1,75 @@
 <?xml version="1.0"?>
 <robot xmlns:xacro="http://www.ros.org/wiki/xacro">
-    <xacro:property name="r_link_00_name" value="chassis_footprint"/>
-    <xacro:property name="r_link_01_name" value="chassis_link"/>
-    <xacro:property name="r_link_02_name" value="steer_link"/>
-    <!-- Color parameters -->
-    <xacro:property name="Red_Value" value="{204/255} ${0.0/255} ${0.0/255} ${255/255}"/>
-    <xacro:property name="Green_Value" value="${0.0/255} ${204/255} ${0.0/255} ${255/255}"/>
-    <xacro:property name="Blue_Value" value="${0.0/255} ${0.0/255} ${204/255} ${255/255}"/>
-    <xacro:property name="Black_Value" value="${0.0/255} ${0.0/255} ${0.0/255} ${255/255}"/>
-    <xacro:property name="White_Value" value="${255/255} ${255/255} ${255/255} ${255/255}"/>
-    <xacro:macro name="Red">
-        <material name="">
-            <color rgba="${Red_Value}"/>
-        </material>
-    </xacro:macro>
-    <xacro:macro name="Green">
-        <material name="">
-            <color rgba="${Green_Value}"/>
-        </material>
-    </xacro:macro>
-    <xacro:macro name="Blue">
-        <material name="">
-            <color rgba="${Blue_Value}"/>
-        </material>
-    </xacro:macro>
-    <xacro:macro name="Black">
-        <material name="">
-            <color rgba="${Black_Value}"/>
-        </material>
-    </xacro:macro>
-    <xacro:macro name="White">
-        <material name="">
-            <color rgba="${White_Value}"/>
-        </material>
-    </xacro:macro>
-    <!-- All the units are in m-kg-s-radians unit system -->
-    <xacro:property name="M_PI" value="3.141592653"/>
-    <xacro:property name="DEG_TO_RAD" value="0.017453293"/>
-    <!-- Chassis dimensions -->
-    <xacro:property name="chassis_length" value="1.016"/>
-    <xacro:property name="chassis_width" value="0.6096"/>
-    <xacro:property name="chassis_height" value="0.4445"/>
-    <xacro:property name="chassis_mass" value="5"/> <!-- in Kg -->
-    <xacro:property name="world_x_origin_to_chassis_x_origin" value="0.0"/>
-    <xacro:property name="world_y_origin_to_chassis_y_origin" value="0.0"/>
-    <xacro:property name="world_z_origin_to_chassis_z_origin" value="0.0"/>
-    <!-- Inverter dimensions -->
-    <xacro:property name="inverter_length" value="0.400"/>
-    <xacro:property name="inverter_width" value="0.2353"/>
-    <xacro:property name="inverter_height" value="0.400"/>
-    <xacro:property name="inverter_mass" value="5"/> <!-- in Kg -->
-    <!-- Steer dimensions -->
-    <xacro:property name="steer_length" value="0.217"/>
-    <xacro:property name="steer_width" value="0.234"/>
-    <xacro:property name="steer_height" value="0.618"/>
-    <xacro:property name="steer_mass" value="5"/> <!-- in Kg -->
-    <xacro:property name="world_x_origin_to_steer_x_origin" value="0.3715"/> <!-- Distance from world origin to mount point in X direction -->
-    <xacro:property name="world_y_origin_to_steer_y_origin" value="0.3148"/> <!-- Distance from world origin to mount point in Y direction -->
-    <xacro:property name="world_z_origin_to_steer_z_origin" value="0.0"/> <!-- Distance from world origin to mount point in Z direction -->
-    <xacro:property name="chassis_z_origin_to_steer_z_origin" value="0.1305"/>
-    <!-- Wheels -->
-    <xacro:property name="wheel_radius" value="0.178"/>
-    <xacro:property name="wheel_height" value="0.114"/>
-    <xacro:property name="wheel_mass" value="1.0"/> <!-- in Kg -->
-    <xacro:property name="world_x_origin_to_wheel_x_origin" value="0.4025"/>
-    <xacro:property name="world_y_origin_to_wheel_y_origin" value="0.3153"/>
-    <xacro:property name="world_z_origin_to_wheel_z_origin" value="0.0"/>
-    <xacro:property name="steer_z_origin_to_wheel_z_origin" value="0.4625"/>
-    <xacro:macro name="cylinder_inertia" params="m r h">
-        <intertia ixx="${m*(3*r*r+h*h)/12}" ixy="0.0" ixz="0.0"
-                  iyy="${m*(3*r*r+h*h)/12}" iyz="0.0"
-                  izz="${m*r*r/2}"/>
-    </xacro:macro>
+  <xacro:property name="r_link_00_name" value="chassis_footprint"/>
+  <xacro:property name="r_link_01_name" value="chassis_link"/>
+  <xacro:property name="r_link_02_name" value="steer_link"/>
+  <!-- Color parameters -->
+  <xacro:property name="Red_Value" value="${204/255} ${0.0/255} ${0.0/255} ${255/255}"/>
+  <xacro:property name="Green_Value" value="${0.0/255} ${204/255} ${0.0/255} ${255/255}"/>
+  <xacro:property name="Blue_Value" value="${0.0/255} ${0.0/255} ${204/255} ${255/255}"/>
+  <xacro:property name="Black_Value" value="${0.0/255} ${0.0/255} ${0.0/255} ${255/255}"/>
+  <xacro:property name="White_Value" value="${255/255} ${255/255} ${255/255} ${255/255}"/>
+  <xacro:macro name="Red">
+    <material name="">
+      <color rgba="${Red_Value}"/>
+    </material>
+  </xacro:macro>
+  <xacro:macro name="Green">
+    <material name="">
+      <color rgba="${Green_Value}"/>
+    </material>
+  </xacro:macro>
+  <xacro:macro name="Blue">
+    <material name="">
+      <color rgba="${Blue_Value}"/>
+    </material>
+  </xacro:macro>
+  <xacro:macro name="Black">
+    <material name="">
+      <color rgba="${Black_Value}"/>
+    </material>
+  </xacro:macro>
+  <xacro:macro name="White">
+    <material name="">
+      <color rgba="${White_Value}"/>
+    </material>
+  </xacro:macro>
+  <!-- All the units are in m-kg-s-radians unit system -->
+  <xacro:property name="M_PI" value="3.141592653"/>
+  <xacro:property name="DEG_TO_RAD" value="0.017453293"/>
+  <!-- Chassis dimensions -->
+  <xacro:property name="chassis_length" value="1.016"/>
+  <xacro:property name="chassis_width" value="0.6096"/>
+  <xacro:property name="chassis_height" value="0.4445"/>
+  <xacro:property name="chassis_mass" value="5"/> <!-- in Kg -->
+  <xacro:property name="world_x_origin_to_chassis_x_origin" value="0.0"/>
+  <xacro:property name="world_y_origin_to_chassis_y_origin" value="0.0"/>
+  <xacro:property name="world_z_origin_to_chassis_z_origin" value="0.0"/>
+  <!-- Inverter dimensions -->
+  <xacro:property name="inverter_length" value="0.400"/>
+  <xacro:property name="inverter_width" value="0.2353"/>
+  <xacro:property name="inverter_height" value="0.400"/>
+  <xacro:property name="inverter_mass" value="5"/> <!-- in Kg -->
+  <!-- Steer dimensions -->
+  <xacro:property name="steer_length" value="0.217"/>
+  <xacro:property name="steer_width" value="0.234"/>
+  <xacro:property name="steer_height" value="0.618"/>
+  <xacro:property name="steer_mass" value="5"/> <!-- in Kg -->
+  <xacro:property name="world_x_origin_to_steer_x_origin" value="0.3715"/> <!-- Distance from world origin to mount point in X direction -->
+  <xacro:property name="world_y_origin_to_steer_y_origin" value="0.3148"/> <!-- Distance from world origin to mount point in Y direction -->
+  <xacro:property name="world_z_origin_to_steer_z_origin" value="0.0"/> <!-- Distance from world origin to mount point in Z direction -->
+  <xacro:property name="chassis_z_origin_to_steer_z_origin" value="0.1305"/>
+  <!-- Wheels -->
+  <xacro:property name="wheel_radius" value="0.178"/>
+  <xacro:property name="wheel_height" value="0.114"/>
+  <xacro:property name="wheel_mass" value="1.0"/> <!-- in Kg -->
+  <xacro:property name="world_x_origin_to_wheel_x_origin" value="0.4025"/>
+  <xacro:property name="world_y_origin_to_wheel_y_origin" value="0.3153"/>
+  <xacro:property name="world_z_origin_to_wheel_z_origin" value="0.0"/>
+  <xacro:property name="steer_z_origin_to_wheel_z_origin" value="0.4625"/>
+  <xacro:macro name="cylinder_inertia" params="m r h">
+    <intertia ixx="${m*(3*r*r+h*h)/12}" ixy="0.0" ixz="0.0"
+              iyy="${m*(3*r*r+h*h)/12}" iyz="0.0"
+              izz="${m*r*r/2}"/>
+  </xacro:macro>
 </robot>

File: rover_desc_pkg/urdf/rover_robot.xacro (robot description, xacro)
@@ -1,63 +1,63 @@
 <?xml version="1.0"?>
 <robot name="rover_robot" xmlns:xacro="http://www.ros.org/wiki/xacro">
-    <!-- Begin - Include -->
-    <xacro:include filename="$(find rover_desc_pkg)/urdf/robot_parameters.xacro"/>
-    <xacro:include filename="$(find rover_desc_pkg)/urdf/links_joints.xacro"/>
-    <xacro:include filename="$(find rover_desc_pkg)/urdf/steer.xacro"/>
-    <xacro:include filename="$(find rover_desc_pkg)/urdf/wheel.xacro"/>
-    <!-- End - Include -->
-    <!-- Begin - Robot Description -->
-    <!-- Chassis footprint -->
-    <m_link_box name="${r_link_00_name}"
-                color="White"
-                origin_rpy="0 0 0" origin_xyz="0 0 0"
-                mass="0.0001"
-                ixx="0.0001" ixy="0.0" ixz="0.0"
-                iyy="0.0001" iyz="0.0"
-                izz="0.0001"
-                size="0.0001 0.0001 0.0001"/>
-    <gazebo reference="${r_link_00_name}">
-        <turnGravityOff>false</turnGravityOff>
-    </gazebo>
-    <m_joint name="${r_link_00_name}__${r_link_01_name}" type="fixed"
-             axis_xyz="0 0 0"
-             origin_rpy="0 0 0" origin_xyz="0 0 0"
-             parent="${r_link_00_name}" child="${r_link_01_name}"
-             limit_e="0" limit_l="0" limit_u="0" limit_v="0"/>
-    <m_link_mesh name="${r_link_01_name}"
-                 color="White"
-                 origin_rpy="0 0 0"
-                 origin_xyz="0 0 ${wheel_radius + steer_z_origin_to_wheel_z_origin - chassis_z_origin_to_steer_z_origin}"
-                 mass="1.0"
-                 ixx="0.0001" ixy="0.0" ixz="0.0"
-                 iyy="0.0001" iyz="0.0"
-                 izz="0.0001"
-                 meshfile="package://rover_desc_pkg/meshes/rover_chassis.dae"
-                 meshscale="1 1 1"/>
-    <gazebo reference="${r_link_01_name}">
-        <visual name="${r_link_01_name}_visual">
-            <material>
-                <ambient>0.5 0.5 0.5 1.0</ambient>
-                <specular>0.8 0.8 0.8 0.1</specular>
-                <diffuse>1.0 1.0 1.0 1.0</diffuse>
-            </material>
-        </visual>
-        <turnGravityOff>false</turnGravityOff>
-    </gazebo>
-    <!-- Steers & Wheels -->
-    <steer fr="front" lr="right" parent="${r_link_01_name}" translateX="1" translateY="-1"/>
-    <wheel fr="front" lr="right" parent="front_right_steer" translateX="1" translateY="-1"/>
-    <steer fr="front" lr="left" parent="${r_link_01_name}" translateX="1" translateY="1"/>
-    <wheel fr="front" lr="left" parent="front_left_steer" translateX="1" translateY="1"/>
-    <steer fr="rear" lr="right" parent="${r_link_01_name}" translateX="-1" translateY="-1"/>
-    <wheel fr="rear" lr="right" parent="rear_right_steer" translateX="-1" translateY="-1"/>
-    <steer fr="rear" lr="left" parent="${r_link_01_name}" translateX="-1" translateY="1"/>
-    <wheel fr="rear" lr="left" parent="rear_left_steer" translateX="-1" translateY="1"/>
-    <!-- End - Robot Description -->
-    <!-- Rover -->
-    <gazebo>
-        <plugin name="gazebo_ros_control" filename="libgazebo_ros_control.so">
-          <robotNamespace>/rover</robotNamespace>
-        </plugin>
-    </gazebo>
+  <!-- Begin - Include -->
+  <xacro:include filename="$(find rover_desc_pkg)/urdf/robot_parameters.xacro"/>
+  <xacro:include filename="$(find rover_desc_pkg)/urdf/links_joints.xacro"/>
+  <xacro:include filename="$(find rover_desc_pkg)/urdf/steer.xacro"/>
+  <xacro:include filename="$(find rover_desc_pkg)/urdf/wheel.xacro"/>
+  <!-- End - Include -->
+  <!-- Begin - Robot Description -->
+  <!-- Chassis footprint -->
+  <m_link_box name="${r_link_00_name}"
+              color="${White_Value}"
+              origin_rpy="0 0 0" origin_xyz="0 0 0"
+              mass="0.0001"
+              ixx="0.0001" ixy="0.0" ixz="0.0"
+              iyy="0.0001" iyz="0.0"
+              izz="0.0001"
+              size="0.0001 0.0001 0.0001"/>
+  <gazebo reference="${r_link_00_name}">
+    <turnGravityOff>false</turnGravityOff>
+  </gazebo>
+  <m_joint name="${r_link_00_name}__${r_link_01_name}" type="fixed"
+           axis_xyz="0 0 0"
+           origin_rpy="0 0 0" origin_xyz="0 0 0"
+           parent="${r_link_00_name}" child="${r_link_01_name}"
+           limit_e="0" limit_l="0" limit_u="0" limit_v="0"/>
+  <m_link_mesh name="${r_link_01_name}"
+               color="${White_Value}"
+               origin_rpy="0 0 0"
+               origin_xyz="0 0 ${wheel_radius + steer_z_origin_to_wheel_z_origin - chassis_z_origin_to_steer_z_origin}"
+               mass="1.0"
+               ixx="0.0001" ixy="0.0" ixz="0.0"
+               iyy="0.0001" iyz="0.0"
+               izz="0.0001"
+               meshfile="package://rover_desc_pkg/meshes/rover_chassis.dae"
+               meshscale="1 1 1"/>
+  <gazebo reference="${r_link_01_name}">
+    <visual name="${r_link_01_name}_visual">
+      <material>
+        <ambient>0.5 0.5 0.5 1.0</ambient>
+        <specular>0.8 0.8 0.8 0.1</specular>
+        <diffuse>1.0 1.0 1.0 1.0</diffuse>
+      </material>
+    </visual>
+    <turnGravityOff>false</turnGravityOff>
+  </gazebo>
+  <!-- Steers & Wheels -->
+  <steer fr="front" lr="right" parent="${r_link_01_name}" translateX="1" translateY="-1"/>
+  <wheel fr="front" lr="right" parent="front_right_steer" translateX="1" translateY="-1"/>
+  <steer fr="front" lr="left" parent="${r_link_01_name}" translateX="1" translateY="1"/>
+  <wheel fr="front" lr="left" parent="front_left_steer" translateX="1" translateY="1"/>
+  <steer fr="rear" lr="right" parent="${r_link_01_name}" translateX="-1" translateY="-1"/>
+  <wheel fr="rear" lr="right" parent="rear_right_steer" translateX="-1" translateY="-1"/>
+  <steer fr="rear" lr="left" parent="${r_link_01_name}" translateX="-1" translateY="1"/>
+  <wheel fr="rear" lr="left" parent="rear_left_steer" translateX="-1" translateY="1"/>
+  <!-- End - Robot Description -->
+  <!-- Rover -->
+  <gazebo>
+    <plugin name="gazebo_ros_control" filename="libgazebo_ros_control.so">
+      <robotNamespace>/rover</robotNamespace>
+    </plugin>
+  </gazebo>
 </robot>
