Commit message: Changed tab size.

File: rover_desc_pkg/urdf/steer.xacro (robot description, xacro)
@@ -1,67 +1,67 @@
 <?xml version="1.0"?>
 <robot name="steer" xmlns:xacro="http://www.ros.org/wiki/xacro">
-    <!-- Begin - Include -->
-    <xacro:include filename="$(find rover_desc_pkg)/urdf/robot_parameters.xacro"/>
-    <xacro:include filename="$(find rover_desc_pkg)/urdf/links_joints.xacro"/>
-    <!-- End - Include -->
-    <xacro:macro name="steer" params="fr lr parent translateX translateY"> <!-- fr: front, rear; lr: left, right -->
-        <!-- Compute steer position based on its location -->
-        <xacro:property name="steer_x" value="${translateX * world_x_origin_to_steer_x_origin}" scope="local"/>
-        <xacro:property name="steer_y" value="${translateY * world_y_origin_to_steer_y_origin}" scope="local"/>
-        <xacro:property name="steer_z" value="${wheel_radius + steer_z_origin_to_wheel_z_origin}" scope="local"/>
-        <xacro:if value="${fr == 'rear'}">
-            <xacro:property name="steer_x"
-                            value="${translateX * (world_x_origin_to_steer_x_origin + 0.063)}"
-                            scope="local"/>
-        </xacro:if>
-        <!-- Decide steer mesh file based on its location -->
-        <xacro:if value="${lr == 'right'}">
-            <xacro:property name="mesh_file" value="package://rover_desc_pkg/meshes/rover_steer_r.dae"/>
-            <xacro:property name="steer_z"
-                            value="${wheel_radius + steer_z_origin_to_wheel_z_origin + 0.0032}"
-                            scope="local"/>
-        </xacro:if>
-        <xacro:if value="${lr == 'left'}">
-            <xacro:property name="mesh_file" value="package://rover_desc_pkg/meshes/rover_steer_l.dae"/>
-            <!-- <xacro:property name="steer_z"
-                                 value="${wheel_radius + steer_z_origin_to_wheel_z_origin}"
-                                 scope="local"/> -->
-        </xacro:if>
-        <!-- Joint description -->
-        <m_joint name="${parent}__${fr}_${lr}_steer" type="fixed"
-                 axis_xyz="0 0 0"
-                 origin_rpy="0 0 0" origin_xyz="0 0 0"
-                 parent="${parent}" child="${fr}_${lr}_steer"
-                 limit_e="0" limit_l="0" limit_u="0" limit_v="0"/>
-        <!-- Link description -->
-        <m_link_mesh name="${fr}_${lr}_steer"
-                     color="White"
-                     origin_rpy="0 0 0"
-                     origin_xyz="${steer_x} ${steer_y} ${steer_z}"
-                     mass="1.0"
-                     ixx="0.0001" ixy="0.0" ixz="0.0"
-                     iyy="0.0001" iyz="0.0"
-                     izz="0.0001"
-                     meshfile="${mesh_file}"
-                     meshscale="1 1 1"/>
-        <gazebo reference="${fr}_${lr}_steer">
-            <visual name="${fr}_${lr}_steer_visual">
-                <material>
-                    <ambient>0.5 0.5 0.5 1.0</ambient>
-                    <specular>0.8 0.8 0.8 0.1</specular>
-                    <diffuse>1.0 1.0 1.0 1.0</diffuse>
-                </material>
-            </visual>
-            <turnGravityOff>false</turnGravityOff>
-        </gazebo>
-        <!-- Transmission is important to link the joints and the controller -->
-        <!-- <transmission name="${fr}_${lr}_steer_joint_trans">
-            <type>transmission_interface/SimpleTransmission</type>
-            <joint name="${fr}_${lr}_steer_joint"/>
-            <actuator name="${fr}_${lr}_steer_joint_motor">
-                <hardwareInterface>EffortJointInterface</hardwareInterface>
-                <mechanicalReduction>1</mechanicalReduction>
-            </actuator>
-        </transmission> -->
-    </xacro:macro>
+  <!-- Begin - Include -->
+  <xacro:include filename="$(find rover_desc_pkg)/urdf/robot_parameters.xacro"/>
+  <xacro:include filename="$(find rover_desc_pkg)/urdf/links_joints.xacro"/>
+  <!-- End - Include -->
+  <xacro:macro name="steer" params="fr lr parent translateX translateY"> <!-- fr: front, rear; lr: left, right -->
+    <!-- Compute steer position based on its location -->
+    <xacro:property name="steer_x" value="${translateX * world_x_origin_to_steer_x_origin}" scope="local"/>
+    <xacro:property name="steer_y" value="${translateY * world_y_origin_to_steer_y_origin}" scope="local"/>
+    <xacro:property name="steer_z" value="${wheel_radius + steer_z_origin_to_wheel_z_origin}" scope="local"/>
+    <xacro:if value="${fr == 'rear'}">
+      <xacro:property name="steer_x"
+                      value="${translateX * (world_x_origin_to_steer_x_origin + 0.063)}"
+                      scope="local"/>
+    </xacro:if>
+    <!-- Decide steer mesh file based on its location -->
+    <xacro:if value="${lr == 'right'}">
+      <xacro:property name="mesh_file" value="package://rover_desc_pkg/meshes/rover_steer_r.dae"/>
+      <xacro:property name="steer_z"
+                      value="${wheel_radius + steer_z_origin_to_wheel_z_origin + 0.0032}"
+                      scope="local"/>
+    </xacro:if>
+    <xacro:if value="${lr == 'left'}">
+      <xacro:property name="mesh_file" value="package://rover_desc_pkg/meshes/rover_steer_l.dae"/>
+      <!-- <xacro:property name="steer_z"
+                           value="${wheel_radius + steer_z_origin_to_wheel_z_origin}"
+                           scope="local"/> -->
+    </xacro:if>
+    <!-- Joint description -->
+    <m_joint name="${parent}__${fr}_${lr}_steer" type="fixed"
+             axis_xyz="0 0 0"
+             origin_rpy="0 0 0" origin_xyz="0 0 0"
+             parent="${parent}" child="${fr}_${lr}_steer"
+             limit_e="0" limit_l="0" limit_u="0" limit_v="0"/>
+    <!-- Link description -->
+    <m_link_mesh name="${fr}_${lr}_steer"
+                 color="${Red_Value}"
+                 origin_rpy="0 0 0"
+                 origin_xyz="${steer_x} ${steer_y} ${steer_z}"
+                 mass="1.0"
+                 ixx="0.0001" ixy="0.0" ixz="0.0"
+                 iyy="0.0001" iyz="0.0"
+                 izz="0.0001"
+                 meshfile="${mesh_file}"
+                 meshscale="1 1 1"/>
+    <gazebo reference="${fr}_${lr}_steer">
+      <visual name="${fr}_${lr}_steer_visual">
+          <material>
+              <ambient>0.5 0.5 0.5 1.0</ambient>
+              <specular>0.8 0.8 0.8 0.1</specular>
+              <diffuse>1.0 1.0 1.0 1.0</diffuse>
+          </material>
+      </visual>
+      <turnGravityOff>false</turnGravityOff>
+    </gazebo>
+    <!-- Transmission is important to link the joints and the controller -->
+    <!-- <transmission name="${fr}_${lr}_steer_joint_trans">
+      <type>transmission_interface/SimpleTransmission</type>
+      <joint name="${fr}_${lr}_steer_joint"/>
+      <actuator name="${fr}_${lr}_steer_joint_motor">
+          <hardwareInterface>EffortJointInterface</hardwareInterface>
+          <mechanicalReduction>1</mechanicalReduction>
+      </actuator>
+    </transmission> -->
+  </xacro:macro>
 </robot>

File: rover_desc_pkg/urdf/wheel.xacro (robot description, xacro)
@@ -1,50 +1,50 @@
 <?xml version="1.0"?>
 <robot name="wheel" xmlns:xacro="http://www.ros.org/wiki/xacro">
-    <!-- Begin - Include -->
-    <xacro:include filename="$(find rover_desc_pkg)/urdf/robot_parameters.xacro"/>
-    <xacro:include filename="$(find rover_desc_pkg)/urdf/links_joints.xacro"/>
-    <!-- End - Include -->
-    <xacro:macro name="wheel" params="fr lr parent translateX translateY"> <!-- fr: front, rear; lr: left, right -->
-        <!-- Compute wheel position based on its location -->
-        <xacro:property name="wheel_x" value="${translateX * world_x_origin_to_wheel_x_origin}" scope="local"/>
-        <xacro:property name="wheel_y" value="${translateY * world_y_origin_to_wheel_y_origin}" scope="local"/>
-        <xacro:property name="wheel_z" value="${wheel_radius}" scope="local"/>
-        <xacro:if value="${lr == 'right'}">
-            <xacro:property name="wheel_z" value="${wheel_radius + 0.0032}" scope="local"/>
-        </xacro:if>
-        <m_joint name="${r_link_01_name}__${fr}_${lr}_wheel" type="fixed"
-                 axis_xyz="0 0 0"
-                 origin_rpy="0 0 0" origin_xyz="0 0 0"
-                 parent="${parent}" child="${fr}_${lr}_wheel"
-                 limit_e="0" limit_l="0" limit_u="0" limit_v="0"/>
-        <m_link_mesh name="${fr}_${lr}_wheel"
-                     color="Black"
-                     origin_rpy="0 0 0"
-                     origin_xyz="${wheel_x} ${wheel_y} ${wheel_z}"
-                     mass="1.0"
-                     ixx="0.0001" ixy="0.0" ixz="0.0"
-                     iyy="0.0001" iyz="0.0"
-                     izz="0.0001"
-                     meshfile="package://rover_desc_pkg/meshes/rover_wheel.dae"
-                     meshscale="1 1 1"/>
-        <gazebo reference="${fr}_${lr}_wheel">
-            <visual name="${fr}_${lr}_wheel_visual">
-                <material>
-                    <ambient>0.5 0.5 0.5 1.0</ambient>
-                    <specular>0.8 0.8 0.8 0.1</specular>
-                    <diffuse>1.0 1.0 1.0 1.0</diffuse>
-                </material>
-            </visual>
-            <turnGravityOff>false</turnGravityOff>
-        </gazebo>
-        <!-- Transmission is important to link the joints and the controller -->
-        <!-- <transmission name="${fr}_${lr}_wheel_joint_trans">
-            <type>transmission_interface/SimpleTransmission</type>
-            <joint name="${fr}_${lr}_wheel_joint"/>
-            <actuator name="${fr}_${lr}_wheel_joint_motor">
-                <hardwareInterface>EffortJointInterface</hardwareInterface>
-                <mechanicalReduction>1</mechanicalReduction>
-            </actuator>
-        </transmission> -->
-    </xacro:macro>
+  <!-- Begin - Include -->
+  <xacro:include filename="$(find rover_desc_pkg)/urdf/robot_parameters.xacro"/>
+  <xacro:include filename="$(find rover_desc_pkg)/urdf/links_joints.xacro"/>
+  <!-- End - Include -->
+  <xacro:macro name="wheel" params="fr lr parent translateX translateY"> <!-- fr: front, rear; lr: left, right -->
+    <!-- Compute wheel position based on its location -->
+    <xacro:property name="wheel_x" value="${translateX * world_x_origin_to_wheel_x_origin}" scope="local"/>
+    <xacro:property name="wheel_y" value="${translateY * world_y_origin_to_wheel_y_origin}" scope="local"/>
+    <xacro:property name="wheel_z" value="${wheel_radius}" scope="local"/>
+    <xacro:if value="${lr == 'right'}">
+        <xacro:property name="wheel_z" value="${wheel_radius + 0.0032}" scope="local"/>
+    </xacro:if>
+    <m_joint name="${r_link_01_name}__${fr}_${lr}_wheel" type="fixed"
+             axis_xyz="0 0 0"
+             origin_rpy="0 0 0" origin_xyz="0 0 0"
+             parent="${parent}" child="${fr}_${lr}_wheel"
+             limit_e="0" limit_l="0" limit_u="0" limit_v="0"/>
+    <m_link_mesh name="${fr}_${lr}_wheel"
+                 color="${Black_Value}"
+                 origin_rpy="0 0 0"
+                 origin_xyz="${wheel_x} ${wheel_y} ${wheel_z}"
+                 mass="1.0"
+                 ixx="0.0001" ixy="0.0" ixz="0.0"
+                 iyy="0.0001" iyz="0.0"
+                 izz="0.0001"
+                 meshfile="package://rover_desc_pkg/meshes/rover_wheel.dae"
+                 meshscale="1 1 1"/>
+    <gazebo reference="${fr}_${lr}_wheel">
+      <visual name="${fr}_${lr}_wheel_visual">
+        <material>
+          <ambient>0.5 0.5 0.5 1.0</ambient>
+          <specular>0.8 0.8 0.8 0.1</specular>
+          <diffuse>1.0 1.0 1.0 1.0</diffuse>
+        </material>
+      </visual>
+      <turnGravityOff>false</turnGravityOff>
+    </gazebo>
+    <!-- Transmission is important to link the joints and the controller -->
+    <!-- <transmission name="${fr}_${lr}_wheel_joint_trans">
+      <type>transmission_interface/SimpleTransmission</type>
+      <joint name="${fr}_${lr}_wheel_joint"/>
+      <actuator name="${fr}_${lr}_wheel_joint_motor">
+        <hardwareInterface>EffortJointInterface</hardwareInterface>
+        <mechanicalReduction>1</mechanicalReduction>
+      </actuator>
+    </transmission> -->
+  </xacro:macro>
 </robot>

Commit message: Defined separate joints of each type.

File: rover_desc_pkg/urdf/links_joints.xacro (robot description, xacro)
@@ -2,6 +2,36 @@
 <robot xmlns:xacro="http://www.ros.org/wiki/xacro">
   <!-- Joint Macro -->
-  <xacro:macro name="m_joint" params="name type axis_xyz origin_xyz origin_rpy parent child limit_e limit_l limit_u limit_v">
-    <joint name="${name}" type="${type}">
+  <!-- fixed joint -->
+  <xacro:macro name="m_joint_fixed" params="name origin_xyz origin_rpy parent child">
+    <!-- fixed joint -->
+    <joint name="${name}" type="fixed">
+      <origin rpy="${origin_rpy}" xyz="${origin_xyz}"/>
+      <parent link="${parent}"/>
+      <child link="${child}"/>
+    </joint>
+  </xacro:macro>
+  <!-- continuous joint -->
+  <xacro:macro name="m_joint_cont" params="name axis_xyz origin_xyz origin_rpy parent child limit_e limit_v">
+    <joint name="${name}" type="continuous">
+      <axis xyz="${axis_xyz}"/>
+      <limit effort="${limit_e}" velocity="${limit_v}"/>
+      <origin rpy="${origin_rpy}" xyz="${origin_xyz}"/>
+      <parent link="${parent}"/>
+      <child link="${child}"/>
+    </joint>
+    <transmission name="trans_${name}">
+      <type>transmission_interface/SimpleTransmission</type>
+      <joint name="${name}">
+        <hardwareInterface>hardware_interface/EffortJointInterface</hardwareInterface>
+      </joint>
+      <actuator name="motor_${name}">
+        <hardwareInterface>hardware_interface/EffortJointInterface</hardwareInterface>
+        <mechanicalReduction>1</mechanicalReduction>
+      </actuator>
+    </transmission>
+  </xacro:macro>
+  <!-- revolute joint -->
+  <xacro:macro name="m_joint_rev" params="name axis_xyz origin_xyz origin_rpy parent child limit_e limit_l limit_u limit_v">
+    <joint name="${name}" type="revolute">
       <axis xyz="${axis_xyz}"/>
       <limit effort="${limit_e}" lower="${limit_l}" upper="${limit_u}" velocity="${limit_v}"/>

Commit message: Corrected material in visual of the links. Removed inertial from m_box_link.

File: rover_desc_pkg/urdf/links_joints.xacro (robot description, xacro)
@@ -70,24 +70,11 @@
           <cylinder radius="${radius}" length="${length}"/>
         </geometry>
-        <material name="">
-          <color rgba="${color}"/>
-        </material>
+        <material name="${color}"/>
       </visual>
     </link>
   </xacro:macro>
   <!-- Box link Macro -->
-  <xacro:macro name="m_link_box" params="name color origin_xyz origin_rpy size mass ixx ixy ixz iyy iyz izz">
+  <xacro:macro name="m_link_box" params="name color origin_xyz origin_rpy size">
     <link name="${name}">
-      <inertial>
-        <mass value="${mass}"/>
-        <origin rpy="${origin_rpy}" xyz="${origin_xyz}"/>
-        <inertia ixx="${ixx}" ixy="${ixy}" ixz="${ixz}" iyy="${iyy}" iyz="${iyz}" izz="${izz}"/>
-      </inertial>
-      <collision>
-        <origin rpy="${origin_rpy}" xyz="${origin_xyz}"/>
-        <geometry>
-          <box size="${size}"/>
-        </geometry>
-      </collision>
       <visual>
         <origin rpy="${origin_rpy}" xyz="${origin_xyz}"/>
@@ -95,7 +82,5 @@
           <box size="${size}"/>
         </geometry>
-        <material name="">
-          <color rgba="${color}"/>
-        </material>
+        <material name="${color}"/>
       </visual>
     </link>
@@ -120,7 +105,5 @@
             <mesh filename="${meshfile}" scale="${meshscale}"/>
         </geometry>
-        <material name="">
-            <color rgba="${color}"/>
-        </material>
+        <material name="${color}"/>
       </visual>
     </link>

Commit message: Added dynamics parameters.

File: rover_desc_pkg/urdf/links_joints.xacro (robot description, xacro)
@@ -32,8 +32,9 @@
   </xacro:macro>
   <!-- revolute joint -->
-  <xacro:macro name="m_joint_rev" params="name axis_xyz origin_xyz origin_rpy parent child limit_e limit_l limit_u limit_v">
+  <xacro:macro name="m_joint_rev" params="name axis_xyz origin_xyz origin_rpy parent child limit_e limit_l limit_u limit_v dynamics_d dynamics_f">
     <joint name="${name}" type="revolute">
       <axis xyz="${axis_xyz}"/>
       <limit effort="${limit_e}" lower="${limit_l}" upper="${limit_u}" velocity="${limit_v}"/>
+      <dynamics damping="${dynamics_d}" friction="${dynamics_f}"/>
       <origin rpy="${origin_rpy}" xyz="${origin_xyz}"/>
       <parent link="${parent}"/>

Commit message: Customized macros for inbuilt inertial. Removed color from mesh macro.

File: rover_desc_pkg/urdf/links_joints.xacro (robot description, xacro)
@@ -32,7 +32,7 @@
   </xacro:macro>
   <!-- revolute joint -->
-  <xacro:macro name="m_joint_rev" params="name axis_xyz origin_xyz origin_rpy parent child limit_e limit_l limit_u limit_v dynamics_d dynamics_f">
+  <xacro:macro name="m_joint_rev" params="name axis_xyz axis_rpy origin_xyz origin_rpy parent child limit_e limit_l limit_u limit_v dynamics_d dynamics_f">
     <joint name="${name}" type="revolute">
-      <axis xyz="${axis_xyz}"/>
+      <axis rpy="axis_rpy" xyz="${axis_xyz}"/>
       <limit effort="${limit_e}" lower="${limit_l}" upper="${limit_u}" velocity="${limit_v}"/>
       <dynamics damping="${dynamics_d}" friction="${dynamics_f}"/>
@@ -52,16 +52,30 @@
     </transmission>
   </xacro:macro>
-  <!-- Cylinder link Macro -->
-  <xacro:macro name="m_link_cylinder" params="name color origin_xyz origin_rpy radius length mass ixx ixy ixz iyy iyz izz">
+  <!-- Cylinder link Macro without inertia -->
+  <xacro:macro name="m_link_cylinder" params="name color origin_xyz origin_rpy r l">
+    <link name="${name}">
+      <visual>
+        <origin rpy="${origin_rpy}" xyz="${origin_xyz}"/>
+        <geometry>
+          <cylinder radius="${r}" length="${l}"/>
+        </geometry>
+        <material name="${color}"/>
+      </visual>
+    </link>
+  </xacro:macro>
+  <!-- Cylinder link Macro with inertia -->
+  <xacro:macro name="m_link_cylinder_inertia" params="name color origin_xyz origin_rpy r l m">
     <link name="${name}">
       <inertial>
-        <mass value="${mass}"/>
+        <mass value="${m}"/>
         <origin rpy="${origin_rpy}" xyz="${origin_xyz}"/>
-        <inertia ixx="${ixx}" ixy="${ixy}" ixz="${ixz}" iyy="${iyy}" iyz="${iyz}" izz="${izz}"/>
+        <inertia ixx="${m*(3*r*r+l*l)/12}" ixy="0.0" ixz="0.0"
+                 iyy="${m*(3*r*r+l*l)/12}" iyz="0.0"
+                 izz="${m*r*r/2}"/>
       </inertial>
       <collision>
         <origin rpy="${origin_rpy}" xyz="${origin_xyz}"/>
         <geometry>
-          <cylinder radius="${radius}" length="${length}"/>
+          <cylinder radius="${r}" length="${l}"/>
         </geometry>
       </collision>
@@ -69,5 +83,5 @@
         <origin rpy="${origin_rpy}" xyz="${origin_xyz}"/>
         <geometry>
-          <cylinder radius="${radius}" length="${length}"/>
+          <cylinder radius="${r}" length="${l}"/>
         </geometry>
         <material name="${color}"/>
@@ -75,11 +89,36 @@
     </link>
   </xacro:macro>
-  <!-- Box link Macro -->
-  <xacro:macro name="m_link_box" params="name color origin_xyz origin_rpy size">
+  <!-- Box link Macro without inertia -->
+  <xacro:macro name="m_link_box" params="name color origin_xyz origin_rpy w d h">
     <link name="${name}">
       <visual>
         <origin rpy="${origin_rpy}" xyz="${origin_xyz}"/>
         <geometry>
-          <box size="${size}"/>
+          <box size="${w} ${d} ${h}"/>
+        </geometry>
+        <material name="${color}"/>
+      </visual>
+    </link>
+  </xacro:macro>
+  <!-- Box link Macro with inertia -->
+  <xacro:macro name="m_link_box_inertia" params="name color origin_xyz origin_rpy m w d h">
+    <link name="${name}">
+      <inertial>
+        <mass value="${m}"/>
+        <origin rpy="${origin_rpy}" xyz="${origin_xyz}"/>
+        <inertia ixx="${m*(d*d+h*h)/12}" ixy="0" ixz="0"
+                 iyy="${m*(w*w+h*h)/12}" iyz="0"
+                 izz="${m*(w*w+d*d)/12}"/>
+      </inertial>
+      <collision>
+        <origin rpy="${origin_rpy}" xyz="${origin_xyz}"/>
+        <geometry>
+          <box size="${w} ${d} ${h}"/>
+        </geometry>
+      </collision>
+      <visual>
+        <origin rpy="${origin_rpy}" xyz="${origin_xyz}"/>
+        <geometry>
+          <box size="${w} ${d} ${h}"/>
         </geometry>
         <material name="${color}"/>
@@ -88,10 +127,12 @@
   </xacro:macro>
   <!-- Mesh link Macro -->
-  <xacro:macro name="m_link_mesh" params="name color origin_xyz origin_rpy meshfile meshscale mass ixx ixy ixz iyy iyz izz">
+  <xacro:macro name="m_link_mesh" params="name origin_xyz origin_rpy meshfile meshscale m w d h">
     <link name="${name}">
       <inertial>
-        <mass value="${mass}"/>
+        <mass value="${m}"/>
         <origin rpy="${origin_rpy}" xyz="${origin_xyz}"/>
-        <inertia ixx="${ixx}" ixy="${ixy}" ixz="${ixz}" iyy="${iyy}" iyz="${iyz}" izz="${izz}"/>
+        <inertia ixx="${m*(d*d+h*h)/12}" ixy="0" ixz="0"
+                 iyy="${m*(w*w+h*h)/12}" iyz="0"
+                 izz="${m*(w*w+d*d)/12}"/>
       </inertial>
       <collision>
@@ -106,5 +147,4 @@
             <mesh filename="${meshfile}" scale="${meshscale}"/>
         </geometry>
-        <material name="${color}"/>
       </visual>
     </link>

Commit message: Seperated inertial based on shape in mesh link.

File: rover_desc_pkg/urdf/links_joints.xacro (robot description, xacro)
@@ -127,12 +127,19 @@
   </xacro:macro>
   <!-- Mesh link Macro -->
-  <xacro:macro name="m_link_mesh" params="name origin_xyz origin_rpy meshfile meshscale m w d h">
+  <xacro:macro name="m_link_mesh" params="name shape origin_xyz origin_rpy meshfile meshscale m w d h">
     <link name="${name}">
       <inertial>
         <mass value="${m}"/>
         <origin rpy="${origin_rpy}" xyz="${origin_xyz}"/>
-        <inertia ixx="${m*(d*d+h*h)/12}" ixy="0" ixz="0"
-                 iyy="${m*(w*w+h*h)/12}" iyz="0"
-                 izz="${m*(w*w+d*d)/12}"/>
+        <xacro:if value="${shape == 'box'}">
+          <inertia ixx="${m*(d*d+h*h)/12}" ixy="0" ixz="0"
+                   iyy="${m*(w*w+h*h)/12}" iyz="0"
+                   izz="${m*(w*w+d*d)/12}"/>
+        </xacro:if>
+        <xacro:if value="${shape == 'cylinder'}">
+          <inertia ixx="${m*(3*w*w+h*h)/12}" ixy="0.0" ixz="0.0"
+                   iyy="${m*(3*w*w+h*h)/12}" iyz="0.0"
+                   izz="${m*h*h/2}"/>
+        </xacro:if>
       </inertial>
       <collision>
