Commit message: Deleted xacro properties and customized the model.

File: rover_desc_pkg/urdf/rover_robot.xacro (robot description, xacro)
@@ -1,78 +1,40 @@
 <?xml version="1.0"?>
 <robot name="rover_robot" xmlns:xacro="http://www.ros.org/wiki/xacro">
-    <xacro:include filename="$(find rover_desc_pkg)/urdf/wheel.urdf.xacro"/>
-    <!-- Defining the colors used in the robot -->
-    <material name="Black">
-        <color rgba="${0.0/255} ${0.0/255} ${0.0/255} ${255/255}"/>
-    </material>
-    <material name="Red">
-        <color rgba="${204/255} ${0.0/255} ${0.0/255} ${255/255}"/>
-    </material>
-    <material name="White">
-        <color rgba="${255/255} ${255/255} ${255/255} ${255/255}"/>
-    </material>
-    <material name="Blue">
-        <color rgba="${0.0/255} ${0.0/255} ${204/255} ${255/255}"/>
-    </material>
-    <!-- Property list -->
-    <!-- All the units are in m-kg-s-radians unit system -->
-    <xacro:property name="M_PI" value="3.141592653"/>
-    <xacro:property name="DEG_TO_RAD" value="0.017453293"/>
-    <!-- Main body dimensions -->
-    <xacro:property name="chassis_length" value="1.02"/>
-    <xacro:property name="chassis_width" value="0.651"/>
-    <xacro:property name="chassis_height" value="0.445"/>
-    <xacro:property name="chassis_mass" value="5"/> <!-- in Kg -->
-    <!-- Base footprint -->
-    <link name="chassis_footprint">
-        <visual>
-            <origin xyz="0 0 0" rpy="0 0 0"/>
-            <geometry>
-                <box size="0.001 0.001 0.001"/>
-            </geometry>
-        </visual>
-        <inertial>
-            <origin xyz="0 0 0"/>
-            <mass value="0.0001"/>
-            <inertia ixx="0.0001" ixy="0.0" ixz="0.0"
-                     iyy="0.0001" iyz="0.0"
-                     izz="0.0001"/>
-        </inertial>
-    </link>
-    <gazebo reference="chassis_footprint">
+    <!-- Begin - Include -->
+    <xacro:include filename="$(find rover_desc_pkg)/urdf/robot_parameters.xacro"/>
+    <xacro:include filename="$(find rover_desc_pkg)/urdf/links_joints.xacro"/>
+    <!-- End - Include -->
+    <!-- Begin - Robot Description -->
+    <!-- Chassis footprint -->
+    <m_link_box name="${r_link_00_name}"
+                color="White"
+                origin_rpy="0 0 0" origin_xyz="0 0 0"
+                mass="0.0001"
+                ixx="0.0001" ixy="0.0" ixz="0.0"
+                iyy="0.0001" iyz="0.0"
+                izz="0.0001"
+                size="0.0001 0.0001 0.0001"/>
+    <gazebo reference="${r_link_00_name}">
         <turnGravityOff>false</turnGravityOff>
     </gazebo>
-    <joint name="chassis_footprint_joint" type="fixed">
-        <parent link="chassis_footprint"/>
-        <child link="chassis_link"/>
-        <origin xyz="0 0 0" rpy="0 0 0"/>
-    </joint>
-    <link name="chassis_link">
-        <visual>
-            <origin xyz="0 0 0" rpy="0 0 0"/>
-            <geometry>
-                <box size ="${chassis_length} ${chassis_width} ${chassis_height}"/>
-            </geometry>
-            <material name="white"/>
-        </visual>
-        <collision>
-            <origin xyz="0 0 0" rpy="0 0 0"/>
-            <geometry>
-                <box size ="${chassis_length} ${chassis_width} ${chassis_height}"/>
-            </geometry>
-        </collision>
-        <inertial>
-            <origin xyz="0 0 0" rpy="0 0 0"/>
-            <mass value="${chassis_mass}"/>
-            <inertia ixx="50" ixy="0" ixz="0"
-                     iyy="50" iyz="0"
-                     izz="50"/>
-        </inertial>
-    </link>
-    <gazebo reference="chassis_link">
+    <m_joint name="${r_link_00_name}__${r_link_01_name}" type="fixed"
+             axis_xyz="0 0 0"
+             origin_rpy="0 0 0" origin_xyz="0 0 0"
+             parent="${r_link_00_name}" child="${r_link_01_name}"
+             limit_e="0" limit_l="0" limit_u="0" limit_v="0"/>
+    <m_link_mesh name="${r_link_01_name}"
+                 color="White"
+                 origin_rpy="0 0 0" origin_xyz="0 0 ${chassis_height/2}"
+                 mass="1.0"
+                 ixx="0.0001" ixy="0.0" ixz="0.0"
+                 iyy="0.0001" iyz="0.0"
+                 izz="0.0001"
+                 meshfile="package://rover_desc_pkg/meshes/rover_chassis.stl"
+                 meshscale="1 1 1"/>
+    <gazebo reference="${r_link_01_name}">
         <material>Gazebo/White</material>
         <turnGravityOff>false</turnGravityOff>
     </gazebo>
-    <!-- Wheels definitions -->
+    <!-- End - Robot Description -->
     <!-- Rover -->
     <gazebo>

Commit message: Added inverter link and corresponding joint.

File: rover_desc_pkg/urdf/rover_robot.xacro (robot description, xacro)
@@ -36,4 +36,22 @@
         <turnGravityOff>false</turnGravityOff>
     </gazebo>
+    <m_joint name="${r_link_01_name}__${r_link_02_name}" type="fixed"
+             axis_xyz="0 0 0"
+             origin_rpy="0 0 0" origin_xyz="0 0 0"
+             parent="${r_link_01_name}" child="${r_link_02_name}"
+             limit_e="0" limit_l="0" limit_u="0" limit_v="0"/>
+    <m_link_mesh name="${r_link_02_name}"
+                 color="Green"
+                 origin_rpy="0 0 0" origin_xyz="0 0 ${inverter_height/2}"
+                 mass="1.0"
+                 ixx="0.0001" ixy="0.0" ixz="0.0"
+                 iyy="0.0001" iyz="0.0"
+                 izz="0.0001"
+                 meshfile="package://rover_desc_pkg/meshes/inverter.stl"
+                 meshscale="1 1 1"/>
+    <gazebo reference="${r_link_02_name}">
+        <material>Gazebo/Green</material>
+        <turnGravityOff>false</turnGravityOff>
+    </gazebo>
     <!-- End - Robot Description -->
     <!-- Rover -->

Commit message: Replaced .stl file with .dae and edited the Gazebo materials.

File: rover_desc_pkg/urdf/rover_robot.xacro (robot description, xacro)
@@ -31,8 +31,14 @@
                  iyy="0.0001" iyz="0.0"
                  izz="0.0001"
-                 meshfile="package://rover_desc_pkg/meshes/rover_chassis.stl"
+                 meshfile="package://rover_desc_pkg/meshes/rover_chassis.dae"
                  meshscale="1 1 1"/>
     <gazebo reference="${r_link_01_name}">
-        <material>Gazebo/White</material>
+        <visual name="visual">
+            <material>
+                <ambient>0 0 0 0</ambient>
+                <specular>0.8 0.8 0.8 0.1</specular>
+                <diffuse>1.0 1.0 1.0 1.0</diffuse>
+            </material>
+        </visual>
         <turnGravityOff>false</turnGravityOff>
     </gazebo>
@@ -49,8 +55,14 @@
                  iyy="0.0001" iyz="0.0"
                  izz="0.0001"
-                 meshfile="package://rover_desc_pkg/meshes/inverter.stl"
+                 meshfile="package://rover_desc_pkg/meshes/inverter.dae"
                  meshscale="1 1 1"/>
     <gazebo reference="${r_link_02_name}">
-        <material>Gazebo/Green</material>
+        <visual name="visual">
+            <material>
+                <ambient>0.5 0.5 0.5 1.0</ambient>
+                <specular>0.8 0.8 0.8 0.1</specular>
+                <diffuse>1.0 1.0 1.0 1.0</diffuse>
+            </material>
+        </visual>
         <turnGravityOff>false</turnGravityOff>
     </gazebo>

Commit message: Renamed visuals

File: rover_desc_pkg/urdf/rover_robot.xacro (robot description, xacro)
@@ -34,7 +34,7 @@
                  meshscale="1 1 1"/>
     <gazebo reference="${r_link_01_name}">
-        <visual name="visual">
+        <visual name="${r_link_01_name}_visual">
             <material>
-                <ambient>0 0 0 0</ambient>
+                <ambient>0.5 0.5 0.5 1.0</ambient>
                 <specular>0.8 0.8 0.8 0.1</specular>
                 <diffuse>1.0 1.0 1.0 1.0</diffuse>
@@ -58,5 +58,5 @@
                  meshscale="1 1 1"/>
     <gazebo reference="${r_link_02_name}">
-        <visual name="visual">
+        <visual name="${r_link_02_name}_visual">
             <material>
                 <ambient>0.5 0.5 0.5 1.0</ambient>

Commit message: Simplified gazebo material properties.

File: rover_desc_pkg/urdf/rover_robot.xacro (robot description, xacro)
@@ -31,11 +31,5 @@
                meshscale="1 1 1"/>
   <gazebo reference="${r_link_01_name}">
-    <visual name="${r_link_01_name}_visual">
-      <material>
-        <ambient>0.5 0.5 0.5 1.0</ambient>
-        <specular>0.8 0.8 0.8 0.1</specular>
-        <diffuse>1.0 1.0 1.0 1.0</diffuse>
-      </material>
-    </visual>
+    <material>Gazebo/Grey</material>
     <turnGravityOff>false</turnGravityOff>
   </gazebo>

File: rover_desc_pkg/urdf/steer.xacro (robot description, xacro)
@@ -40,11 +40,5 @@
                  meshscale="1 1 1"/>
     <gazebo reference="${fr}_${lr}_steer">
-      <visual name="${fr}_${lr}_steer_visual">
-        <material>
-          <ambient>0.5 0.5 0.5 1.0</ambient>
-          <specular>0.8 0.8 0.8 0.1</specular>
-          <diffuse>1.0 1.0 1.0 1.0</diffuse>
-        </material>
-      </visual>
+      <material>Gazebo/Grey</material>
       <turnGravityOff>false</turnGravityOff>
     </gazebo>

File: rover_desc_pkg/urdf/wheel.xacro (robot description, xacro)
@@ -29,9 +29,10 @@
     <gazebo reference="${fr}_${lr}_wheel">
       <visual name="${fr}_${lr}_wheel_visual">
-        <material>
-          <ambient>0.5 0.5 0.5 1.0</ambient>
-          <specular>0.8 0.8 0.8 0.1</specular>
-          <diffuse>1.0 1.0 1.0 1.0</diffuse>
-        </material>
+        <mu1 value="1.0"/>
+        <mu2 value="1.0"/>
+        <kp value="10000000.0"/>
+        <kd value="1.0"/>
+        <fdir1 value="0 1 0"/>
+        <material>Gazebo/Grey</material>
       </visual>
       <turnGravityOff>false</turnGravityOff>

Commit message: Suppressed xml warning by xacro to the links and joints. Fixed colors of the links. Fixed gazebo color references.

File: rover_desc_pkg/urdf/rover_robot.xacro (robot description, xacro)
@@ -9,41 +9,36 @@
   <!-- Begin - Robot Description -->
   <!-- Chassis footprint -->
-  <m_link_box name="${r_link_00_name}"
-              color="${White_Value}"
-              origin_rpy="0 0 0" origin_xyz="0 0 0"
-              mass="0.0001"
-              ixx="0.0" ixy="0.0" ixz="0.0"
-              iyy="0.0" iyz="0.0"
-              izz="0.0"
-              size="0.0001 0.0001 0.0001"/>
+  <xacro:m_link_box name="${r_link_00_name}"
+                    color="white"
+                    origin_rpy="0 0 0" origin_xyz="0 0 0"
+                    size="0.0001 0.0001 0.0001"/>
   <gazebo reference="${r_link_00_name}">
-    <turnGravityOff>false</turnGravityOff>
+    <material>Gazebo/White</material>
   </gazebo>
-  <m_link_mesh name="${r_link_01_name}"
-               color="${White_Value}"
-               origin_rpy="0 0 0"
-               origin_xyz="0 0 ${wheel_radius + steer_z_origin_to_wheel_z_origin - chassis_z_origin_to_steer_z_origin}"
-               mass="1.0"
-               ixx="0.0001" ixy="0.0" ixz="0.0"
-               iyy="0.0001" iyz="0.0"
-               izz="0.0001"
-               meshfile="package://rover_desc_pkg/meshes/rover_chassis.dae"
-               meshscale="1 1 1"/>
+  <xacro:m_link_mesh name="${r_link_01_name}"
+                     color="gray"
+                     origin_rpy="0 0 0"
+                     origin_xyz="0 0 ${wheel_radius + steer_z_origin_to_wheel_z_origin - chassis_z_origin_to_steer_z_origin}"
+                     mass="1.0"
+                     ixx="0.0001" ixy="0.0" ixz="0.0"
+                     iyy="0.0001" iyz="0.0"
+                     izz="0.0001"
+                     meshfile="package://rover_desc_pkg/meshes/rover_chassis.dae"
+                     meshscale="1 1 1"/>
   <gazebo reference="${r_link_01_name}">
-    <material>Gazebo/Grey</material>
-    <turnGravityOff>false</turnGravityOff>
+    <material>Gazebo/Yellow</material>
   </gazebo>
-  <m_joint_fixed name="${r_link_00_name}__${r_link_01_name}"
-                 origin_rpy="0 0 0" origin_xyz="0 0 0"
-                 parent="${r_link_00_name}" child="${r_link_01_name}"/>
+  <xacro:m_joint_fixed name="${r_link_00_name}__${r_link_01_name}"
+                       origin_rpy="0 0 0" origin_xyz="0 0 0"
+                       parent="${r_link_00_name}" child="${r_link_01_name}"/>
   <!-- Steers & Wheels -->
-  <steer fr="front" lr="right" parent="${r_link_01_name}" type="revolute" translateX="1" translateY="-1"/>
-  <steer fr="front" lr="left" parent="${r_link_01_name}" type="revolute" translateX="1" translateY="1"/>
-  <steer fr="rear" lr="right" parent="${r_link_01_name}" type="fixed" translateX="-1" translateY="-1"/>
-  <steer fr="rear" lr="left" parent="${r_link_01_name}" type="fixed" translateX="-1" translateY="1"/>
-  <wheel fr="front" lr="right" parent="front_right_steer" translateX="1" translateY="-1"/>
-  <wheel fr="front" lr="left" parent="front_left_steer" translateX="1" translateY="1"/>
-  <wheel fr="rear" lr="right" parent="rear_right_steer" translateX="-1" translateY="-1"/>
-  <wheel fr="rear" lr="left" parent="rear_left_steer" translateX="-1" translateY="1"/>
+  <xacro:steer fr="front" lr="right" parent="${r_link_01_name}" type="revolute" translateX="1" translateY="-1"/>
+  <xacro:steer fr="front" lr="left" parent="${r_link_01_name}" type="revolute" translateX="1" translateY="1"/>
+  <xacro:steer fr="rear" lr="right" parent="${r_link_01_name}" type="fixed" translateX="-1" translateY="-1"/>
+  <xacro:steer fr="rear" lr="left" parent="${r_link_01_name}" type="fixed" translateX="-1" translateY="1"/>
+  <xacro:wheel fr="front" lr="right" parent="front_right_steer" translateX="1" translateY="-1"/>
+  <xacro:wheel fr="front" lr="left" parent="front_left_steer" translateX="1" translateY="1"/>
+  <xacro:wheel fr="rear" lr="right" parent="rear_right_steer" translateX="-1" translateY="-1"/>
+  <xacro:wheel fr="rear" lr="left" parent="rear_left_steer" translateX="-1" translateY="1"/>
   <!-- End - Robot Description -->
   <!-- Rover -->
