Commit message: Merged 'development' into 'master' after fixing.
Squashed commit of the following:

commit b23850bf296459da051ec37ecf808b5c054982ba
Author: mturktest123 <mturktest123@gmail.com>
Date:   Sun May 10 09:18:04 2020 -0500

    Update README.md

commit 6ba9ecd410c74782c9c26ba214c5853ccd4270b6
Author: mturktest123 <mturktest123@gmail.com>
Date:   Sun May 10 07:21:01 2020 -0500

    Update README.md

commit 2594f331aba4700fc4ba715a4201365113689bb2
Author: Ravi Sharma <s2007.ravi@gmail.com>
Date:   Wed May 6 20:01:24 2020 +0530

    Corrected the formatting.

commit 9172442f28aa6c8fc558baaba35d83cd843a2a0e
Merge: dd8e596 d86b988
Author: Ravi Sharma <s2007.ravi@gmail.com>
Date:   Wed May 6 19:53:12 2020 +0530

    Merge branch 'development' of github.com:mturktest123/RoverROS into development

commit dd8e596296abf33542306af7b09f4eefdfe449e9
Author: Ravi Sharma <s2007.ravi@gmail.com>
Date:   Wed May 6 19:45:59 2020 +0530

    Change the mesh of link3 to match actual arm.
    Reduced length of link3a.
    Corrected the Z value of arm position wrt rover.

commit d86b9883d5d05e8aa34402bb9a2326aa778f54ec
Author: mturktest123 <mturktest123@gmail.com>
Date:   Mon May 4 21:55:50 2020 -0500

    Update README.md

commit 4473015fa4bb11322a4bda959d06acd6c5701d65
Author: mturktest123 <mturktest123@gmail.com>
Date:   Mon May 4 10:37:16 2020 -0500

    Update README.md

commit 5047dffbcaa0a04c02a30fb43954bb3b37b127e4
Author: Ravi Sharma <s2007.ravi@gmail.com>
Date:   Sun May 3 18:51:24 2020 +0530

    Corrected grammar & spelling mistakes.

commit b0750c551d3479b7b2598dc3a0889c7fb2f8c6d1
Author: Ravi Sharma <s2007.ravi@gmail.com>
Date:   Sun May 3 18:13:14 2020 +0530

    Corrected tabs.

commit a0016fb5670985f4950e385fc338a4f2e8733aae
Author: Ravi Sharma <s2007.ravi@gmail.com>
Date:   Sun May 3 18:01:13 2020 +0530

    Corrected tabs.

commit c5d500589c057277cb56c1240b5ee4da98cc95de
Author: Ravi Sharma <s2007.ravi@gmail.com>
Date:   Sun May 3 17:58:32 2020 +0530

    Updated code formatting.

commit 5eb22535df046ddfe0a250e1319ee4f39cbb9ebe
Author: Ravi Sharma <s2007.ravi@gmail.com>
Date:   Sun May 3 17:52:56 2020 +0530

    Again Corrected the formatting.

commit 6e9ae1cc5276290bac0fed461b63cee85fb14b4c
Author: Ravi Sharma <s2007.ravi@gmail.com>
Date:   Sun May 3 17:48:57 2020 +0530

    Corrected the formatting.

commit 6ad7b4a04d6b1bcfd4b44d707e03d4d299506282
Author: Ravi Sharma <s2007.ravi@gmail.com>
Date:   Sun May 3 17:42:08 2020 +0530

    Updated with packages description.

commit 622715ef1bbe84c0e0eaf5fc0ef0b46bb973c7c6
Author: Ravi Sharma <s2007.ravi@gmail.com>
Date:   Sat May 2 22:54:16 2020 +0530

    Keyboard control of Rover & MoveIT control of Arm.

commit 2958deaaab7fcb50c633b34383bf2ddf4c0176d4
Author: Ravi Sharma <s2007.ravi@gmail.com>
Date:   Sat May 2 21:56:26 2020 +0530

    Corrected the comments.

commit 89bd3ac848bceb344d88f10a025dfb66590d44c9
Author: Ravi Sharma <s2007.ravi@gmail.com>
Date:   Sat May 2 21:55:16 2020 +0530

    Removed rover_controller from the config.
    Rover gets controlled using keyboard commands.

commit 20c434da4bf6e484df9cc8cf120e536916401341
Author: Ravi Sharma <s2007.ravi@gmail.com>
Date:   Wed Apr 29 23:03:59 2020 +0530

    Relaxed params to execute trajectory motions.

commit 58d6dd56b897a90417b32c7625058af728a1ad75
Author: Ravi Sharma <s2007.ravi@gmail.com>
Date:   Wed Apr 29 23:01:57 2020 +0530

    Fine tuned PID and relaxed constraints.

commit 65d66d17f77430980049329572fca2dfd4d593aa
Author: Ravi Sharma <s2007.ravi@gmail.com>
Date:   Wed Apr 29 22:56:19 2020 +0530

    Fine tuned PID values.

commit a70cab25629697e20ab361336e8c1ee080b56e46
Author: Ravi Sharma <s2007.ravi@gmail.com>
Date:   Wed Apr 29 22:53:15 2020 +0530

    Added Damping and Friction.

commit 1ffbc4bea73abf30d075ee664cec1596edbca0df
Author: Ravi Sharma <s2007.ravi@gmail.com>
Date:   Wed Apr 29 22:50:41 2020 +0530

    Raised arm along Z.

commit f93d5448f3776f81b9fbdf4494b643f909aa8dd5
Author: Ravi Sharma <s2007.ravi@gmail.com>
Date:   Wed Apr 29 22:49:43 2020 +0530

    Changed joint limits.

commit a2816e2c2d6bfdd80133b6da8a8661f77ef7b5b8
Author: Ravi Sharma <s2007.ravi@gmail.com>
Date:   Tue Apr 28 01:23:06 2020 +0530

    Launch MoveIT control of arm in Gazebo.

commit 50612c5e2b774fed7363d9073d3723f7391e5792
Author: Ravi Sharma <s2007.ravi@gmail.com>
Date:   Tue Apr 28 01:21:52 2020 +0530

    Fixed many things to be able to control arm in Gazebo from MoveIT.

commit 3f5fe7b455fd93c8e5ec20401cb6ac9a37edac60
Author: Ravi Sharma <s2007.ravi@gmail.com>
Date:   Sun Apr 26 23:10:37 2020 +0530

    Added JointTrajectoryControllers.

commit b9d5916e0079bca30fd0c2d74bf68bd39f891344
Author: Ravi Sharma <s2007.ravi@gmail.com>
Date:   Sun Apr 26 23:09:48 2020 +0530

    Modified config.

commit dd826fde2640db959ff5d3642f8941c8ffcf07c1
Author: Ravi Sharma <s2007.ravi@gmail.com>
Date:   Sun Apr 26 23:09:06 2020 +0530

    Modified MoveIT config to add ros_controllers.

commit 847e8f567c78a9ba75482293c80c83559c8bb1fe
Author: Ravi Sharma <s2007.ravi@gmail.com>
Date:   Sun Apr 26 19:27:52 2020 +0530

    New MoveIT package to simulate the arm.

commit 6054b7f336ac48cc247f1efdcb0cad7cb2b9a353
Author: Ravi Sharma <s2007.ravi@gmail.com>
Date:   Sun Apr 26 17:24:08 2020 +0530

    Updated the definitions according to new package.

commit 5ab54ff9d20e7f33ee70c256b72fed3ba716b2f5
Author: Ravi Sharma <s2007.ravi@gmail.com>
Date:   Sun Apr 26 17:23:12 2020 +0530

    Customized the definitions according to new package.

commit 3f6fee01625e03422b183578dc7c51e9d3611d43
Author: Ravi Sharma <s2007.ravi@gmail.com>
Date:   Sun Apr 26 17:21:19 2020 +0530

    Renamed the package.

commit 0211f6d52a33fd151a4e4d5f889d4d609c7233cb
Author: Ravi Sharma <s2007.ravi@gmail.com>
Date:   Sun Apr 26 12:22:25 2020 +0530

    Added new package to define common parameters.

commit d02b24b61b6535bc72dd6e0d0c52c9412de48556
Author: Ravi Sharma <s2007.ravi@gmail.com>
Date:   Thu Apr 23 09:51:39 2020 +0530

    Launch keyboard control of Rover with Arm.

commit c0d54377fcf9215e4b417e8b1dc3853a4f58fc3b
Author: Ravi Sharma <s2007.ravi@gmail.com>
Date:   Wed Apr 22 22:03:32 2020 +0530

    Rotated chassis by 180 degrees across Z.
    Corrected steer position across X because of chassis rotation.

commit 886ae0383dfa4af237d99ab8dffbc60c656789d1
Author: Ravi Sharma <s2007.ravi@gmail.com>
Date:   Wed Apr 22 22:03:11 2020 +0530

    Renamed arm_base_link to arm_foot_cyl.

commit deaabe7bd7e5cc3e149facca39b70a94fc0251eb
Author: Ravi Sharma <s2007.ravi@gmail.com>
Date:   Wed Apr 22 22:01:29 2020 +0530

    Renamed arm_base_link to arm_foot_cyl.
    Corrected the location of arm at Z.

commit 7ab508370fd4edbe81a7ec7e45e0bb034c64a084
Author: Ravi Sharma <s2007.ravi@gmail.com>
Date:   Wed Apr 22 17:27:20 2020 +0530

    Renamed plotjuggler node.

commit 0b9188fdb55774875d75002b594554686b476e8a
Author: Ravi Sharma <s2007.ravi@gmail.com>
Date:   Wed Apr 22 17:17:30 2020 +0530

    Added plotjuggler.

commit db7a66b7ed7ba353a10d34f1b1d4dbe2d05732fa
Author: Ravi Sharma <s2007.ravi@gmail.com>
Date:   Wed Apr 22 15:47:39 2020 +0530

    Avoided instantiation of gazebo_ros_control twice.

commit 12f354e2ea72f96a61b72cd160b57791887a7057
Author: Ravi Sharma <s2007.ravi@gmail.com>
Date:   Tue Apr 21 23:17:12 2020 +0530

    Launch rover & arm in Gazebo.

commit 359f8702ae0fb5dfa249b7202510d5f1fab6a435
Author: Ravi Sharma <s2007.ravi@gmail.com>
Date:   Tue Apr 21 22:10:45 2020 +0530

    Updated package dependencies.

commit d4749b23316e120de0b52b845c792c554f57e03d
Author: Ravi Sharma <s2007.ravi@gmail.com>
Date:   Tue Apr 21 20:29:31 2020 +0530

    New launch files for Gazebo world.

commit b244e865fc79f8b686aa5d0f12364549487cf954
Author: Ravi Sharma <s2007.ravi@gmail.com>
Date:   Tue Apr 21 20:27:15 2020 +0530

    Optimized PID to keep arm intact.

commit 9bb74bd7eb55a1052a3d3d2b2e926f51e612cc56
Author: Ravi Sharma <s2007.ravi@gmail.com>
Date:   Tue Apr 21 00:20:30 2020 +0530

    Launch arm in Gazebo.

commit 8fe20d206e6edabd6861ed6c18ac8fec7c4e1c04
Author: Ravi Sharma <s2007.ravi@gmail.com>
Date:   Tue Apr 21 00:19:15 2020 +0530

    Renamed controller manager & moved control nodes to one file.

commit a691717cd933174e40165cb51f9e1c6f70498da7
Author: Ravi Sharma <s2007.ravi@gmail.com>
Date:   Tue Apr 21 00:17:20 2020 +0530

    Renamed joint state controller.

commit a1f2dd06d6f853f54095cd00b76ce266bab35e85
Author: Ravi Sharma <s2007.ravi@gmail.com>
Date:   Tue Apr 21 00:16:20 2020 +0530

    Added dependency.

commit 0b36d5990f626666ffd03d0025f33ed935de1409
Author: Ravi Sharma <s2007.ravi@gmail.com>
Date:   Tue Apr 21 00:15:21 2020 +0530

    Added base_link to the arm.

commit 7bfb9e15fcbf38cdc2266c4d0a6c3f999a6b2d03
Author: Ravi Sharma <s2007.ravi@gmail.com>
Date:   Tue Apr 21 00:12:41 2020 +0530

    Added TF to RViz config.

commit 8a49420d45d58d37484560b3630b0e534ccfb7cf
Author: Ravi Sharma <s2007.ravi@gmail.com>
Date:   Mon Apr 20 19:06:17 2020 +0530

    Arm's joint parameters.

commit 3bb9bc3a1e71e2a134e8cfc35af5ff16bbc37ae7
Author: Ravi Sharma <s2007.ravi@gmail.com>
Date:   Mon Apr 20 18:53:33 2020 +0530

    Package to control 5DOF arm in Gazebo.

commit 687007006633697ab0e6c5fa0fdb2af113301f25
Author: Ravi Sharma <s2007.ravi@gmail.com>
Date:   Mon Apr 20 18:34:46 2020 +0530

    Rover & Arm Gazebo control package.

commit 010389580f3bbe85c8df1dbd7b366c6eafde1f90
Author: Ravi Sharma <s2007.ravi@gmail.com>
Date:   Mon Apr 20 17:26:24 2020 +0530

    Rover+Arm description file.

commit a8559a2c4e634c7330d18bcaa1a69019d1762511
Author: Ravi Sharma <s2007.ravi@gmail.com>
Date:   Mon Apr 20 17:18:36 2020 +0530

    Changed RViz configuration.

commit d52e42f6e94c9f8dcaf7f688709d4a1f88185fca
Author: Ravi Sharma <s2007.ravi@gmail.com>
Date:   Mon Apr 20 17:18:07 2020 +0530

    Added higher level xacros.

commit 8ab186637d617b4fe621d4d705244ea705e68eba
Author: Ravi Sharma <s2007.ravi@gmail.com>
Date:   Mon Apr 20 17:14:35 2020 +0530

    Converted Rover & Arm descriptions to macros.

commit 379f1ba092d1d0eb3032247e8e664ca7d108a81c
Author: Ravi Sharma <s2007.ravi@gmail.com>
Date:   Sun Apr 19 23:04:30 2020 +0530

    Experimenting to launch rover and arm together.

commit 830882fc03f4bc65a1d444d8b69e90d17605ecd0
Author: Ravi Sharma <s2007.ravi@gmail.com>
Date:   Sun Apr 19 23:03:27 2020 +0530

    Createdd RViz configuration.

commit 4b954160c82be4017fb05725dcfbc17b5b408d5a
Author: Ravi Sharma <s2007.ravi@gmail.com>
Date:   Sun Apr 19 23:02:49 2020 +0530

    Created launch files.

commit ccd0a78875e0becf78733cff81c288ccea26177b
Author: Ravi Sharma <s2007.ravi@gmail.com>
Date:   Sun Apr 19 23:02:08 2020 +0530

    Corrected the comments.

commit 3361b9adca130796be1113c850a03ab9a6f04a80
Author: Ravi Sharma <s2007.ravi@gmail.com>
Date:   Sun Apr 19 21:42:39 2020 +0530

    New xacro to stitch arm with rover.

commit 7f6f55211e8848ae971ff27db8af31ca00e0b2bb
Author: Ravi Sharma <s2007.ravi@gmail.com>
Date:   Sun Apr 19 21:39:29 2020 +0530

    New package to spawn rover with arm.

commit 876c33da73b008ee5800b23492aed2f9327f72f6
Author: Ravi Sharma <s2007.ravi@gmail.com>
Date:   Thu Apr 16 13:59:52 2020 +0530

    Changed type to mesh.

commit 37b71f3ee73f2732a653193ae026c98a4bff6a11
Author: Ravi Sharma <s2007.ravi@gmail.com>
Date:   Thu Apr 16 13:59:19 2020 +0530

    Removed dynamics and changes to box shape mesh.

commit 1be47fb1c919f79416fccc637fc5080253c3ffec
Author: Ravi Sharma <s2007.ravi@gmail.com>
Date:   Thu Apr 16 13:57:29 2020 +0530

    Removed cylinder inertia.

commit db0b0e9ebb925f33f528852f41bfdc0381d7c43d
Author: Ravi Sharma <s2007.ravi@gmail.com>
Date:   Thu Apr 16 13:55:56 2020 +0530

    Removed dynamics from revolute joint description.
    Separated mesh description for box and cylinder shapes.

commit eadec733779e98afa9cf4d9d820ec01ffc0e2b42
Author: Ravi Sharma <s2007.ravi@gmail.com>
Date:   Thu Apr 16 13:54:49 2020 +0530

    Changed mesh description.

commit a0d0ebb6e368673c881b35d271d71cc5a9253d40
Author: Ravi Sharma <s2007.ravi@gmail.com>
Date:   Thu Apr 16 13:48:19 2020 +0530

    Changed display settings.

commit 9ae068e28d3a3f2f94323426b54ab82928c2f96f
Author: Ravi Sharma <s2007.ravi@gmail.com>
Date:   Wed Apr 15 22:01:05 2020 +0530

    Included shape and size parameters.

commit 95185ffa5276e77f9118905b7b0f01df3eb4e002
Author: Ravi Sharma <s2007.ravi@gmail.com>
Date:   Wed Apr 15 22:00:11 2020 +0530

    Included shape, size parameters and dynamics.

commit edcf46eae41c16b1b07c5da1b85cd1a0f8f50de1
Author: Ravi Sharma <s2007.ravi@gmail.com>
Date:   Wed Apr 15 21:58:46 2020 +0530

    Changed size parameters for chassis footprint.
    Included shape and size parameters in chassis link.

commit f6e7be4b3de91efb12c6f7527eaf457895f4792d
Author: Ravi Sharma <s2007.ravi@gmail.com>
Date:   Wed Apr 15 21:57:54 2020 +0530

    Changed mass values.

commit 8b30af8ea8679a2f3a376afe6a99f1988cacc944
Author: Ravi Sharma <s2007.ravi@gmail.com>
Date:   Wed Apr 15 21:57:16 2020 +0530

    Seperated inertial based on shape in mesh link.

commit bba2860f417bedb438c6b46e31bda027c61c0de7
Author: Ravi Sharma <s2007.ravi@gmail.com>
Date:   Wed Apr 15 21:56:03 2020 +0530

    Included shape in mesh links.

commit 1ca863ac986e892a006a3b5e4983e26ffdd55a1d
Author: Ravi Sharma <s2007.ravi@gmail.com>
Date:   Wed Apr 15 21:12:30 2020 +0530

    Customized macros for inbuilt inertial.
    Removed color from mesh macro.

commit d8fc1d8b6f3734905e2240f0328297265dfb851a
Author: Ravi Sharma <s2007.ravi@gmail.com>
Date:   Wed Apr 15 21:11:29 2020 +0530

    Completed rover arm description.

commit a8b6454bcff0663b164b79119ac9b1839cecf49b
Author: Ravi Sharma <s2007.ravi@gmail.com>
Date:   Wed Apr 15 21:10:40 2020 +0530

    More arm parameters.

commit 4470a6a09aa3aa0e52c32af86d8f94a353ba2e4f
Author: Ravi Sharma <s2007.ravi@gmail.com>
Date:   Wed Apr 15 21:09:57 2020 +0530

    Customized as per different link types.

commit fb1cb9a3a1e753bec798885c68331a4922930c04
Author: Ravi Sharma <s2007.ravi@gmail.com>
Date:   Wed Apr 15 21:08:15 2020 +0530

    Rover arm links meshes.

commit 166c4f12b8ec0f6f53c6cc11f97677df25503e72
Author: Ravi Sharma <s2007.ravi@gmail.com>
Date:   Mon Apr 13 22:48:22 2020 +0530

    Continuation of arm description.

commit 09b7fc2601d1c3020cec2ab87e317076c009586c
Author: Ravi Sharma <s2007.ravi@gmail.com>
Date:   Mon Apr 13 22:47:14 2020 +0530

    Added dynamics parameters.

commit 94f92bd1e7c9333e199b4bb7593ce05412b655c9
Author: Ravi Sharma <s2007.ravi@gmail.com>
Date:   Mon Apr 13 22:46:31 2020 +0530

    Removed joint_state_publisher as it got duplicated.

commit 84fa293e9d86e8d6983dfdae01f05207f47d4af7
Author: Ravi Sharma <s2007.ravi@gmail.com>
Date:   Mon Apr 13 22:44:46 2020 +0530

    Arm links definitions.

commit a8f08e4fba38c61c499d2cdaf1a04a54e4175666
Author: Ravi Sharma <s2007.ravi@gmail.com>
Date:   Sun Apr 12 23:03:27 2020 +0530

    RViz configuration file.

commit 4cf059ab083128b4099bc783a9792c1c61b54e42
Author: Ravi Sharma <s2007.ravi@gmail.com>
Date:   Sun Apr 12 23:02:57 2020 +0530

    Created RViz launch files

commit b15c8ff172da76ca08a95742110d67376a25d949
Author: Ravi Sharma <s2007.ravi@gmail.com>
Date:   Sun Apr 12 23:02:00 2020 +0530

    Created the first cylindrical link.

commit 13048ec498212d47fb281a96b68869f708bbdfd0
Author: Ravi Sharma <s2007.ravi@gmail.com>
Date:   Sun Apr 12 22:26:55 2020 +0530

    Created arm_parameters and rover_arm description.

commit f61cd0e799783e93afd14f03bdcf896a3087b612
Author: Ravi Sharma <s2007.ravi@gmail.com>
Date:   Sun Apr 12 22:00:01 2020 +0530

    Renamed robot_parameters to rover_parameters.

commit 112f24620c31c9cf3653f66a885347dc4e6a058b
Author: Ravi Sharma <s2007.ravi@gmail.com>
Date:   Sun Apr 12 20:49:26 2020 +0530

    New package to describe Rover Arm.

commit 140d2c6419f3e0eaae17f6e149c89aed9d96c084
Author: Ravi Sharma <s2007.ravi@gmail.com>
Date:   Fri Apr 10 17:17:36 2020 +0530

    Fixed various bugs to publish velocity in steps.

commit b441359d74a481011ccd3ac4eb7844799d3f63e0
Author: Ravi Sharma <s2007.ravi@gmail.com>
Date:   Fri Apr 10 17:16:26 2020 +0530

    Changed subscribing topic to listen rover_teleop node.

commit 8918cd764dff08ac53089f6190ea8a5e86b13cbe
Author: Ravi Sharma <s2007.ravi@gmail.com>
Date:   Fri Apr 10 17:14:38 2020 +0530

    Added rover_teleop node and resepective parameters.

commit dd605ebb7f17249caa3dd37c17d7565d8fc115c4
Author: Ravi Sharma <s2007.ravi@gmail.com>
Date:   Fri Apr 10 12:11:32 2020 +0530

    New node to teleop the rover.

commit c2cfe02dbf6d9c2dfae874f8c6bb829b47bd7061
Author: Ravi Sharma <s2007.ravi@gmail.com>
Date:   Thu Apr 9 17:48:32 2020 +0530

    Switch to AckermannDrive.

commit 74f94e29b5a4a2441afeda87ae53ce90b91eeabd
Author: Ravi Sharma <s2007.ravi@gmail.com>
Date:   Thu Apr 9 17:46:21 2020 +0530

    Revert back to AckermannDrive message.
    Corrected type of theta_left and theta_right.
    Removed loginfo.

commit 9cf9fd82d02c34c7177589784900b0d055901615
Author: Ravi Sharma <s2007.ravi@gmail.com>
Date:   Thu Apr 9 17:44:46 2020 +0530

    Speed and turn limits to teleop.

commit 9c0e62abf6ea628cd08f260f04c2dedcd395f945
Author: Ravi Sharma <s2007.ravi@gmail.com>
Date:   Thu Apr 9 15:08:08 2020 +0530

    Added publish frequency as an argument.

commit 6b17ae4127d5d79723a5943cb111ae799430aa53
Author: Ravi Sharma <s2007.ravi@gmail.com>
Date:   Thu Apr 9 15:06:10 2020 +0530

    Corrected publisher topic (included namespace).
    Fetch correct value of wheelbase.

commit aaae8036d4a66cc0d2b7e98ecb47202b6623108f
Author: Ravi Sharma <s2007.ravi@gmail.com>
Date:   Thu Apr 9 15:03:04 2020 +0530

    Graceful shutdown of the node.
    Changed Ackermann message type.
    Added more logging statements.

commit 1488d799e87b38ed143a2488062076899bc0cee3
Author: Ravi Sharma <s2007.ravi@gmail.com>
Date:   Thu Apr 9 15:01:00 2020 +0530

    Delayed launch of cmd_vel_to_ackermann_drive to properly fetch
    wheelbase.

commit 58ae40bba0b25606f2d7a902b85b0a365ef92d88
Author: Ravi Sharma <s2007.ravi@gmail.com>
Date:   Thu Apr 9 12:04:08 2020 +0530

    Created new launch file to control rover using keyboard.

commit 98a2b4794e0f267a326bb21dc48906cc03118a9a
Author: Ravi Sharma <s2007.ravi@gmail.com>
Date:   Wed Apr 8 17:50:01 2020 +0530

    New node to convert cmd_vel to ackermann_drive.

commit b576f1d2089a0e92451e90961c63ef85d0950ade
Author: Ravi Sharma <s2007.ravi@gmail.com>
Date:   Wed Apr 8 17:49:22 2020 +0530

    Updated package dependencies.

commit 79ca36ecb04591a9c5bd67907d8749d96577fa82
Author: Ravi Sharma <s2007.ravi@gmail.com>
Date:   Tue Apr 7 12:14:24 2020 +0530

    Fine-tuned PID parameters.

commit aa84c1a27ec282f12b69740a847d73f6635b2cbb
Author: Ravi Sharma <s2007.ravi@gmail.com>
Date:   Tue Apr 7 12:12:40 2020 +0530

    Changed velocity limit.
    Removed friction parameters.

commit bde3de8e277f4bb443468cc83353d601cdc41d55
Author: Ravi Sharma <s2007.ravi@gmail.com>
Date:   Tue Apr 7 11:51:14 2020 +0530

    Steering limits=+-75 deg.

commit 745fc0d255266a2ffddca73b35690cbdad11333a
Author: Ravi Sharma <s2007.ravi@gmail.com>
Date:   Mon Apr 6 23:25:56 2020 +0530

    Debug the code for various errors.

commit 8904b84ae1ebb26fdeaab0e4764641e424552c99
Author: Ravi Sharma <s2007.ravi@gmail.com>
Date:   Mon Apr 6 23:23:50 2020 +0530

    Enabled use_sim_time.
    Renamed controller_spawner node.
    Enabled rover_controller node.

commit 40b3904d3749166378b5b5c55d7d66d432ad99cc
Author: Ravi Sharma <s2007.ravi@gmail.com>
Date:   Mon Apr 6 23:22:50 2020 +0530

    Rearranged parameters.

commit 6f970abb69f33819a3fd401d9eb3fcc527a7d48a
Author: Ravi Sharma <s2007.ravi@gmail.com>
Date:   Mon Apr 6 09:53:28 2020 +0530

    New rover_controller node.

commit 3706afd8b58044899995b717c8604d2ebdfeb91e
Author: Ravi Sharma <s2007.ravi@gmail.com>
Date:   Mon Apr 6 09:38:36 2020 +0530

    Set use_sim_time to false & enabled rover_controller node.

commit 902f8f3fcfeab37d1d690116b70d97e2489da684
Author: Ravi Sharma <s2007.ravi@gmail.com>

File: rover_desc_pkg/urdf/steer.xacro (robot description, xacro)
@@ -2,6 +2,7 @@
 <robot name="steer" xmlns:xacro="http://www.ros.org/wiki/xacro">
   <!-- Begin - Include -->
-  <xacro:include filename="$(find rover_desc_pkg)/urdf/robot_parameters.xacro"/>
-  <xacro:include filename="$(find rover_desc_pkg)/urdf/links_joints.xacro"/>
+  <xacro:include filename="$(find rover_desc_pkg)/urdf/rover_parameters.xacro"/>
+  <xacro:include filename="$(find rover_arm_resources_pkg)/urdf/links_joints.xacro"/>
+  <xacro:include filename="$(find rover_arm_resources_pkg)/urdf/common_constants.xacro"/>
   <!-- End - Include -->
   <xacro:macro name="steer" params="fr lr parent type translateX translateY"> <!-- fr: front, rear; lr: left, right -->
@@ -10,8 +11,7 @@
     <xacro:property name="steer_y" value="${translateY * world_y_origin_to_steer_y_origin}" scope="local"/>
     <xacro:property name="steer_z" value="${wheel_radius + steer_z_origin_to_wheel_z_origin}" scope="local"/>
-    <xacro:if value="${fr == 'rear'}">
+    <xacro:if value="${fr == 'front'}">
       <xacro:property name="steer_x"
-                      value="${translateX * (world_x_origin_to_steer_x_origin + 0.063)}"
-                      scope="local"/>
+                      value="${translateX * (world_x_origin_to_steer_x_origin + 0.063)}" scope="local"/>
     </xacro:if>
     <!-- Decide steer mesh file based on its location -->
@@ -19,6 +19,5 @@
       <xacro:property name="mesh_file" value="package://rover_desc_pkg/meshes/rover_steer_r.dae"/>
       <xacro:property name="steer_z"
-                      value="${wheel_radius + steer_z_origin_to_wheel_z_origin + 0.0032}"
-                      scope="local"/>
+                      value="${wheel_radius + steer_z_origin_to_wheel_z_origin + 0.0032}" scope="local"/>
     </xacro:if>
     <xacro:if value="${lr == 'left'}">
@@ -29,14 +28,13 @@
     </xacro:if>
     <!-- Link description -->
-    <m_link_mesh name="${fr}_${lr}_steer"
-                 color="${Red_Value}"
-                 origin_rpy="0 0 0"
-                 origin_xyz="0 0 0"
-                 mass="1.0"
-                 ixx="0.0001" ixy="0.0" ixz="0.0"
-                 iyy="0.0001" iyz="0.0"
-                 izz="0.0001"
-                 meshfile="${mesh_file}"
-                 meshscale="1 1 1"/>
+    <xacro:m_link_mesh_box name="${fr}_${lr}_steer"
+                           origin_rpy="0 0 0"
+                           origin_xyz="0 0 0"
+                           m="${steer_mass}"
+                           w="${steer_width}"
+                           d="${steer_length}"
+                           h="${steer_height}"
+                           meshfile="${mesh_file}"
+                           meshscale="1 1 1"/>
     <gazebo reference="${fr}_${lr}_steer">
       <material>Gazebo/Grey</material>
@@ -45,24 +43,18 @@
     <!-- Joint description -->
     <xacro:if value="${type == 'fixed'}">
-      <m_joint_fixed name="${parent}__${fr}_${lr}_steer"
-                     origin_rpy="0 0 0" origin_xyz="${steer_x} ${steer_y} ${steer_z}"
-                     parent="${parent}" child="${fr}_${lr}_steer"/>
+      <xacro:m_joint_fixed name="${parent}__${fr}_${lr}_steer"
+                           origin_rpy="0 0 0" origin_xyz="${steer_x} ${steer_y} ${steer_z}"
+                           parent="${parent}" child="${fr}_${lr}_steer"/>
     </xacro:if>
     <xacro:if value="${type == 'revolute'}">
-      <m_joint_rev name="${parent}__${fr}_${lr}_steer"
-                   axis_xyz="0 0 1"
-                   origin_rpy="0 0 0" origin_xyz="${steer_x} ${steer_y} ${steer_z}"
-                   parent="${parent}" child="${fr}_${lr}_steer"
-                   limit_e="100" limit_l="-${M_PI/2}" limit_u="${M_PI/2}" limit_v="100"/>
+      <xacro:m_joint_rev name="${parent}__${fr}_${lr}_steer"
+                         axis_xyz="0 0 1"
+                         axis_rpy="0 0 0"
+                         origin_rpy="0 0 0" origin_xyz="${steer_x} ${steer_y} ${steer_z}"
+                         parent="${parent}" child="${fr}_${lr}_steer"
+                         limit_e="1000" limit_l="-${5*M_PI/12}"
+                         limit_u="${5*M_PI/12}" limit_v="100"
+                         damp="25.0" fric="10.0"/>
     </xacro:if>
-    <!-- Transmission is important to link the joints and the controller -->
-    <!-- <transmission name="${fr}_${lr}_steer_joint_trans">
-      <type>transmission_interface/SimpleTransmission</type>
-      <joint name="${fr}_${lr}_steer_joint"/>
-      <actuator name="${fr}_${lr}_steer_joint_motor">
-          <hardwareInterface>EffortJointInterface</hardwareInterface>
-          <mechanicalReduction>1</mechanicalReduction>
-      </actuator>
-    </transmission> -->
   </xacro:macro>
 </robot>
