Commit message: Changed mass values.

File: rover_desc_pkg/urdf/rover_parameters.xacro (robot description, xacro)
@@ -51,5 +51,5 @@
   <xacro:property name="chassis_width" value="0.6096"/>
   <xacro:property name="chassis_height" value="0.4445"/>
-  <xacro:property name="chassis_mass" value="5"/> <!-- in Kg -->
+  <xacro:property name="chassis_mass" value="1.0"/> <!-- in Kg -->
   <xacro:property name="world_x_origin_to_chassis_x_origin" value="0.0"/>
   <xacro:property name="world_y_origin_to_chassis_y_origin" value="0.0"/>
@@ -64,5 +64,5 @@
   <xacro:property name="steer_width" value="0.234"/>
   <xacro:property name="steer_height" value="0.618"/>
-  <xacro:property name="steer_mass" value="5"/> <!-- in Kg -->
+  <xacro:property name="steer_mass" value="1.0"/> <!-- in Kg -->
   <xacro:property name="world_x_origin_to_steer_x_origin" value="0.3715"/> <!-- Distance from world origin to mount point in X direction -->
   <xacro:property name="world_y_origin_to_steer_y_origin" value="0.3148"/> <!-- Distance from world origin to mount point in Y direction -->

Commit message: Removed cylinder inertia.

File: rover_desc_pkg/urdf/rover_parameters.xacro (robot description, xacro)
@@ -79,8 +79,3 @@
   <xacro:property name="steer_y_origin_to_wheel_y_origin" value="0.0"/>
   <xacro:property name="steer_z_origin_to_wheel_z_origin" value="0.4620"/>
-  <xacro:macro name="cylinder_inertia" params="m r h">
-    <intertia ixx="${m*(3*r*r+h*h)/12}" ixy="0.0" ixz="0.0"
-              iyy="${m*(3*r*r+h*h)/12}" iyz="0.0"
-              izz="${m*r*r/2}"/>
-  </xacro:macro>
 </robot>

Commit message: Updated the definitions according to new package.

File: rover_desc_pkg/urdf/rover_parameters.xacro (robot description, xacro)
@@ -3,48 +3,4 @@
   <xacro:property name="r_link_00_name" value="chassis_footprint"/>
   <xacro:property name="r_link_01_name" value="chassis_link"/>
-  <!-- Color parameters -->
-  <xacro:macro name="red">
-    <material name="">
-      <color rgba="${204/255} ${0.0/255} ${0.0/255} ${255/255}"/>
-    </material>
-  </xacro:macro>
-  <xacro:macro name="green">
-    <material name="">
-      <color rgba="${0.0/255} ${204/255} ${0.0/255} ${255/255}"/>
-    </material>
-  </xacro:macro>
-  <xacro:macro name="blue">
-    <material name="">
-      <color rgba="${0.0/255} ${0.0/255} ${204/255} ${255/255}"/>
-    </material>
-  </xacro:macro>
-  <xacro:macro name="black">
-    <material name="">
-      <color rgba="${0.0/255} ${0.0/255} ${0.0/255} ${255/255}"/>
-    </material>
-  </xacro:macro>
-  <xacro:macro name="white">
-    <material name="">
-      <color rgba="${255/255} ${255/255} ${255/255} ${255/255}"/>
-    </material>
-  </xacro:macro>
-  <xacro:macro name="gray">
-    <material name="">
-      <color rgba="${178.5/255} ${178.5/255} ${178.5/255} ${255/255}"/>
-    </material>
-  </xacro:macro>
-  <xacro:macro name="darkgray">
-    <material name="">
-      <color rgba="${76.5/255} ${76.5/255} ${76.5/255} ${255/255}"/>
-    </material>
-  </xacro:macro>
-  <xacro:macro name="yellow">
-    <material name="">
-      <color rgba="${204/255} ${204/255} ${204/255} ${255/255}"/>
-    </material>
-  </xacro:macro>
-  <!-- All the units are in m-kg-s-radians unit system -->
-  <xacro:property name="M_PI" value="3.141592653"/>
-  <xacro:property name="DEG_TO_RAD" value="0.017453293"/>
   <!-- Chassis dimensions -->
   <xacro:property name="chassis_length" value="1.016"/>

File: rover_desc_pkg/urdf/rover_robot_macro.xacro (robot description, xacro)
@@ -2,6 +2,6 @@
 <robot name="rover_robot" xmlns:xacro="http://www.ros.org/wiki/xacro">
   <!-- Begin - Include -->
+  <xacro:include filename="$(find rover_arm_resources_pkg)/urdf/links_joints.xacro"/>
   <xacro:include filename="$(find rover_desc_pkg)/urdf/rover_parameters.xacro"/>
-  <xacro:include filename="$(find rover_desc_pkg)/urdf/links_joints.xacro"/>
   <xacro:include filename="$(find rover_desc_pkg)/urdf/steer.xacro"/>
   <xacro:include filename="$(find rover_desc_pkg)/urdf/wheel.xacro"/>
@@ -12,5 +12,4 @@
     <!-- Chassis footprint -->
     <xacro:m_link_box name="${r_link_00_name}"
-                      color="white"
                       origin_rpy="0 0 0" origin_xyz="0 0 0"
                       w="0.0001" d="0.0001" h="0.0001"/>

File: rover_desc_pkg/urdf/steer.xacro (robot description, xacro)
@@ -3,5 +3,6 @@
   <!-- Begin - Include -->
   <xacro:include filename="$(find rover_desc_pkg)/urdf/rover_parameters.xacro"/>
-  <xacro:include filename="$(find rover_desc_pkg)/urdf/links_joints.xacro"/>
+  <xacro:include filename="$(find rover_arm_resources_pkg)/urdf/links_joints.xacro"/>
+  <xacro:include filename="$(find rover_arm_resources_pkg)/urdf/common_constants.xacro"/>
   <!-- End - Include -->
   <xacro:macro name="steer" params="fr lr parent type translateX translateY"> <!-- fr: front, rear; lr: left, right -->

File: rover_desc_pkg/urdf/wheel.xacro (robot description, xacro)
@@ -3,5 +3,6 @@
   <!-- Begin - Include -->
   <xacro:include filename="$(find rover_desc_pkg)/urdf/rover_parameters.xacro"/>
-  <xacro:include filename="$(find rover_desc_pkg)/urdf/links_joints.xacro"/>
+  <xacro:include filename="$(find rover_arm_resources_pkg)/urdf/links_joints.xacro"/>
+  <xacro:include filename="$(find rover_arm_resources_pkg)/urdf/common_constants.xacro"/>
   <!-- End - Include -->
   <xacro:macro name="wheel" params="fr lr parent translateX translateY"> <!-- fr: front, rear; lr: left, right -->

Commit message: New chassis model: corrected necessary params.

File: rover_desc_pkg/urdf/rover_parameters.xacro (robot description, xacro)
@@ -4,16 +4,11 @@
   <xacro:property name="r_link_01_name" value="chassis_link"/>
   <!-- Chassis dimensions -->
-  <xacro:property name="chassis_length" value="1.016"/>
-  <xacro:property name="chassis_width" value="0.6096"/>
-  <xacro:property name="chassis_height" value="0.4445"/>
+  <xacro:property name="chassis_length" value="1.2500"/>
+  <xacro:property name="chassis_width" value="1.0012"/>
+  <xacro:property name="chassis_height" value="0.1651"/>
   <xacro:property name="chassis_mass" value="1.0"/> <!-- in Kg -->
   <xacro:property name="world_x_origin_to_chassis_x_origin" value="0.0"/>
   <xacro:property name="world_y_origin_to_chassis_y_origin" value="0.0"/>
   <xacro:property name="world_z_origin_to_chassis_z_origin" value="0.0"/>
-  <!-- Inverter dimensions -->
-  <xacro:property name="inverter_length" value="0.400"/>
-  <xacro:property name="inverter_width" value="0.2353"/>
-  <xacro:property name="inverter_height" value="0.400"/>
-  <xacro:property name="inverter_mass" value="5"/> <!-- in Kg -->
   <!-- Steer dimensions -->
   <xacro:property name="steer_length" value="0.217"/>
@@ -21,8 +16,8 @@
   <xacro:property name="steer_height" value="0.618"/>
   <xacro:property name="steer_mass" value="1.0"/> <!-- in Kg -->
-  <xacro:property name="world_x_origin_to_steer_x_origin" value="0.3715"/> <!-- Distance from world origin to mount point in X direction -->
-  <xacro:property name="world_y_origin_to_steer_y_origin" value="0.3148"/> <!-- Distance from world origin to mount point in Y direction -->
+  <xacro:property name="world_x_origin_to_steer_x_origin" value="0.45675"/> <!-- Distance from world origin to mount point in X direction -->
+  <xacro:property name="world_y_origin_to_steer_y_origin" value="${chassis_width/2 + 0.017}"/> <!-- Distance from world origin to mount point in Y direction -->
   <xacro:property name="world_z_origin_to_steer_z_origin" value="0.0"/> <!-- Distance from world origin to mount point in Z direction -->
-  <xacro:property name="chassis_z_origin_to_steer_z_origin" value="0.1305"/>
+  <xacro:property name="chassis_z_origin_to_steer_z_origin" value="${chassis_height/2 - 0.00928}"/>
   <!-- Wheels -->
   <xacro:property name="wheel_radius" value="0.178"/>

File: rover_desc_pkg/urdf/steer.xacro (robot description, xacro)
@@ -13,5 +13,5 @@
     <xacro:if value="${fr == 'front'}">
       <xacro:property name="steer_x"
-                      value="${translateX * (world_x_origin_to_steer_x_origin + 0.063)}" scope="local"/>
+                      value="${translateX * (world_x_origin_to_steer_x_origin + 0.07913)}" scope="local"/>
     </xacro:if>
     <!-- Decide steer mesh file based on its location -->

Commit message: update masses

File: rover_desc_pkg/urdf/rover_parameters.xacro (robot description, xacro)
@@ -7,5 +7,5 @@
   <xacro:property name="chassis_width" value="1.0012"/>
   <xacro:property name="chassis_height" value="0.1651"/>
-  <xacro:property name="chassis_mass" value="1.0"/> <!-- in Kg -->
+  <xacro:property name="chassis_mass" value="40.0"/> <!-- in Kg -->
   <xacro:property name="world_x_origin_to_chassis_x_origin" value="0.0"/>
   <xacro:property name="world_y_origin_to_chassis_y_origin" value="0.0"/>
@@ -15,5 +15,5 @@
   <xacro:property name="steer_width" value="0.234"/>
   <xacro:property name="steer_height" value="0.618"/>
-  <xacro:property name="steer_mass" value="1.0"/> <!-- in Kg -->
+  <xacro:property name="steer_mass" value="4.0"/> <!-- in Kg -->
   <xacro:property name="world_x_origin_to_steer_x_origin" value="0.45675"/> <!-- Distance from world origin to mount point in X direction -->
   <xacro:property name="world_y_origin_to_steer_y_origin" value="${chassis_width/2 + 0.017}"/> <!-- Distance from world origin to mount point in Y direction -->
@@ -23,5 +23,5 @@
   <xacro:property name="wheel_radius" value="0.178"/>
   <xacro:property name="wheel_height" value="0.114"/>
-  <xacro:property name="wheel_mass" value="1.0"/> <!-- in Kg -->
+  <xacro:property name="wheel_mass" value="3.0"/> <!-- in Kg -->
   <xacro:property name="world_x_origin_to_wheel_x_origin" value="0.4025"/>
   <xacro:property name="world_y_origin_to_wheel_y_origin" value="0.3153"/>
