Commit message: Experimenting to launch rover and arm together.

File: rover_with_arm_desc_pkg/urdf/rover_with_arm.xacro (robot description, xacro)
@@ -5,5 +5,10 @@
   <xacro:include filename="$(find rover_arm_desc_pkg)/urdf/rover_arm.xacro"/>
   <!-- End - Include -->
-  <link name="world"/>
+  <!-- <link name="world">
+    <origin xyz="0 0 0" rpy="0 0 0"/>
+    <geometry>
+      <box size="0.0001 0.0001 0.0001" />
+    </geometry>
+  </link>
   <joint name="world_chassis_joint" type="fixed">
       <parent link="world"/>
@@ -15,4 +20,11 @@
       <child link="arm_footprint"/>
       <origin xyz="0.0 0.0 0..0" rpy="0.0 0.0 0.0"/>
-  </joint>
+  </joint> -->
+  <!-- Using the models -->
+  <xacro:rover_robot name="rover">
+    <origin xyz="0.0 0.0 0..0" rpy="0.0 0.0 0.0"/>
+  </xacro:rover_robot>
+  <xacro:rover_arm name="arm">
+    <origin xyz="0.0 0.0 0..0" rpy="0.0 0.0 0.0"/>
+  </xacro:rover_arm>
 </robot>

Commit message: Rover+Arm description file.

File: rover_with_arm_desc_pkg/urdf/rover_with_arm.xacro (robot description, xacro)
@@ -1,30 +1,19 @@
 <?xml version="1.0"?>
 <robot name="rover_with_arm" xmlns:xacro="http://www.ros.org/wiki/xacro">
-  <!-- Begin - Include -->
-  <xacro:include filename="$(find rover_desc_pkg)/urdf/rover_robot.xacro"/>
-  <xacro:include filename="$(find rover_arm_desc_pkg)/urdf/rover_arm.xacro"/>
+  <!-- Begin - Include macros of rover and the arm -->
+  <xacro:include filename="$(find rover_desc_pkg)/urdf/rover_robot_macro.xacro"/>
+  <xacro:include filename="$(find rover_arm_desc_pkg)/urdf/rover_arm_macro.xacro"/>
   <!-- End - Include -->
-  <!-- <link name="world">
-    <origin xyz="0 0 0" rpy="0 0 0"/>
-    <geometry>
-      <box size="0.0001 0.0001 0.0001" />
-    </geometry>
-  </link>
-  <joint name="world_chassis_joint" type="fixed">
-      <parent link="world"/>
-      <child link = "chassis_footprint"/>
-      <origin xyz="0.0 0.0 0.0" rpy="0.0 0.0 0.0"/>
+  <!-- Create the rover + arm combo itself as a macro -->
+  <!-- Instantiate rover and arm models -->
+  <xacro:rover_robot/>
+  <xacro:rover_arm/>
+  <!-- Attach the arm to the rover -->
+  <!-- Note: This assumes that the 'arm' macro defines a 'footprint'
+     link which is the start of it's kinemtic chain (if any)-->
+  <joint name="chassis_footprint__arm_footprint_joint" type="fixed">
+    <origin xyz="0 0 0" rpy="0 0 0" />
+    <parent link="chassis_footprint" />
+    <child link="arm_footprint" />
   </joint>
-  <joint name="chassis_arm_joint" type="fixed">
-      <parent link="chassis_footprint"/>
-      <child link="arm_footprint"/>
-      <origin xyz="0.0 0.0 0..0" rpy="0.0 0.0 0.0"/>
-  </joint> -->
-  <!-- Using the models -->
-  <xacro:rover_robot name="rover">
-    <origin xyz="0.0 0.0 0..0" rpy="0.0 0.0 0.0"/>
-  </xacro:rover_robot>
-  <xacro:rover_arm name="arm">
-    <origin xyz="0.0 0.0 0..0" rpy="0.0 0.0 0.0"/>
-  </xacro:rover_arm>
 </robot>
