Commit message: Customized as per different link types.

File: rover_arm_desc_pkg/urdf/arm_links.xacro (robot description, xacro)
@@ -7,32 +7,52 @@
   <!-- End - Include -->
   <!-- Links -->
-  <xacro:macro name="arm_link" params="name parent length width height link_xyz link_rpy joint_xyz joint_rpy axis_xyz lim_l lim_u">
+  <xacro:macro name="arm_link" params="name type parent x_dim y_dim z_dim link_xyz link_rpy m file scale joint_xyz joint_rpy axis_xyz axis_rpy lim_l lim_u">
     <!-- Joint for link movement -->
     <xacro:m_joint_rev name="${parent}__${name}_joint"
-                       axis_xyz="${axis_xyz}"
+                       axis_rpy="${axis_rpy}" axis_xyz="${axis_xyz}"
                        origin_rpy="${joint_rpy}" origin_xyz="${joint_xyz}"
                        parent="${parent}" child="${name}"
                        limit_e="1000.0" limit_l="${lim_l}" limit_u="${lim_u}" limit_v="1"
                        dynamics_d="50" dynamics_f="1"/>
-    <!-- Link 01 -->
-    <xacro:m_link_cylinder name="${name}"
-                           color="darkgray"
-                           origin_rpy="${link_rpy}"
-                           origin_xyz="${link_xyz}"
-                           radius="0.05"
-                           length="0.06"
-                           mass="1.0"
-                           ixx="0.0001" ixy="0.0" ixz="0.0"
-                           iyy="0.0001" iyz="0.0"
-                           izz="0.0001"/>
+    <!-- Link -->
+    <xacro:if value="${type == 'cyl_iner'}">
+      <xacro:m_link_cylinder_inertia name="${name}"
+                                     color="darkgray"
+                                     origin_rpy="${link_rpy}"
+                                     origin_xyz="${link_xyz}"
+                                     r="${x_dim}"
+                                     l="${z_dim}"
+                                     m="${m}"/>
+    </xacro:if>
+    <xacro:if value="${type == 'box_iner'}">
+      <xacro:m_link_box_inertia name="${name}"
+                                color="darkgray"
+                                origin_rpy="${link_rpy}"
+                                origin_xyz="${link_xyz}"
+                                w="${x_dim}"
+                                d="${y_dim}"
+                                h="${z_dim}"
+                                m="${m}"/>
+    </xacro:if>
+    <xacro:if value="${type == 'mesh'}">
+      <xacro:m_link_mesh name="${name}"
+                         origin_rpy="${link_rpy}"
+                         origin_xyz="${link_xyz}"
+                         w="${x_dim}"
+                         d="${y_dim}"
+                         h="${z_dim}"
+                         m="${m}"
+                         meshfile="${file}"
+                         meshscale="${scale}"/>
+    </xacro:if>
     <gazebo reference="${name}">
-      <material>Gazebo/Gray</material>
+      <material>Gazebo/Silver</material>
     </gazebo>
     <!-- fixed joint -->
-    <xacro:m_joint_fixed name="${name}__${name}_box_joint"
+    <!--  <xacro:m_joint_fixed name="${name}__${name}_box_joint"
                          origin_rpy="0 0 0" origin_xyz="0 0 0"
-                         parent="${name}" child="${name}_box"/>
+                         parent="${name}" child="${name}_box"/> -->
     <!-- Link Arm -->
-    <xacro:m_link_box name="${name}_box"
+    <!-- <xacro:m_link_box name="${name}_box"
                       color="white"
                       origin_rpy="0 0 0" origin_xyz="${length/2 + 0.045} 0 0"
@@ -40,5 +60,5 @@
     <gazebo reference="${name}_box">
       <material>Gazebo/Silver</material>
-    </gazebo>
+    </gazebo> -->
   </xacro:macro>
 </robot>

Commit message: Removed dynamics and changes to box shape mesh.

File: rover_arm_desc_pkg/urdf/arm_links.xacro (robot description, xacro)
@@ -13,10 +13,9 @@
                        origin_rpy="${joint_rpy}" origin_xyz="${joint_xyz}"
                        parent="${parent}" child="${name}"
-                       limit_e="1000.0" limit_l="${lim_l}" limit_u="${lim_u}" limit_v="1"
-                       dynamics_d="50" dynamics_f="1"/>
+                       limit_e="1000.0" limit_l="${lim_l}" limit_u="${lim_u}" limit_v="1"/>
     <!-- Link -->
     <xacro:if value="${type == 'cyl_iner'}">
       <xacro:m_link_cylinder_inertia name="${name}"
-                                     color="darkgray"
+                                     color="blue"
                                      origin_rpy="${link_rpy}"
                                      origin_xyz="${link_xyz}"
@@ -27,5 +26,5 @@
     <xacro:if value="${type == 'box_iner'}">
       <xacro:m_link_box_inertia name="${name}"
-                                color="darkgray"
+                                color="blue"
                                 origin_rpy="${link_rpy}"
                                 origin_xyz="${link_xyz}"
@@ -36,30 +35,17 @@
     </xacro:if>
     <xacro:if value="${type == 'mesh'}">
-      <xacro:m_link_mesh name="${name}"
-                         shape="box"
-                         origin_rpy="${link_rpy}"
-                         origin_xyz="${link_xyz}"
-                         w="${x_dim}"
-                         d="${y_dim}"
-                         h="${z_dim}"
-                         m="${m}"
-                         meshfile="${file}"
-                         meshscale="${scale}"/>
+      <xacro:m_link_mesh_box name="${name}"
+                             origin_rpy="${link_rpy}"
+                             origin_xyz="${link_xyz}"
+                             w="${x_dim}"
+                             d="${y_dim}"
+                             h="${z_dim}"
+                             m="${m}"
+                             meshfile="${file}"
+                             meshscale="${scale}"/>
     </xacro:if>
     <gazebo reference="${name}">
       <material>Gazebo/Silver</material>
     </gazebo>
-    <!-- fixed joint -->
-    <!--  <xacro:m_joint_fixed name="${name}__${name}_box_joint"
-                         origin_rpy="0 0 0" origin_xyz="0 0 0"
-                         parent="${name}" child="${name}_box"/> -->
-    <!-- Link Arm -->
-    <!-- <xacro:m_link_box name="${name}_box"
-                      color="white"
-                      origin_rpy="0 0 0" origin_xyz="${length/2 + 0.045} 0 0"
-                      size="${length} ${width} ${height}"/>
-    <gazebo reference="${name}_box">
-      <material>Gazebo/Silver</material>
-    </gazebo> -->
   </xacro:macro>
 </robot>

Commit message: Changed joint limits.

File: rover_arm_desc_pkg/urdf/arm_links.xacro (robot description, xacro)
@@ -7,5 +7,7 @@
   <!-- End - Include -->
   <!-- Links -->
-  <xacro:macro name="arm_link" params="name type parent x_dim y_dim z_dim link_xyz link_rpy m file scale joint_xyz joint_rpy axis_xyz axis_rpy lim_l lim_u">
+  <xacro:macro name="arm_link" params="name type parent x_dim y_dim z_dim
+               link_xyz link_rpy m file scale joint_xyz joint_rpy axis_xyz
+               axis_rpy lim_l lim_u d f">
     <!-- Joint for link movement -->
     <xacro:m_joint_rev name="${parent}__${name}_joint"
@@ -13,5 +15,7 @@
                        origin_rpy="${joint_rpy}" origin_xyz="${joint_xyz}"
                        parent="${parent}" child="${name}"
-                       limit_e="1000.0" limit_l="${lim_l}" limit_u="${lim_u}" limit_v="1"/>
+                       limit_e="10000.0" limit_l="${lim_l}"
+                       limit_u="${lim_u}" limit_v="10"
+                       damp="${d}" fric="${f}"/>
     <!-- Link -->
     <xacro:if value="${type == 'cyl_iner'}">
@@ -45,4 +49,5 @@
     <gazebo reference="${name}">
       <material>Gazebo/Silver</material>
+      <!-- <turnGravityOff>false</turnGravityOff> -->
     </gazebo>
   </xacro:macro>

File: rover_desc_pkg/urdf/steer.xacro (robot description, xacro)
@@ -53,6 +53,7 @@
                          origin_rpy="0 0 0" origin_xyz="${steer_x} ${steer_y} ${steer_z}"
                          parent="${parent}" child="${fr}_${lr}_steer"
-                         limit_e="100" limit_l="-${5*M_PI/12}"
-                         limit_u="${5*M_PI/12}" limit_v="100"/>
+                         limit_e="1000" limit_l="-${5*M_PI/12}"
+                         limit_u="${5*M_PI/12}" limit_v="100"
+                         damp="25.0" fric="10.0"/>
     </xacro:if>
   </xacro:macro>

File: rover_desc_pkg/urdf/wheel.xacro (robot description, xacro)
@@ -37,5 +37,6 @@
                                     ${-steer_z_origin_to_wheel_z_origin}"
                         parent="${parent}" child="${fr}_${lr}_wheel"
-                        limit_e="100" limit_v="25"/>
+                        limit_e="1000" limit_v="25"
+                        damp="10.0" fric="1.0"/>
   </xacro:macro>
 </robot>
