Commit message: Added Damping and Friction.

File: rover_arm_desc_pkg/urdf/rover_arm_macro.xacro (robot description, xacro)
@@ -53,5 +53,7 @@
                     axis_rpy="0 0 0"
                     lim_l="-${M_PI/2}"
-                    lim_u="${M_PI/2}"/>
+                    lim_u="${30*M_PI/157}"
+                    d="2.0"
+                    f="1.0"/>
     <!-- Link 02 -->
     <xacro:arm_link name="${a_link_02_name}"
@@ -75,5 +77,7 @@
                     axis_rpy="0 0 0"
                     lim_l="-${M_PI/2}"
-                    lim_u="${M_PI/2}"/>
+                    lim_u="${M_PI/2}"
+                    d="0.1"
+                    f="0.1"/>
     <!-- Link 03 -->
     <xacro:arm_link name="${a_link_03_name}"
@@ -97,5 +101,7 @@
                     axis_rpy="0 0 0"
                     lim_l="${-125*M_PI/314}"
-                    lim_u="${25*M_PI/157}"/>
+                    lim_u="${25*M_PI/157}"
+                    d="1.50"
+                    f="0.75"/>
     <!-- Link 03a -->
     <xacro:arm_link name="${a_link_03a_name}"
@@ -119,5 +125,7 @@
                     axis_rpy="0 0 0"
                     lim_l="${-125*M_PI/314}"
-                    lim_u="${25*M_PI/157}"/>
+                    lim_u="${25*M_PI/157}"
+                    d="1.0"
+                    f="0.5"/>
     <!-- Link 04 -->
     <xacro:arm_link name="${a_link_04_name}"
@@ -141,5 +149,7 @@
                     axis_rpy="0 0 0"
                     lim_l="${-100*M_PI/157}"
-                    lim_u="${25*M_PI/157}"/>
+                    lim_u="${25*M_PI/157}"
+                    d="0.25"
+                    f="0.05"/>
     <!-- Arm -->
     <xacro:if value="${without_rover}">

File: rover_arm_resources_pkg/urdf/links_joints.xacro (robot description, xacro)
@@ -15,5 +15,6 @@
   </xacro:macro>
   <!-- continuous joint -->
-  <xacro:macro name="m_joint_cont" params="name axis_xyz origin_xyz origin_rpy parent child limit_e limit_v">
+  <xacro:macro name="m_joint_cont" params="name axis_xyz origin_xyz origin_rpy
+               parent child limit_e limit_v damp fric">
     <joint name="${name}" type="continuous">
       <axis xyz="${axis_xyz}"/>
@@ -22,4 +23,5 @@
       <parent link="${parent}"/>
       <child link="${child}"/>
+      <dynamics damping="${damp}" friction="${fric}"/>
     </joint>
     <transmission name="trans_${name}">
@@ -35,5 +37,7 @@
   </xacro:macro>
   <!-- revolute joint -->
-  <xacro:macro name="m_joint_rev" params="name axis_xyz axis_rpy origin_xyz origin_rpy parent child limit_e limit_l limit_u limit_v">
+  <xacro:macro name="m_joint_rev" params="name axis_xyz axis_rpy origin_xyz
+               origin_rpy parent child limit_e limit_l limit_u limit_v damp
+               fric">
     <joint name="${name}" type="revolute">
       <axis rpy="axis_rpy" xyz="${axis_xyz}"/>
@@ -42,4 +46,5 @@
       <parent link="${parent}"/>
       <child link="${child}"/>
+      <dynamics damping="${damp}" friction="${fric}"/>
     </joint>
     <transmission name="trans_${name}">
