Commit message: More arm parameters.

File: rover_arm_desc_pkg/urdf/arm_parameters.xacro (robot description, xacro)
@@ -5,23 +5,77 @@
   <xacro:property name="a_link_02_name" value="arm_link_02"/>
   <xacro:property name="a_link_03_name" value="arm_link_03"/>
+  <xacro:property name="a_link_03a_name" value="arm_link_03a"/>
   <xacro:property name="a_link_04_name" value="arm_link_04"/>
   <!-- All the units are in m-kg-s-radians unit system -->
   <xacro:property name="M_PI" value="3.141592653"/>
   <xacro:property name="DEG_TO_RAD" value="0.017453293"/>
+  <!-- Footprint dimensions -->
+  <xacro:property name="arm_foot_cyl_radius" value="0.02"/>
+  <xacro:property name="arm_foot_cyl_height" value="0.02"/>
+  <!-- Footprint position coordinates -->
+  <xacro:property name="world_x_origin_to_arm_x_origin" value="${chassis_length/2 + arm_foot_cyl_radius}"/> <!-- Distance from world origin to mount point in X direction -->
+  <xacro:property name="world_y_origin_to_arm_y_origin" value="-0.122"/> <!-- Distance from world origin to mount point in Y direction -->
+  <xacro:property name="world_z_origin_to_arm_z_origin" value="${0.562 - arm_foot_cyl_radius}"/> <!-- Distance from world origin to mount point in Z direction -->
+  <!-- Arm joints -->
+  <xacro:property name="arm_link_cyl_radius" value="0.05"/>
+  <xacro:property name="arm_link_cyl_height" value="0.06"/>
+  <xacro:property name="arm_link_cyl_mass" value="0.2"/> <!-- in Kg -->
   <!-- Arm Link 01 dimensions -->
-  <xacro:property name="arm_link_01_length" value="1.016"/>
-  <xacro:property name="arm_link_01_width" value="0.6096"/>
-  <xacro:property name="arm_link_01_mass" value="5"/> <!-- in Kg -->
+  <xacro:property name="arm_link01_x" value="0.080"/>
+  <xacro:property name="arm_link01_y" value="0.125"/>
+  <xacro:property name="arm_link01_z" value="0.400"/>
+  <xacro:property name="arm_link01_m" value="0.2"/> <!-- in Kg -->
+  <!-- Arm Link 01 translations -->
+  <xacro:property name="arm_link01_x_trans" value="0.0000"/>
+  <xacro:property name="arm_link01_y_trans" value="0.1050"/>
+  <xacro:property name="arm_link01_z_trans" value="0.0000"/>
   <!-- Arm Link 02 dimensions -->
-  <xacro:property name="arm_link_02_length" value="1.016"/>
-  <xacro:property name="arm_link_02_width" value="0.6096"/>
-  <xacro:property name="arm_link_02_mass" value="5"/> <!-- in Kg -->
+  <xacro:property name="arm_link02_x" value="0.0384"/>
+  <xacro:property name="arm_link02_y" value="0.0340"/>
+  <xacro:property name="arm_link02_z" value="0.0485"/>
+  <xacro:property name="arm_link02_m" value="0.2"/> <!-- in Kg -->
+  <!-- Arm Link 02 translations -->
+  <xacro:property name="arm_link02_x_trans" value="0.0147"/>
+  <xacro:property name="arm_link02_y_trans" value="0.0000"/>
+  <xacro:property name="arm_link02_z_trans" value="-0.025"/>
   <!-- Arm Link 03 dimensions -->
-  <xacro:property name="arm_link_03_length" value="1.016"/>
-  <xacro:property name="arm_link_03_width" value="0.6096"/>
-  <xacro:property name="arm_link_03_mass" value="5"/> <!-- in Kg -->
+  <xacro:property name="arm_link03_x" value="0.0280"/>
+  <xacro:property name="arm_link03_y" value="0.0650"/>
+  <xacro:property name="arm_link03_z" value="0.0485"/>
+  <xacro:property name="arm_link03_m" value="0.2"/> <!-- in Kg -->
+  <!-- Arm Link 03 translations -->
+  <xacro:property name="arm_link03_x_trans" value="0.0000"/>
+  <xacro:property name="arm_link03_y_trans" value="0.0000"/>
+  <xacro:property name="arm_link03_z_trans" value="-0.066"/>
+  <!-- Arm Link 03a dimensions -->
+  <xacro:property name="arm_link03a_x" value="0.0200"/>
+  <xacro:property name="arm_link03a_y" value="0.0200"/>
+  <xacro:property name="arm_link03a_z" value="0.4000"/>
+  <xacro:property name="arm_link03a_m" value="0.2"/> <!-- in Kg -->
+  <!-- Arm Link 03a translations -->
+  <xacro:property name="arm_link03a_x_trans" value="0.0000"/>
+  <xacro:property name="arm_link03a_y_trans" value="0.0000"/>
+  <xacro:property name="arm_link03a_z_trans" value="${-arm_link03a_z/2}"/>
   <!-- Arm Link 04 dimensions -->
-  <xacro:property name="arm_link_04_length" value="1.016"/>
-  <xacro:property name="arm_link_04_width" value="0.6096"/>
-  <xacro:property name="arm_link_04_mass" value="5"/> <!-- in Kg -->
+  <xacro:property name="arm_link04_x" value="0.0200"/>
+  <xacro:property name="arm_link04_y" value="0.0200"/>
+  <xacro:property name="arm_link04_z" value="0.0940"/>
+  <xacro:property name="arm_link04_m" value="0.2"/> <!-- in Kg -->
+  <!-- Arm Link 04 translations -->
+  <xacro:property name="arm_link04_x_trans" value="0.0200"/>
+  <xacro:property name="arm_link04_y_trans" value="0.0000"/>
+  <xacro:property name="arm_link04_z_trans" value="${-arm_link04_z/2}"/>
+  <!-- joints translations -->
+  <xacro:property name="link01_link02_x" value="0.0825"/>
+  <xacro:property name="link01_link02_y" value="0.1050"/>
+  <xacro:property name="link01_link02_z" value="0.0000"/>
+  <xacro:property name="link02_link03_x" value="0.0150"/>
+  <xacro:property name="link02_link03_y" value="0.0000"/>
+  <xacro:property name="link02_link03_z" value="-0.023"/>
+  <xacro:property name="link03_link03a_x" value="0.0000"/>
+  <xacro:property name="link03_link03a_y" value="0.0000"/>
+  <xacro:property name="link03_link03a_z" value="-0.065"/>
+  <xacro:property name="link03a_link04_x" value="0.0000"/>
+  <xacro:property name="link03a_link04_y" value="0.0000"/>
+  <xacro:property name="link03a_link04_z" value="${-arm_link03a_z}"/>
 </robot>

Commit message: Added base_link to the arm.

File: rover_arm_desc_pkg/urdf/arm_parameters.xacro (robot description, xacro)
@@ -2,4 +2,5 @@
 <robot xmlns:xacro="http://www.ros.org/wiki/xacro">
   <xacro:property name="a_link_00_name" value="arm_footprint"/>
+  <xacro:property name="a_link_0a_name" value="arm_base_link"/>
   <xacro:property name="a_link_01_name" value="arm_link_01"/>
   <xacro:property name="a_link_02_name" value="arm_link_02"/>

File: rover_arm_desc_pkg/urdf/rover_arm_macro.xacro (robot description, xacro)
@@ -11,20 +11,33 @@
     <!-- Begin - Robot Description -->
     <!-- Arm footprint -->
-    <xacro:m_link_cylinder name="${a_link_00_name}"
-                           color="gray"
-                           origin_rpy="0 0 0"
-                           origin_xyz="${world_x_origin_to_arm_x_origin}
-                                       ${world_y_origin_to_arm_y_origin}
-                                       ${world_z_origin_to_arm_z_origin}"
-                           r="${arm_foot_cyl_radius}"
-                           l="${arm_foot_cyl_height}"/>
-    <gazebo reference="${r_link_00_name}">
+    <xacro:m_link_box name="${a_link_00_name}"
+                      color="white"
+                      origin_rpy="0 0 0" origin_xyz="0 0 0"
+                      w="0.0001" d="0.0001" h="0.0001"/>
+    <gazebo reference="${a_link_00_name}">
       <material>Gazebo/White</material>
     </gazebo>
     <!-- Arm Links -->
+    <!-- Base Link -->
+    <xacro:m_link_cylinder_inertia name="${a_link_0a_name}"
+                                   color="gray"
+                                   origin_rpy="0 0 0"
+                                   origin_xyz="0 0 0"
+                                   m="0.010"
+                                   r="${arm_foot_cyl_radius}"
+                                   l="${arm_foot_cyl_height}"/>
+    <gazebo reference="${a_link_0a_name}">
+      <material>Gazebo/Black</material>
+    </gazebo>
+    <xacro:m_joint_fixed name="${a_link_00_name}__${a_link_0a_name}_joint"
+                         origin_rpy="0 0 0"
+                         origin_xyz="${world_x_origin_to_arm_x_origin}
+                                     ${world_y_origin_to_arm_y_origin}
+                                     ${world_z_origin_to_arm_z_origin}"
+                         parent="${a_link_00_name}" child="${a_link_0a_name}"/>
     <!-- Link 01 -->
     <xacro:arm_link name="${a_link_01_name}"
                     type="mesh"
-                    parent="${a_link_00_name}"
+                    parent="${a_link_0a_name}"
                     x_dim="${arm_link01_x}"
                     y_dim="${arm_link01_y}"
@@ -37,7 +50,5 @@
                     file="package://rover_arm_desc_pkg/meshes/link1.dae"
                     scale="1.0 1.0 1.0"
-                    joint_xyz="${world_x_origin_to_arm_x_origin}
-                               ${world_y_origin_to_arm_y_origin}
-                               ${world_z_origin_to_arm_z_origin}"
+                    joint_xyz="0 0 0"
                     joint_rpy="0 0 0"
                     axis_xyz="0 0 1"
@@ -133,4 +144,8 @@
                     lim_l="${-100*M_PI/157}"
                     lim_u="${25*M_PI/157}"/>
+    <!-- Rover -->
+    <gazebo>
+      <plugin name="gazebo_ros_control" filename="libgazebo_ros_control.so"/>
+    </gazebo>
   </xacro:macro>
 </robot>

Commit message: Renamed arm_base_link to arm_foot_cyl. Corrected the location of arm at Z.

File: rover_arm_desc_pkg/urdf/arm_parameters.xacro (robot description, xacro)
@@ -2,5 +2,5 @@
 <robot xmlns:xacro="http://www.ros.org/wiki/xacro">
   <xacro:property name="a_link_00_name" value="arm_footprint"/>
-  <xacro:property name="a_link_0a_name" value="arm_base_link"/>
+  <xacro:property name="a_link_0a_name" value="arm_foot_cyl"/>
   <xacro:property name="a_link_01_name" value="arm_link_01"/>
   <xacro:property name="a_link_02_name" value="arm_link_02"/>
@@ -17,5 +17,5 @@
   <xacro:property name="world_x_origin_to_arm_x_origin" value="${chassis_length/2 + arm_foot_cyl_radius}"/> <!-- Distance from world origin to mount point in X direction -->
   <xacro:property name="world_y_origin_to_arm_y_origin" value="-0.122"/> <!-- Distance from world origin to mount point in Y direction -->
-  <xacro:property name="world_z_origin_to_arm_z_origin" value="${0.562 - arm_foot_cyl_radius}"/> <!-- Distance from world origin to mount point in Z direction -->
+  <xacro:property name="world_z_origin_to_arm_z_origin" value="${0.56665-arm_foot_cyl_height}"/> <!-- Distance from world origin to mount point in Z direction -->
   <!-- Arm joints -->
   <xacro:property name="arm_link_cyl_radius" value="0.05"/>

Commit message: Raised arm along Z.

File: rover_arm_desc_pkg/urdf/arm_parameters.xacro (robot description, xacro)
@@ -17,5 +17,6 @@
   <xacro:property name="world_x_origin_to_arm_x_origin" value="${chassis_length/2 + arm_foot_cyl_radius}"/> <!-- Distance from world origin to mount point in X direction -->
   <xacro:property name="world_y_origin_to_arm_y_origin" value="-0.122"/> <!-- Distance from world origin to mount point in Y direction -->
-  <xacro:property name="world_z_origin_to_arm_z_origin" value="${0.56665-arm_foot_cyl_height}"/> <!-- Distance from world origin to mount point in Z direction -->
+  <!-- <xacro:property name="world_z_origin_to_arm_z_origin" value="${0.56665-arm_foot_cyl_height}"/> --> <!-- Distance from world origin to mount point in Z direction -->
+  <xacro:property name="world_z_origin_to_arm_z_origin" value="${0.59+arm_foot_cyl_height}"/>
   <!-- Arm joints -->
   <xacro:property name="arm_link_cyl_radius" value="0.05"/>

Commit message: Change the mesh of link3 to match actual arm. Reduced length of link3a. Corrected the Z value of arm position wrt rover.

File: rover_arm_desc_pkg/urdf/arm_parameters.xacro (robot description, xacro)
@@ -17,6 +17,5 @@
   <xacro:property name="world_x_origin_to_arm_x_origin" value="${chassis_length/2 + arm_foot_cyl_radius}"/> <!-- Distance from world origin to mount point in X direction -->
   <xacro:property name="world_y_origin_to_arm_y_origin" value="-0.122"/> <!-- Distance from world origin to mount point in Y direction -->
-  <!-- <xacro:property name="world_z_origin_to_arm_z_origin" value="${0.56665-arm_foot_cyl_height}"/> --> <!-- Distance from world origin to mount point in Z direction -->
-  <xacro:property name="world_z_origin_to_arm_z_origin" value="${0.59+arm_foot_cyl_height}"/>
+  <xacro:property name="world_z_origin_to_arm_z_origin" value="${0.56665-arm_foot_cyl_height}"/> <!-- Distance from world origin to mount point in Z direction -->
   <!-- Arm joints -->
   <xacro:property name="arm_link_cyl_radius" value="0.05"/>
@@ -49,9 +48,9 @@
   <xacro:property name="arm_link03_x_trans" value="0.0000"/>
   <xacro:property name="arm_link03_y_trans" value="0.0000"/>
-  <xacro:property name="arm_link03_z_trans" value="-0.066"/>
+  <xacro:property name="arm_link03_z_trans" value="-0.095"/>
   <!-- Arm Link 03a dimensions -->
   <xacro:property name="arm_link03a_x" value="0.0200"/>
   <xacro:property name="arm_link03a_y" value="0.0200"/>
-  <xacro:property name="arm_link03a_z" value="0.4000"/>
+  <xacro:property name="arm_link03a_z" value="0.1900"/>
   <xacro:property name="arm_link03a_m" value="0.2"/> <!-- in Kg -->
   <!-- Arm Link 03a translations -->
@@ -77,5 +76,5 @@
   <xacro:property name="link03_link03a_x" value="0.0000"/>
   <xacro:property name="link03_link03a_y" value="0.0000"/>
-  <xacro:property name="link03_link03a_z" value="-0.065"/>
+  <xacro:property name="link03_link03a_z" value="${arm_link03_z_trans}"/>
   <xacro:property name="link03a_link04_x" value="0.0000"/>
   <xacro:property name="link03a_link04_y" value="0.0000"/>

Commit message: Lowered arm wrt rover.

File: rover_arm_desc_pkg/urdf/arm_parameters.xacro (robot description, xacro)
@@ -17,5 +17,6 @@
   <xacro:property name="world_x_origin_to_arm_x_origin" value="${chassis_length/2 + arm_foot_cyl_radius}"/> <!-- Distance from world origin to mount point in X direction -->
   <xacro:property name="world_y_origin_to_arm_y_origin" value="-0.122"/> <!-- Distance from world origin to mount point in Y direction -->
-  <xacro:property name="world_z_origin_to_arm_z_origin" value="${0.56665-arm_foot_cyl_height}"/> <!-- Distance from world origin to mount point in Z direction -->
+  <!-- <xacro:property name="world_z_origin_to_arm_z_origin" value="${0.56665-arm_foot_cyl_height}"/> --> <!-- Distance from world origin to mount point in Z direction -->
+  <xacro:property name="world_z_origin_to_arm_z_origin" value="0.433"/> <!-- Distance from world origin to mount point in Z direction -->
   <!-- Arm joints -->
   <xacro:property name="arm_link_cyl_radius" value="0.05"/>
