Commit message: Renamed the package.

File: rover_arm_resources_pkg/urdf/links_joints.xacro (robot description, xacro)
@@ -1,4 +1,7 @@
 <?xml version="1.0"?>
 <robot xmlns:xacro="http://www.ros.org/wiki/xacro">
+  <!-- Begin - Include -->
+    <xacro:include filename="$(find rover_arm_resources_pkg)/urdf/common_materials.xacro"/>
+  <!-- End - Include -->
   <!-- Joint Macro -->
   <!-- fixed joint -->
@@ -52,5 +55,5 @@
   </xacro:macro>
   <!-- Cylinder link Macro without inertia -->
-  <xacro:macro name="m_link_cylinder" params="name color origin_xyz origin_rpy r l">
+  <xacro:macro name="m_link_cylinder" params="name origin_xyz origin_rpy r l">
     <link name="${name}">
       <visual>
@@ -59,10 +62,10 @@
           <cylinder radius="${r}" length="${l}"/>
         </geometry>
-        <material name="${color}"/>
+        <xacro:material_gray/>
       </visual>
     </link>
   </xacro:macro>
   <!-- Cylinder link Macro with inertia -->
-  <xacro:macro name="m_link_cylinder_inertia" params="name color origin_xyz origin_rpy r l m">
+  <xacro:macro name="m_link_cylinder_inertia" params="name origin_xyz origin_rpy r l m">
     <link name="${name}">
       <inertial>
@@ -84,10 +87,10 @@
           <cylinder radius="${r}" length="${l}"/>
         </geometry>
-        <material name="${color}"/>
+        <xacro:material_darkgray/>
       </visual>
     </link>
   </xacro:macro>
   <!-- Box link Macro without inertia -->
-  <xacro:macro name="m_link_box" params="name color origin_xyz origin_rpy w d h">
+  <xacro:macro name="m_link_box" params="name origin_xyz origin_rpy w d h">
     <link name="${name}">
       <visual>
@@ -96,10 +99,10 @@
           <box size="${w} ${d} ${h}"/>
         </geometry>
-        <material name="${color}"/>
+        <xacro:material_white/>
       </visual>
     </link>
   </xacro:macro>
   <!-- Box link Macro with inertia -->
-  <xacro:macro name="m_link_box_inertia" params="name color origin_xyz origin_rpy m w d h">
+  <xacro:macro name="m_link_box_inertia" params="name origin_xyz origin_rpy m w d h">
     <link name="${name}">
       <inertial>
@@ -121,5 +124,5 @@
           <box size="${w} ${d} ${h}"/>
         </geometry>
-        <material name="${color}"/>
+        <xacro:material_clay_brown/>
       </visual>
     </link>

Commit message: Corrected box link visual & collision

File: rover_arm_resources_pkg/urdf/links_joints.xacro (robot description, xacro)
@@ -121,5 +121,5 @@
         <origin rpy="${origin_rpy}" xyz="${origin_xyz}"/>
         <geometry>
-          <box size="${w} ${d} ${h}"/>
+          <box size="${d} ${w} ${h}"/>
         </geometry>
       </collision>
@@ -127,5 +127,5 @@
         <origin rpy="${origin_rpy}" xyz="${origin_xyz}"/>
         <geometry>
-          <box size="${w} ${d} ${h}"/>
+          <box size="${d} ${w} ${h}"/>
         </geometry>
         <xacro:material_clay_brown/>
